File: board_sierra/board_sierra.sch (KiCad schematic (older format))
At the start: 121 parts, among them J1 Conn_01x08, M1 CY15B102Q, M2 CY15B102Q, M3 CY15B102Q, M4 S25FLxL, M5 S25FLxL, M6 S25FLxL, SW1 SW_DPDT_x2, SW2 SW_Push_Dual, U1 TCAN1051, U2 TCAN1051, U3 STM32L496QGIx, U4 ADuM142E, U5 ADuM142E, U6 ADuM142E, U7 ADuM142E, U8 LSF0102-Q1, U9 LSF0102-Q1, Y1 ABS07AIG, Y2 SiT8924

Commit message: before meeting
Parts:
- removed C47, C48, C49, C50, C51, C52, C53, C54, C? (x4): 100n, symbol Device:C_Small
- removed U4, U5, U6, U7: ADuM142E, Package_SO:QSOP-16_3.9x4.9mm_P0.635mm, symbol VST104:digital_isolator_4_2x2
- removed U? (x2): ADuM141E, Package_SO:QSOP-16_3.9x4.9mm_P0.635mm, symbol VST104:digital_isolator_4_3x1
- added C47, C48, C49, C50, C51, C52, C53, C54, C57, C? (x10): 100n, symbol Device:C
- added R20, R21: 200K, symbol Device:R
- added U10, U11, U12, U13, U14, U4, U5, U6, U7, U? (x10): DGQ2788A, VST104_footprints:mini_QFN-16-1.8x2.6mm, symbol VST104:DGQ2788A
Connections:
- net +3V3: now also C47.2, C48.2, C49.2, C50.2, C51.2, C52.2, C54.2, C57.2, C?.2, C?.2, C?.2, C?.2, C?.2, C?.2, C?.2, C?.2, C?.2, C?.2, U10.10 (VCC), U11.10 (VCC), U13.10 (VCC), U14.10 (VCC), U4.10 (VCC), U5.10 (VCC), U6.10 (VCC), U7.10 (VCC), U?.10 (VCC), U?.10 (VCC), U?.10 (VCC), U?.10 (VCC), U?.10 (VCC), U?.10 (VCC), U?.10 (VCC), U?.10 (VCC), U?.10 (VCC), U?.10 (VCC)
- net +5V: now also C53.2, U12.10 (VCC)
- net CAN1_EN: now also U12.14 (EN12); no longer U1.8 (STBY)
- net CAN2_EN: now also U12.6 (EN34); no longer U2.8 (STBY)
- net CAN_1_H: now also U12.11 (NO1); no longer C19.2, L2.2, R7.1
- net CAN_1_L: now also U12.15 (NO2); no longer C20.2, L2.3, R8.1
- net CAN_2_H: now also U12.3 (NO3); no longer C22.2, L3.2, R11.1
- net CAN_2_L: now also U12.7 (NO4); no longer C23.2, L3.3, R12.1
- net CPU_SELECT: now also U?.3 (NO3)
- net GLO_FAULT: now also U?.15 (NO2)
- net GLO_SYNC: now also U?.11 (NO1)
- net GND: now also C47.1, C48.1, C49.1, C50.1, C51.1, C52.1, C53.1, C54.1, C57.1, C?.1, C?.1, C?.1, C?.1, C?.1, C?.1, C?.1, C?.1, C?.1, C?.1, R20.2, R21.2, U10.2 (GND), U11.2 (GND), U12.2 (GND), U13.2 (GND), U14.2 (GND), U4.2 (GND), U5.2 (GND), U6.2 (GND), U7.2 (GND), U?.2 (GND), U?.2 (GND), U?.2 (GND), U?.2 (GND), U?.2 (GND), U?.2 (GND), U?.2 (GND), U?.2 (GND), U?.2 (GND), U?.2 (GND)
- net I2C4_SDA: no longer R6.2, TS1.1 (SDA), TS2.1 (SDA), TS3.1 (SDA), TS4.1 (SDA), TS5.1 (SDA), TS6.1 (SDA), TS7.1 (SDA), TS8.1 (SDA)
- net SPI1_CLK: now also U10.4 (COM3)
- net SPI1_CS1: now also U10.8 (COM4)
- net SPI1_EN: now also U10.14 (EN12), U10.6 (EN34)
- net SPI1_MISO: now also U10.16 (COM2)
- net SPI1_MOSI: now also U10.12 (COM1)
- net SPI2_CLK: now also U11.4 (COM3)
- net SPI2_CS1: now also U11.8 (COM4)
- net SPI2_EN: now also U11.14 (EN12), U11.6 (EN34)
- net SPI2_MISO: now also U11.16 (COM2)
- net SPI2_MOSI: now also U11.12 (COM1)
- net SPI_1_CLK: now also U10.3 (NO3)
- net SPI_1_CS1: now also U10.7 (NO4)
- net SPI_1_CS2: now also U?.11 (NO1)
- net SPI_1_MISO: now also U10.15 (NO2)
- net SPI_1_MOSI: now also U10.11 (NO1)
- net SPI_2_CLK: now also U11.3 (NO3)
- net SPI_2_CS1: now also U11.7 (NO4)
- net SPI_2_CS2: now also U?.3 (NO3)
- net SPI_2_MISO: now also U11.15 (NO2)
- net SPI_2_MOSI: now also U11.11 (NO1)
- net UART1_CTS: now also U4.4 (COM3)
- net UART1_EN: now also U4.14 (EN12), U4.6 (EN34)
- net UART1_RST: now also U4.8 (COM4)
- net UART1_RX: now also U4.16 (COM2)
- net UART1_TX: now also U4.12 (COM1)
- net UART2_CTS: now also U5.4 (COM3)
- net UART2_EN: now also U5.14 (EN12), U5.6 (EN34)
- net UART2_RST: now also U5.8 (COM4)
- net UART2_RX: now also U5.16 (COM2)
- net UART2_TX: now also U5.12 (COM1)
- net UART3_CTS: now also U6.4 (COM3)
- net UART3_EN: now also U6.14 (EN12), U6.6 (EN34)
- net UART3_RST: now also U6.8 (COM4)
- net UART3_RX: now also U6.16 (COM2)
- net UART3_TX: now also U6.12 (COM1)
- net UART4_CTS: now also U7.4 (COM3)
- net UART4_EN: now also U7.14 (EN12), U7.6 (EN34)
- net UART4_RST: now also U7.8 (COM4)
- net UART4_RX: now also U7.16 (COM2)
- net UART4_TX: now also U7.12 (COM1)
- net UART_1_CTS: now also U6.3 (NO3)
- net UART_1_RTS: now also U6.7 (NO4)
- net UART_1_RX: now also U6.15 (NO2)
- net UART_1_TX: now also U6.11 (NO1)
- net UART_2_CTS: now also U7.3 (NO3)
- net UART_2_RTS: now also U7.7 (NO4)
- net UART_2_RX: now also U7.15 (NO2)
- net UART_2_TX: now also U7.11 (NO1)
- net UART_RCS_1_CTS: now also U4.3 (NO3)
- net UART_RCS_1_RTS: now also U4.7 (NO4)
- net UART_RCS_1_RX: now also U4.15 (NO2)
- net UART_RCS_1_TX: now also U4.11 (NO1)
- net UART_RCS_2_CTS: now also U5.3 (NO3)
- net UART_RCS_2_RTS: now also U5.7 (NO4)
- net UART_RCS_2_RX: now also U5.15 (NO2)
- net UART_RCS_2_TX: now also U5.11 (NO1)
- net H2_1: now reaches H2.1 (Pin_1)
- net H2_1: now also U?.11 (NO1)
- net H2_10: now reaches H2.10 (Pin_10)
- net H2_10: now also U?.7 (NO4)
- net H2_2: now reaches H2.2 (Pin_2)
- net H2_2: now also U?.3 (NO3)
- net H2_3: now reaches H2.3 (Pin_3)
- net H2_3: now also U?.15 (NO2)
- net H2_4: now reaches H2.4 (Pin_4)
- net H2_4: now also U?.7 (NO4)
- net H2_41: now reaches H2.41 (Pin_41)
- net H2_41: now also U?.11 (NO1)
- net H2_42: now reaches H2.42 (Pin_42)
- net H2_42: now also U?.3 (NO3)
- net H2_43: now reaches H2.43 (Pin_43)
- net H2_43: now also U?.15 (NO2)
- net H2_44: now reaches H2.44 (Pin_44)
- net H2_44: now also U?.7 (NO4)
- net H2_45: now reaches H2.45 (Pin_45)
- net H2_45: now also U?.11 (NO1)
- net H2_46: now reaches H2.46 (Pin_46)
- net H2_46: now also U?.3 (NO3)
- net H2_47: now reaches H2.47 (Pin_47)
- net H2_47: now also U?.15 (NO2)
- net H2_48: now reaches H2.48 (Pin_48)
- net H2_48: now also U?.7 (NO4)
- net H2_49: now reaches H2.49 (Pin_49)
- net H2_49: now also U?.11 (NO1)
- net H2_5: now reaches H2.5 (Pin_5)
- net H2_5: now also U?.11 (NO1)
- net H2_50: now reaches H2.50 (Pin_50)
- net H2_50: now also U?.3 (NO3)
- net H2_51: now reaches H2.51 (Pin_51)
- net H2_51: now also U?.15 (NO2)
- net H2_52: now reaches H2.52 (Pin_52)
- net H2_52: now also U?.7 (NO4)
- net H2_6: now reaches H2.6 (Pin_6)
- net H2_6: now also U?.3 (NO3)
- net H2_7: now reaches H2.7 (Pin_7)
- net H2_7: now also U?.15 (NO2)
- net H2_8: now reaches H2.8 (Pin_8)
- net H2_8: now also U?.7 (NO4)
- net H1_1: now reaches H1.1 (Pin_1)
- net H1_1: now also U?.11 (NO1)
- net H1_10: now reaches H1.10 (Pin_10)
- net H1_10: now also U?.15 (NO2)
- net H1_2: now reaches H1.2 (Pin_2)
- net H1_2: now also U?.3 (NO3)
- net H1_3: now reaches H1.3 (Pin_3)
- net H1_3: now also U?.15 (NO2)
- net H1_4: now reaches H1.4 (Pin_4)
- net H1_4: now also U?.7 (NO4)
- net H1_41: now reaches H1.41 (Pin_41)
- net H1_41: now also U?.11 (NO1)
- net H1_42: now reaches H1.42 (Pin_42)
- net H1_42: now also U?.3 (NO3)
- net H1_43: now reaches H1.43 (Pin_43)
- net H1_43: now also U?.15 (NO2)
- net H1_44: now reaches H1.44 (Pin_44)
- net H1_44: now also U?.7 (NO4)
- net H1_45: now reaches H1.45 (Pin_45)
- net H1_45: now also U13.11 (NO1)
- net H1_46: now reaches H1.46 (Pin_46)
- net H1_46: now also U13.3 (NO3)
- net H1_47: now reaches H1.47 (Pin_47)
- net H1_47: now also U13.15 (NO2)
- net H1_48: now reaches H1.48 (Pin_48)
- net H1_48: now also U13.7 (NO4)
- net H1_49: now reaches H1.49 (Pin_49)
- net H1_49: now also U14.11 (NO1)
- net H1_5: now reaches H1.5 (Pin_5)
- net H1_5: now also U?.11 (NO1)
- net H1_50: now reaches H1.50 (Pin_50)
- net H1_50: now also U14.3 (NO3)
- net H1_51: now reaches H1.51 (Pin_51)
- net H1_51: now also U14.15 (NO2)
- net H1_52: now reaches H1.52 (Pin_52)
- net H1_52: now also U14.7 (NO4)
- net H1_6: now reaches H1.6 (Pin_6)
- net H1_6: now also U?.3 (NO3)
- net H1_7: now reaches H1.7 (Pin_7)
- net H1_7: now also U?.15 (NO2)
- net H1_8: now reaches H1.8 (Pin_8)
- net H1_8: now also U?.7 (NO4)
- net CPU_WD_2: no longer names the net of H1.36 (Pin_36)
- net GLO_KS_2: no longer names the net of H1.38 (Pin_38)
- net GLO_KS_3: no longer names the net of H1.39 (Pin_39)
- net GLO_KS_4: no longer names the net of H1.40 (Pin_40)
- net GLO_KS_5: no longer names the net of H2.37 (Pin_37)
- net GLO_KS_6: no longer names the net of H2.38 (Pin_38)
- net GLO_KS_7: no longer names the net of H2.39 (Pin_39)
- net GLO_KS_8: no longer names the net of H2.40 (Pin_40)
- new net: R20.1, U1.8 (STBY)
- new net: R21.1, U2.8 (STBY)
- new net: R6.2, TS1.1 (SDA), TS2.1 (SDA), TS3.1 (SDA), TS4.1 (SDA), TS5.1 (SDA), TS6.1 (SDA), TS7.1 (SDA), TS8.1 (SDA)
- new net: C22.2, L3.2, R11.1, U12.4 (COM3)
- new net: C23.2, L3.3, R12.1, U12.8 (COM4)
- new net: C19.2, L2.2, R7.1, U12.12 (COM1)
- new net: C20.2, L2.3, R8.1, U12.16 (COM2)
- new net FAULT: U?.16 (COM2)
- new net GLO_EN: U?.14 (EN12), U?.6 (EN34)
- new net H12_EN: U?.14 (EN12), U?.6 (EN34)
- new net H1_1-4_EN: U?.14 (EN12), U?.6 (EN34)
- new net H1_10_IO: U?.16 (COM2)
- new net H1_1_IO: U?.12 (COM1)
- new net H1_2_IO: U?.4 (COM3)
- new net H1_3_IO: U?.16 (COM2)
- new net H1_41-44_EN: U?.14 (EN12), U?.6 (EN34)
- new net H1_41_IO: U?.12 (COM1)
- new net H1_42_IO: U?.4 (COM3)
- new net H1_43_IO: U?.16 (COM2)
- new net H1_44_IO: U?.8 (COM4)
- new net H1_45-48_EN: U13.14 (EN12), U13.6 (EN34)
- new net H1_45_IO: U13.12 (COM1)
- new net H1_46_IO: U13.4 (COM3)
- new net H1_47_IO: U13.16 (COM2)
- new net H1_48_IO: U13.8 (COM4)
- new net H1_49-52_EN: U14.14 (EN12), U14.6 (EN34)
- new net H1_49_IO: U14.12 (COM1)
- new net H1_4_IO: U?.8 (COM4)
- new net H1_5-8_EN: U?.14 (EN12), U?.6 (EN34)
- new net H1_50_IO: U14.4 (COM3)
- new net H1_51_IO: U14.16 (COM2)
- new net H1_52_IO: U14.8 (COM4)
- new net H1_5_IO: U?.12 (COM1)
- new net H1_6_IO: U?.4 (COM3)
- new net H1_7_IO: U?.16 (COM2)
- new net H1_8_IO: U?.8 (COM4)
- new net H2_1-4_EN: U?.14 (EN12), U?.6 (EN34)
- new net H2_10_IO: U?.8 (COM4)
- new net H2_1_IO: U?.12 (COM1)
- new net H2_2_IO: U?.4 (COM3)
- new net H2_3_IO: U?.16 (COM2)
- new net H2_41-44_EN: U?.14 (EN12), U?.6 (EN34)
- new net H2_41_IO: U?.12 (COM1)
- new net H2_42_IO: U?.4 (COM3)
- new net H2_43_IO: U?.16 (COM2)
- new net H2_44_IO: U?.8 (COM4)
- new net H2_45-48_EN: U?.14 (EN12), U?.6 (EN34)
- new net H2_45_IO: U?.12 (COM1)
- new net H2_46_IO: U?.4 (COM3)
- new net H2_47_IO: U?.16 (COM2)
- new net H2_48_IO: U?.8 (COM4)
- new net H2_49-52_EN: U?.14 (EN12), U?.6 (EN34)
- new net H2_49_IO: U?.12 (COM1)
- new net H2_4_IO: U?.8 (COM4)
- new net H2_5-8_EN: U?.14 (EN12), U?.6 (EN34)
- new net H2_50_IO: U?.4 (COM3)
- new net H2_51_IO: U?.16 (COM2)
- new net H2_52_IO: U?.8 (COM4)
- new net H2_5_IO: U?.12 (COM1)
- new net H2_6_IO: U?.4 (COM3)
- new net H2_7_IO: U?.16 (COM2)
- new net H2_8_IO: U?.8 (COM4)
- new net SELECT: U?.4 (COM3)
- new net SPI1_CS2: U?.12 (COM1)
- new net SPI2_CS2: U?.4 (COM3)
- new net SYNC: U?.12 (COM1)
- no-connect marks 12 -> 98
Other:
- note added: "Global signals isolator"
- note added: "Radio subs. UART isolators"
- note added: "SPI isolators"
- note added: "UART isolators"
- note added: "User IO H1&H2 isolators"
- note added: "User IO bottom H1 isolators"
- note added: "User IO bottom H2 isolators"
- note added: "User IO top H1 isolators"
- note added: "User IO top H2 isolators"
- note removed: "Radio subs. UART isolator"
- note removed: "SPI isolator"
- note removed: "UART isolator"
- moved on the sheet: C10, C11, C12, C13, C14, C15, C16, C17, C18, C19, C20, C21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
