File: board_sierra/board_sierra.sch (KiCad schematic (older format))
At the start: 143 parts, among them J1 Conn_01x08, M1 CY15B102Q, M2 CY15B102Q, M3 CY15B102Q, M4 S25FLxL, M5 S25FLxL, M6 S25FLxL, SW1 SW_DPDT_x2, SW2 SW_Push_Dual, U1 TCAN1051, U10 DGQ2788A, U11 DGQ2788A, U12 DGQ2788A, U13 DGQ2788A, U14 DGQ2788A, U2 TCAN1051, U3 STM32L496QGIx, U4 DGQ2788A, U5 DGQ2788A, U6 DGQ2788A, U7 DGQ2788A, U8 LSF0102-Q1, U9 LSF0102-Q1, Y1 ABS07AIG, Y2 SiT8924

Commit message: night update
Parts:
- removed C55, C56: 100n, symbol Device:C_Small
- removed U8, U9: LSF0102-Q1, Package_SO:VSSOP-8_2.3x2mm_P0.5mm, symbol VST104:level_shifter
- added C55: 10n, Capacitor_SMD:C_0402_1005Metric, symbol Device:C
- added R22, R23, R24, R25, R26, R27, R28, R29, R30, R31, R32, R33, R34, R35, R36, R37, R38, R39, R40, R41: 200k, Resistor_SMD:R_0402_1005Metric, symbol Device:R
- added U8: DGQ2788A, VST104_footprints:mini_QFN-16-1.8x2.6mm, symbol VST104:DGQ2788A
- C1, C10, C11, C12, C13, C14, C15, C16, C17, C18, C19, C2, C20, C21, C22, C23, C24, C25, C26, C27, C28, C29, C3, C30, C31, C32, C33, C34, C35, C36, C37, C38, C39, C4, C40, C41, C42, C43, C44, C45, C46, C5, C6, C7, C8, C9: footprint Capacitor_SMD:C_0603_1608Metric -> Capacitor_SMD:C_0402_1005Metric
- C47, C48, C49, C50, C51, C52, C54, C57: value 100n -> 10n; footprint (none) -> Capacitor_SMD:C_0402_1005Metric
- C53: footprint (none) -> Capacitor_SMD:C_0402_1005Metric
- C58, C59, C60, C61, C62, C63, C64, C65, C66, C67: renamed from C?; value 100n -> 10n; footprint (none) -> Capacitor_SMD:C_0402_1005Metric
- M4, M5, M6: footprint VST104_footprints:WSON-8-EP-6.0x8.0mm -> VST104_footprints:WSON-8_EP_6.0x8.0mm
- R1, R10, R11, R12, R13, R14, R15, R16, R17, R18, R2, R3, R4, R5, R6, R7, R8: footprint Resistor_SMD:R_0603_1608Metric -> Resistor_SMD:R_0402_1005Metric
- R19, R20, R21, R9: footprint (none) -> Resistor_SMD:R_0402_1005Metric
- gave numbers to parts that had none: 10
Connections:
- net labels added: GLO_EN_OU, UART5_RX, UART5_TX
- net labels removed: GLO_EN, SUP_UNREG
- wire segments 1144 -> 1146
- no-connect marks 98 -> 104
Other:
- note added: "I2C isolator"
- note removed: "I2C level shifter and isolator"
- moved on the sheet: C1, C2, C3, C36, C37, C38, C39, C4, C40, C41, C42, C43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

Commit message: before professor check
Parts:
- removed C24, C25, C26, C33, C34, C35: 100n, Capacitor_SMD:C_0402_1005Metric, symbol Device:C
- removed M1, M2, M3: CY15B102Q, Package_SO:SOIC-8_5.275x5.275mm_P1.27mm, symbol VST104:memory
- removed M4, M5, M6: S25FLxL, VST104_footprints:WSON-8_EP_6.0x8.0mm, symbol board_sierra-rescue:S25FLxL-VST104
- removed R13, R14, R15, R17, R18: 10k, Resistor_SMD:R_0402_1005Metric, symbol Device:R
- removed U1, U2: TCAN1051, Package_SON:WSON-8-1EP_3x3mm_P0.5mm_EP1.6x2.0mm, symbol VST104:TCAN1051
- added C56: 10n, Capacitor_SMD:C_0402_1005Metric, symbol Device:C
- added C68, C70, C72, C73: 100n, Capacitor_SMD:C_0402_1005Metric, symbol Device:C
- added C69, C71: C, Capacitor_SMD:C_0402_1005Metric, symbol Device:C
- added C74, C75: 100u, Capacitor_SMD:C_0402_1005Metric, symbol Device:C
- added C? (x6): 100n, symbol Device:C_Small
- added M? (x3): CY15B102Q, symbol VST104:CY15B102Q
- added M? (x3): S25FL256L, VST104_footprints:FAC024, symbol VST104:S25FL256L
- added R42: 200k, Resistor_SMD:R_0402_1005Metric, symbol Device:R
- added R43, R44, R45, R46, R47, R48: R, Resistor_SMD:R_0402_1005Metric, symbol Device:R_Small
- added R49, R50, R51, R52: R, Resistor_SMD:R_0402_1005Metric, symbol Device:R
- added R? (x5): 10k, Resistor_SMD:R_0402_1005Metric, symbol Device:R
- added U1, U2: TCAN1051-Q1, symbol VST104:TCAN1051-Q1
- added U25, U26: TPS25940-Q1, symbol VST104:TPS25940-Q1
- added U27, U28: TPS22965-Q1, Package_SON:WSON-8-1EP_2x2mm_P0.5mm_EP0.9x1.6mm, symbol VST104:TPS22965-Q1
- added U9: DGQ2788A, VST104_footprints:mini_QFN-16-1.8x2.6mm, symbol VST104:DGQ2788A
Connections:
- net labels added: EFSE_3_VOUT, EFSE_5_VOUT, I2C4_EN, QSPI_B1_RST, RS, SC, SPI_A, SPI_B, SPI_C, SPI_CLK, SPI_HOLD, SPI_SI, SPI_SO, SPI_WP, SUP_3v3
- net labels removed: QSPI_B2_0, QSPI_B2_1, QSPI_B2_2, QSPI_B2_3
- wire segments 1146 -> 1213
- no-connect marks 104 -> 113
Other:
- note added: "Bank 1 : triple redundant FLASH memory"
- note added: "Power UV, OV, current protection and KillSwitch\n"
- note added: "Triple redundant F-RAM memory"
- note removed: "Bank 1 : triple redundant F-RAM memory"
- note removed: "Bank 2 : triple redundant FLASH memory"
- moved on the sheet: C1, C10, C11, C12, C13, C14, C15, C16, C17, C18, C19, C2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

Commit message: consultation
Parts:
- removed C56: 10n, Capacitor_SMD:C_0402_1005Metric, symbol Device:C
- removed D1: VCAN16A2, Package_TO_SOT_SMD:SOT-323_SC-70, symbol Device:D_TVS_x2_AAC
- removed L2: L, VST104_footprints:CMCH_1210, symbol Device:L_Core_Iron_Coupled_Small_1243
- removed U9: DGQ2788A, VST104_footprints:mini_QFN-16-1.8x2.6mm, symbol VST104:DGQ2788A
- added U22: TPS22965-Q1, Package_SON:WSON-8-1EP_2x2mm_P0.5mm_EP0.9x1.6mm, symbol VST104:TPS22965-Q1
- U26: renamed from U1; footprint (none) -> Package_SON:WSON-8-1EP_3x3mm_P0.5mm_EP1.6x2.0mm
- U27: renamed from U2; footprint (none) -> Package_SON:WSON-8-1EP_3x3mm_P0.5mm_EP1.6x2.0mm
- gave numbers to parts that had none: 17
- renumbered C8 to C1, C38 to C10, C4 to C11, C3 to C12, C2 to C13, C1 to C14, C7 to C15, C43 to C16, C44 to C17, C45 to C18, C46 to C19, C39 to C2, C5 to C20, C6 to C21, C49 to C22, C50 to C23, C9 to C24, C10 to C25, C60 to C26, C54 to C27, C57 to C28, C61 to C29, C40 to C3, C62 to C30, C63 to C31, C11 to C32, C68 to C33, C69 to C34, C70 to C35, C71 to C36, C55 to C37, C64 to C38, C65 to C39, C41 to C4, C72 to C43, C73 to C44, C74 to C45, C75 to C46, C58 to C47, C51 to C48, C52 to C49, C42 to C5, C59 to C53, C66 to C54, C67 to C55, C14 to C56, C17 to C57, C15 to C58, C18 to C59, C47 to C6, C12 to C60, C30 to C61, C16 to C62, C19 to C63, C20 to C64, C31 to C65, C27 to C66, C21 to C67, C22 to C68, C23 to C69, C48 to C7, C13 to C70, C28 to C71, C29 to C72, C32 to C73, C53 to C74, C36 to C8, C37 to C9, D2 to D1, L3 to L2, MH4 to MH3, MH3 to MH4, R22 to R1, R2 to R10, R35 to R11, R36 to R12, R37 to R13, R4 to R14, R9 to R18, R23 to R2, R38 to R20, R39 to R21, R43 to R22, R44 to R23, R45 to R24, R46 to R25, R47 to R26, R48 to R27, R49 to R28, R50 to R29, R1 to R3, R51 to R30, R52 to R31, R28 to R32, R26 to R33, R27 to R34, R16 to R35, R29 to R38, R40 to R39, R24 to R4, R41 to R40, R5 to R41, R6 to R43, R20 to R44, R21 to R45, R7 to R46, R8 to R47, R11 to R48, R12 to R49, R25 to R5, R30 to R50, R31 to R51, R10 to R52, R32 to R6, R33 to R7, R34 to R8, R3 to R9, SW2 to SW1, SW1 to SW2, TS5 to TS2, TS6 to TS3, TS2 to TS4, TS7 to TS5, TS3 to TS6, TS4 to TS7, U4 to U1, U19 to U10, U20 to U11, U8 to U12, U21 to U13, U22 to U14, U25 to U15, U26 to U16, U27 to U17, U28 to U18, U15 to U19, U5 to U2, U10 to U20, U11 to U21, U16 to U23, U23 to U24, U24 to U25, U12 to U28, U6 to U4, U7 to U5, U17 to U6, U13 to U7, U14 to U8, U18 to U9
Connections:
- wire segments 1213 -> 1207
- no-connect marks 113 -> 106
Other:
- moved on the sheet: C62, C63, C64, R42, R46, R47

Commit message: schematic checked, new footprints created, simulations on the way
Parts:
- removed D1: VCAN16A2, Package_TO_SOT_SMD:SOT-323_SC-70, symbol Device:D_TVS_x2_AAC
- removed L2: L, VST104_footprints:CMCH_1210, symbol Device:L_Core_Iron_Coupled_Small_1243
- C1, C10, C11, C12, C13, C14, C15, C16, C17, C18, C19, C2, C20, C21, C22, C23, C24, C25, C26, C27, C28, C29, C3, C30, C31, C32, C33, C34, C35, C36, C37, C38, C39, C4, C43, C44, C45, C46, C47, C48, C49, C5, C53, C54, C55, C56, C57, C58, C59, C6, C60, C61, C62, C63, C64, C65, C66, C67, C68, C69, C7, C70, C71, C72, C73, C74, C8, C9: footprint Capacitor_SMD:C_0402_1005Metric -> VST104_footprints:C_SMD_0402_wave
- C40, C41, C42, C50, C51, C52: footprint (none) -> VST104_footprints:C_SMD_0402_wave
- FB1, L1: footprint Inductor_SMD:L_0603_1608Metric -> (none)
- H1, H2: footprint Connector_Samtec_HLE_THT:Samtec_HLE-126-02-xx-DV-TE_2x26_P2.54mm_Horizontal -> (none)
- J1: footprint VST104_footprints:5014610891 -> (none)
- M4, M5, M6: footprint VST104_footprints:FAC024 -> (none)
- MH1, MH2, MH3, MH4: footprint MountingHole:MountingHole_3.2mm_M3_Pad_Via -> (none)
- R1, R10, R11, R12, R13, R14, R15, R16, R17, R18, R19, R2, R20, R21, R22, R23, R24, R25, R26, R27, R28, R29, R3, R30, R31, R32, R33, R34, R35, R36, R37, R38, R39, R4, R40, R41, R42, R43, R44, R45, R46, R47, R48, R49, R5, R50, R51, R52, R6, R7, R8, R9: footprint Resistor_SMD:R_0402_1005Metric -> VST104_footprints:R_SMD_0402_wave
- SW1: footprint VST104_footprints:EVPBB0AAB000 -> (none)
- TS1, TS2, TS3, TS4, TS5, TS6, TS7, TS8: footprint Package_DFN_QFN:DFN-8-1EP_3x2mm_P0.5mm_EP1.75x1.45mm -> (none)
- U1, U19, U2, U20, U21, U23, U24, U25, U28: footprint VST104_footprints:mini_QFN-16-1.8x2.6mm -> (none)
- U17, U18, U22: footprint Package_SON:WSON-8-1EP_2x2mm_P0.5mm_EP0.9x1.6mm -> (none)
- U26, U27: footprint Package_SON:WSON-8-1EP_3x3mm_P0.5mm_EP1.6x2.0mm -> VST104_footprints:VSON-8_3.0x3.0mm_EPV
- U3: footprint Package_BGA:UFBGA-132_7x7mm_Layout12x12_P0.5mm -> VST104_footprints:UFBGA-132_7.0x7.0mm
- Y1: footprint Crystal:Crystal_SMD_3215-2Pin_3.2x1.5mm -> (none)
- Y2: footprint Crystal:Crystal_SMD_2016-4Pin_2.0x1.6mm -> (none)
Connections:
- wire segments 1207 -> 1194
Other:
- moved on the sheet: C45, C46, C56, C57, C58, C59, C62, C63, C64, C67, J1, MH1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

Commit message: UPDATUS MAJORUS
Parts:
- removed C33, C44: 100n, VST104_footprints:C_SMD_0402_wave, symbol Device:C
- removed C36: C, VST104_footprints:C_SMD_0402_wave, symbol Device:C
- removed C46: 100u, VST104_footprints:C_SMD_0402_wave, symbol Device:C
- removed R9: 280k, VST104_footprints:R_SMD_0402_wave, symbol Device:R
- removed SW2: SW_DPDT_x2, symbol Switch:SW_DPDT_x2
- removed U16: TPS25940-Q1, symbol VST104:TPS25940-Q1
- removed U18: TPS22965-Q1, symbol VST104:TPS22965-Q1
- added C2, C43: 100n, VST104_footprints:C_SMD_0402, symbol Device:C
- added C48, C49, C50, C57: 100u, VST104_footprints:C_SMD_0402, symbol Device:C
- added EF2: TPS25940-Q1, VST104_footprints:WQFN-20_4.0x3.0mm_EPV, symbol VST104:TPS25940-Q1
- added LG1: 74LVC1G11-Q100, VST104_footprints:SOT-363_TSSOP-6_2.0x1.25mm, symbol VST104:74LVC1G11-Q100
- added NT1: Ground, symbol Device:Net-Tie_2
- added Q2: TPS22965-Q1, VST104_footprints:WSON-8_2.0x2.0mm_EPV, symbol VST104:TPS22965-Q1
- added R1: 1k, VST104_footprints:R_SMD_0402, symbol Device:R
- added R28, R44: 100k, VST104_footprints:R_SMD_0402, symbol Device:R
- added R33, R36: 4, VST104_footprints:R_SMD_0402, symbol Device:R_Small
- added R34, R35: 1, VST104_footprints:R_SMD_0402, symbol Device:R_Small
- added R37: R, VST104_footprints:R_SMD_0402, symbol Device:R
- added R? (x4): 22, symbol Device:R_Small
- added SW2: nrst_sw, VST104_footprints:tactileSW_EVPBB_2.6x1.6mm, symbol Switch:SW_Push_Dual
- AS1: renamed from U1; footprint (none) -> VST104_footprints:mini_QFN-16-1.8x2.6mm
- AS14: renamed from U19; footprint (none) -> VST104_footprints:mini_QFN-16-1.8x2.6mm
- AS15: renamed from U20; footprint (none) -> VST104_footprints:mini_QFN-16-1.8x2.6mm
- AS16: renamed from U21; footprint (none) -> VST104_footprints:mini_QFN-16-1.8x2.6mm
- AS17: renamed from U23; footprint (none) -> VST104_footprints:mini_QFN-16-1.8x2.6mm
- AS18: renamed from U24; footprint (none) -> VST104_footprints:mini_QFN-16-1.8x2.6mm
- AS19: renamed from U25; footprint (none) -> VST104_footprints:mini_QFN-16-1.8x2.6mm
- AS2: renamed from U2; footprint (none) -> VST104_footprints:mini_QFN-16-1.8x2.6mm
- AS20: renamed from U28; footprint (none) -> VST104_footprints:mini_QFN-16-1.8x2.6mm
- C1, C34, C67: footprint VST104_footprints:C_SMD_0402_wave -> VST104_footprints:C_SMD_0402
- C10: renamed from C9; footprint VST104_footprints:C_SMD_0402_wave -> VST104_footprints:C_SMD_0402
- C11: renamed from C10; footprint VST104_footprints:C_SMD_0402_wave -> VST104_footprints:C_SMD_0402
- C12: renamed from C11; footprint VST104_footprints:C_SMD_0402_wave -> VST104_footprints:C_SMD_0402
- C13: renamed from C12; footprint VST104_footprints:C_SMD_0402_wave -> VST104_footprints:C_SMD_0402
- C14: renamed from C13; footprint VST104_footprints:C_SMD_0402_wave -> VST104_footprints:C_SMD_0402
- C15: renamed from C14; footprint VST104_footprints:C_SMD_0402_wave -> VST104_footprints:C_SMD_0402
- C16: renamed from C15; footprint VST104_footprints:C_SMD_0402_wave -> VST104_footprints:C_SMD_0402
- C17: renamed from C16; footprint VST104_footprints:C_SMD_0402_wave -> VST104_footprints:C_SMD_0402
- C18: renamed from C17; footprint VST104_footprints:C_SMD_0402_wave -> VST104_footprints:C_SMD_0402
- C19: renamed from C18; footprint VST104_footprints:C_SMD_0402_wave -> VST104_footprints:C_SMD_0402
- C20: renamed from C19; footprint VST104_footprints:C_SMD_0402_wave -> VST104_footprints:C_SMD_0402
- C21: renamed from C20; footprint VST104_footprints:C_SMD_0402_wave -> VST104_footprints:C_SMD_0402
- C22: renamed from C21; footprint VST104_footprints:C_SMD_0402_wave -> VST104_footprints:C_SMD_0402
- C23: renamed from C22; footprint VST104_footprints:C_SMD_0402_wave -> VST104_footprints:C_SMD_0402
- C24: renamed from C23; footprint VST104_footprints:C_SMD_0402_wave -> VST104_footprints:C_SMD_0402
- C25: renamed from C24; footprint VST104_footprints:C_SMD_0402_wave -> VST104_footprints:C_SMD_0402
- C26: renamed from C25; footprint VST104_footprints:C_SMD_0402_wave -> VST104_footprints:C_SMD_0402
- C27: renamed from C26; footprint VST104_footprints:C_SMD_0402_wave -> VST104_footprints:C_SMD_0402
- C28: renamed from C27; footprint VST104_footprints:C_SMD_0402_wave -> VST104_footprints:C_SMD_0402
- C29: renamed from C28; footprint VST104_footprints:C_SMD_0402_wave -> VST104_footprints:C_SMD_0402
- C3: renamed from C2; footprint VST104_footprints:C_SMD_0402_wave -> VST104_footprints:C_SMD_0402
- C30: renamed from C29; footprint VST104_footprints:C_SMD_0402_wave -> VST104_footprints:C_SMD_0402
- C31: renamed from C30; footprint VST104_footprints:C_SMD_0402_wave -> VST104_footprints:C_SMD_0402
- C32: renamed from C31; footprint VST104_footprints:C_SMD_0402_wave -> VST104_footprints:C_SMD_0402
- C33: renamed from C32; footprint VST104_footprints:C_SMD_0402_wave -> VST104_footprints:C_SMD_0402
- C35: value 100n -> C; footprint VST104_footprints:C_SMD_0402_wave -> VST104_footprints:C_SMD_0402
- C36: renamed from C41; footprint VST104_footprints:C_SMD_0402_wave -> VST104_footprints:C_SMD_0402
- C37: renamed from C42; footprint VST104_footprints:C_SMD_0402_wave -> VST104_footprints:C_SMD_0402
- C38: renamed from C40; footprint VST104_footprints:C_SMD_0402_wave -> VST104_footprints:C_SMD_0402
- C39: renamed from C37; footprint VST104_footprints:C_SMD_0402_wave -> VST104_footprints:C_SMD_0402
- C4: renamed from C3; footprint VST104_footprints:C_SMD_0402_wave -> VST104_footprints:C_SMD_0402
- C40: renamed from C38; footprint VST104_footprints:C_SMD_0402_wave -> VST104_footprints:C_SMD_0402
- C41: renamed from C39; footprint VST104_footprints:C_SMD_0402_wave -> VST104_footprints:C_SMD_0402
- C42: renamed from C43; footprint VST104_footprints:C_SMD_0402_wave -> VST104_footprints:C_SMD_0402
- C44: renamed from C47; footprint VST104_footprints:C_SMD_0402_wave -> VST104_footprints:C_SMD_0402
- C45: renamed from C48; footprint VST104_footprints:C_SMD_0402_wave -> VST104_footprints:C_SMD_0402
- C46: renamed from C49; footprint VST104_footprints:C_SMD_0402_wave -> VST104_footprints:C_SMD_0402
- C47: renamed from C45; footprint VST104_footprints:C_SMD_0402_wave -> VST104_footprints:C_SMD_0402
- C5: renamed from C4; footprint VST104_footprints:C_SMD_0402_wave -> VST104_footprints:C_SMD_0402
- C51: renamed from C50; footprint VST104_footprints:C_SMD_0402_wave -> VST104_footprints:C_SMD_0402
- C52: renamed from C51; footprint VST104_footprints:C_SMD_0402_wave -> VST104_footprints:C_SMD_0402
- C53: renamed from C52; footprint VST104_footprints:C_SMD_0402_wave -> VST104_footprints:C_SMD_0402
- C54: renamed from C53; footprint VST104_footprints:C_SMD_0402_wave -> VST104_footprints:C_SMD_0402
- C55: renamed from C54; footprint VST104_footprints:C_SMD_0402_wave -> VST104_footprints:C_SMD_0402
- C56: renamed from C55; footprint VST104_footprints:C_SMD_0402_wave -> VST104_footprints:C_SMD_0402
- C58: renamed from C60; footprint VST104_footprints:C_SMD_0402_wave -> VST104_footprints:C_SMD_0402
- C59: renamed from C61; footprint VST104_footprints:C_SMD_0402_wave -> VST104_footprints:C_SMD_0402
- C6: renamed from C5; footprint VST104_footprints:C_SMD_0402_wave -> VST104_footprints:C_SMD_0402
- C60: renamed from C56; footprint VST104_footprints:C_SMD_0402_wave -> VST104_footprints:C_SMD_0402
- C61: renamed from C57; footprint VST104_footprints:C_SMD_0402_wave -> VST104_footprints:C_SMD_0402
- C62: renamed from C58; footprint VST104_footprints:C_SMD_0402_wave -> VST104_footprints:C_SMD_0402
- C63: renamed from C59; footprint VST104_footprints:C_SMD_0402_wave -> VST104_footprints:C_SMD_0402
- C64: renamed from C65; footprint VST104_footprints:C_SMD_0402_wave -> VST104_footprints:C_SMD_0402
- C65: renamed from C66; footprint VST104_footprints:C_SMD_0402_wave -> VST104_footprints:C_SMD_0402
- C66: renamed from C62; footprint VST104_footprints:C_SMD_0402_wave -> VST104_footprints:C_SMD_0402
- C68: renamed from C63; footprint VST104_footprints:C_SMD_0402_wave -> VST104_footprints:C_SMD_0402
- C69: renamed from C68; footprint VST104_footprints:C_SMD_0402_wave -> VST104_footprints:C_SMD_0402
- C7: renamed from C6; footprint VST104_footprints:C_SMD_0402_wave -> VST104_footprints:C_SMD_0402
- C70: renamed from C64; footprint VST104_footprints:C_SMD_0402_wave -> VST104_footprints:C_SMD_0402
- C71: renamed from C69; footprint VST104_footprints:C_SMD_0402_wave -> VST104_footprints:C_SMD_0402
- C72: renamed from C70; footprint VST104_footprints:C_SMD_0402_wave -> VST104_footprints:C_SMD_0402
- C73: renamed from C71; footprint VST104_footprints:C_SMD_0402_wave -> VST104_footprints:C_SMD_0402
- C74: renamed from C72; footprint VST104_footprints:C_SMD_0402_wave -> VST104_footprints:C_SMD_0402
- C75: renamed from C73; footprint VST104_footprints:C_SMD_0402_wave -> VST104_footprints:C_SMD_0402
- C76: renamed from C74; footprint VST104_footprints:C_SMD_0402_wave -> VST104_footprints:C_SMD_0402
- C8: renamed from C7; footprint VST104_footprints:C_SMD_0402_wave -> VST104_footprints:C_SMD_0402
- C9: renamed from C8; footprint VST104_footprints:C_SMD_0402_wave -> VST104_footprints:C_SMD_0402
- EF1: renamed from U15; footprint (none) -> VST104_footprints:WQFN-20_4.0x3.0mm_EPV
- FB1: value ??? -> 120 @ 100M; footprint (none) -> VST104_footprints:R_SMD_0402
- H1, H2: footprint (none) -> VST104_footprints:ESQ-129-39-x-D
- JC1: renamed from J1; value Conn_01x08 -> SW&UART; footprint (none) -> VST104_footprints:MOLEX_501461-0891
- L1: footprint (none) -> VST104_footprints:L_SMD_1212_3.0x3.0x1.1mm_muRata
- M1, M2, M3: footprint (none) -> VST104_footprints:SOIC-8_208_5.23x5.23mm
- M4, M5, M6: footprint (none) -> VST104_footprints:BGA-24_FAC024_6.0x8.0mm
- MH1, MH2, MH3, MH4: footprint (none) -> VST104_footprints:MountingHole_3.2mm_M3_Pad_Via
- Q1: renamed from U17; footprint (none) -> VST104_footprints:WSON-8_2.0x2.0mm_EPV
- Q3: renamed from U22; footprint (none) -> VST104_footprints:WSON-8_2.0x2.0mm_EPV
- R10, R11, R12, R13, R14, R15, R16, R17, R18, R19, R20, R21, R22, R23, R24, R25, R26, R27, R31: footprint VST104_footprints:R_SMD_0402_wave -> VST104_footprints:R_SMD_0402
- R2: renamed from R1; footprint VST104_footprints:R_SMD_0402_wave -> VST104_footprints:R_SMD_0402
- R29: value R -> 100k; footprint VST104_footprints:R_SMD_0402_wave -> VST104_footprints:R_SMD_0402
- R3: renamed from R2; footprint VST104_footprints:R_SMD_0402_wave -> VST104_footprints:R_SMD_0402
- R30: renamed from R28; footprint VST104_footprints:R_SMD_0402_wave -> VST104_footprints:R_SMD_0402
- R32: renamed from R30; footprint VST104_footprints:R_SMD_0402_wave -> VST104_footprints:R_SMD_0402
- R38: renamed from R32; footprint VST104_footprints:R_SMD_0402_wave -> VST104_footprints:R_SMD_0402
- R39: renamed from R33; footprint VST104_footprints:R_SMD_0402_wave -> VST104_footprints:R_SMD_0402
- R4: renamed from R3; footprint VST104_footprints:R_SMD_0402_wave -> VST104_footprints:R_SMD_0402
- R40: renamed from R34; footprint VST104_footprints:R_SMD_0402_wave -> VST104_footprints:R_SMD_0402
- R41: renamed from R35; footprint VST104_footprints:R_SMD_0402_wave -> VST104_footprints:R_SMD_0402
- R42: renamed from R36; footprint VST104_footprints:R_SMD_0402_wave -> VST104_footprints:R_SMD_0402
- R43: renamed from R37; footprint VST104_footprints:R_SMD_0402_wave -> VST104_footprints:R_SMD_0402
- R45: renamed from R38; footprint VST104_footprints:R_SMD_0402_wave -> VST104_footprints:R_SMD_0402
- R46: renamed from R39; footprint VST104_footprints:R_SMD_0402_wave -> VST104_footprints:R_SMD_0402
- R47: renamed from R40; footprint VST104_footprints:R_SMD_0402_wave -> VST104_footprints:R_SMD_0402
- R48: renamed from R41; footprint VST104_footprints:R_SMD_0402_wave -> VST104_footprints:R_SMD_0402
- R49: renamed from R42; footprint VST104_footprints:R_SMD_0402_wave -> VST104_footprints:R_SMD_0402
- R5: renamed from R4; footprint VST104_footprints:R_SMD_0402_wave -> VST104_footprints:R_SMD_0402
- R50: renamed from R43; footprint VST104_footprints:R_SMD_0402_wave -> VST104_footprints:R_SMD_0402
- R51: renamed from R52; footprint VST104_footprints:R_SMD_0402_wave -> VST104_footprints:R_SMD_0402
- R52: renamed from R44; footprint VST104_footprints:R_SMD_0402_wave -> VST104_footprints:R_SMD_0402
- R53: renamed from R45; footprint VST104_footprints:R_SMD_0402_wave -> VST104_footprints:R_SMD_0402
- R54: renamed from R46; footprint VST104_footprints:R_SMD_0402_wave -> VST104_footprints:R_SMD_0402
- R55: renamed from R48; footprint VST104_footprints:R_SMD_0402_wave -> VST104_footprints:R_SMD_0402
- R56: renamed from R47; footprint VST104_footprints:R_SMD_0402_wave -> VST104_footprints:R_SMD_0402
- R57: renamed from R49; footprint VST104_footprints:R_SMD_0402_wave -> VST104_footprints:R_SMD_0402
- R58: renamed from R50; footprint VST104_footprints:R_SMD_0402_wave -> VST104_footprints:R_SMD_0402
- R59: renamed from R51; footprint VST104_footprints:R_SMD_0402_wave -> VST104_footprints:R_SMD_0402
- R6: renamed from R5; footprint VST104_footprints:R_SMD_0402_wave -> VST104_footprints:R_SMD_0402
- R7: renamed from R6; footprint VST104_footprints:R_SMD_0402_wave -> VST104_footprints:R_SMD_0402
- R8: renamed from R7; footprint VST104_footprints:R_SMD_0402_wave -> VST104_footprints:R_SMD_0402
- R9: renamed from R8; footprint VST104_footprints:R_SMD_0402_wave -> VST104_footprints:R_SMD_0402
- SW1: value SW_Push_Dual -> nrst_sw; footprint (none) -> VST104_footprints:tactileSW_EVPBB_2.6x1.6mm
- TS1, TS2, TS3, TS4, TS5, TS6, TS7, TS8: footprint (none) -> VST104_footprints:DFN-8_3.0x2.0mm_EP
- Y1: footprint (none) -> VST104_footprints:LSE_3.2x1.5mm
- Y2: footprint (none) -> VST104_footprints:HSE_2.0x1.6mm
- renumbered U11 to AS10, U12 to AS11, U13 to AS12, U14 to AS13, U4 to AS3, U5 to AS4, U6 to AS5, U7 to AS6, U8 to AS7, U9 to AS8, U10 to AS9, U3 to MCU1, U26 to U1, U27 to U2
Connections:
- net labels added: ADC1-3_IN1, ADC1-3_IN2, ADC1-3_IN3, ADC1-3_IN4, BOOT, COMP1_INP, COMP2_INP, DAC1_OUT1, DAC1_OUT2, GNDPWR, I2C3_SCL, I2C3_SDA, OPAMP1, OPAMP1_VINP, OPAMP1_VOUT, OPAMP2, OPAMP2_VINP, OPAMP2_VOUT, QSPI_BK1_IO0, QSPI_BK1_IO1, QSPI_BK1_IO2, QSPI_BK1_IO3, QSPI_BK1_RST, QSPI_BK_~CS~_A, QSPI_~CS~_A, QSPI_~CS~_B, QSPI_~CS~_C, RCC_MCO, SPI1_SCK, SPI1_~CS~_A, SPI1_~CS~_B, SPI1_~CS~_C, SPI1_~HOLD, SPI1_~WP, SPI2_SCK, SPI3_CLK, SPI3_CS1, SPI3_EN, SPI3_MISO, SPI3_MOSI, SPI3_SCK, SPI_1_SCK, SPI_2_SCK, SYS_WKUP2, SYS_WKUP3, SYS_WKUP4, SYS_WKUP5, TIM1_CH1, TIM2_CH2, TIM3_CH3, TIM4_CH4, VREF+
- net labels removed: BOOT0, QSPI_B1_0, QSPI_B1_1, QSPI_B1_2, QSPI_B1_3, QSPI_B1_A, QSPI_B1_B, QSPI_B1_C, QSPI_B1_RST, QSPI_B2_A, QSPI_B2_B, QSPI_B2_C, SPI1_CLK, SPI1_CS1, SPI1_EN, SPI_1_CLK, SPI_2_CLK, SPI_A, SPI_B, SPI_C, SPI_CLK, SPI_HOLD, SPI_SI, SPI_SO, SPI_WP, SUP_3v3
- wire segments 1194 -> 1282
Other:
- note added: "Abbreviations:\nKS - kill switch\nRBF - remove before flight"
- note added: "SW & UART"
- note added: "Triple redundant FLASH memory"
- note removed: "Bank 1 : triple redundant FLASH memory"
- note removed: "LCL - latching current limiter\nFCL - foldback current limiter\nKS - kill switch\nRBF - remove before flight"
- note removed: "USART & SW"
- moved on the sheet: AS11, AS18, AS19, AS3, C1, C10, C11, C12, C13, C14, C15, C16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

Commit message: end of the day
Parts:
- removed C48, C50, C57: 100u, VST104_footprints:C_SMD_0402, symbol Device:C
- removed MCU1: STM32L496QGIx, VST104_footprints:UFBGA-132_7.0x7.0mm, symbol MCU_ST_STM32L4:STM32L496QGIx
- removed R31, R37: R, VST104_footprints:R_SMD_0402, symbol Device:R
- removed R51: 470, VST104_footprints:R_SMD_0402, symbol Device:R
- removed R? (x4): 22, symbol Device:R_Small
- added C44, C45, C56: 1n, VST104_footprints:C_SMD_0402, symbol Device:C
- added C46, C47, C57: 100u, VST104_footprints:C_SMD_0402, symbol Device:C_Small
- added D1, D2, D3, D4, D6, D7, D8: CDBQR40, VST104_footprints:D_SMD_0402, symbol Device:D_Schottky
- added D5: BZT52C3V3TQ-7-F, VST104_footprints:D_SMD_SOD523_1.2x0.8mm, symbol Device:D_Zener
- added ESD1: SP3012-06, VST104_footprints:µDFN-14_3.5x1.35mm, symbol VST104:SP3012-06
- added FB2: 120 @ 100M, VST104_footprints:R_SMD_0402, symbol Device:Ferrite_Bead_Small
- added R34, R38, R43, R44, R56: R, VST104_footprints:R_SMD_0402, symbol Device:R
- added R45, R54: 43, VST104_footprints:R_SMD_0402, symbol Device:R
- added R46, R55, R68, R70: 30, VST104_footprints:R_SMD_0402, symbol Device:R
- added R62, R63, R64, R65, R66, R67: 22, VST104_footprints:R_SMD_0402, symbol Device:R_Small
- added R73: 470, VST104_footprints:R_SMD_0402, symbol Device:R_Small
- added R78, R79, R80, R81, R84, R85, R86, R87: 4k7, VST104_footprints:R_SMD_0402, symbol Device:R_Small
- added U3: STM32L496ZGTx, Package_QFP:LQFP-144_20x20mm_P0.5mm, symbol MCU_ST_STM32L4:STM32L496ZGTx
- M4, M5, M6: footprint VST104_footprints:BGA-24_FAC024_6.0x8.0mm -> VST104_footprints:WSON-8_6.0x8.0mm_EP
- NT1: footprint (none) -> VST104_footprints:R_SMD_0402
- renumbered C33 to C30, C30 to C31, C31 to C32, C32 to C33, C44 to C48, C45 to C49, C46 to C50, C47 to C51, C49 to C52, C51 to C53, C52 to C54, C53 to C55, C54 to C58, C55 to C59, C56 to C60, C58 to C61, C59 to C62, C60 to C63, C61 to C64, C62 to C65, C63 to C66, C64 to C67, C65 to C68, C66 to C69, C67 to C70, C68 to C71, C69 to C72, C70 to C73, C71 to C74, C72 to C75, C73 to C76, C74 to C77, C75 to C78, C76 to C79, R10 to R12, R7 to R13, R8 to R14, R9 to R15, R11 to R16, R12 to R17, R13 to R18, R14 to R19, R15 to R20, R16 to R21, R17 to R22, R22 to R23, R23 to R24, R24 to R25, R25 to R26, R26 to R27, R27 to R28, R18 to R29, R19 to R30, R20 to R31, R21 to R32, R30 to R33, R28 to R35, R29 to R36, R32 to R37, R33 to R39, R34 to R40, R35 to R41, R36 to R42, R44 to R47, R38 to R48, R39 to R49, R40 to R50, R41 to R51, R42 to R52, R43 to R53, R48 to R57, R45 to R58, R46 to R59, R47 to R60, R49 to R61, R50 to R69, R52 to R71, R53 to R72, R54 to R74, R55 to R75, R56 to R76, R57 to R77, R5 to R8, R58 to R82, R59 to R83, R6 to R9
Connections:
- net +3.3VADC: now also U3.25 (NRST)
- net +3V3: now also M4.8 (VCC), M5.8 (VCC), M6.8 (VCC), Q2.7 (OUT), Q2.8 (OUT), Q3.1 (IN), Q3.2 (IN), D7.1 (K), D8.1 (K), R55.1, R56.1, R68.2, R78.1, R79.1, R80.1, R81.1, R84.2, R85.2, R86.2, R87.2
- net +5V: now also Q1.7 (OUT), Q1.8 (OUT), D5.1 (K), R54.1
- net BOOT: now also U3.138 (PH3)
- net EFSE_3_VOUT: now also R38.2
- net GLO_KS_1: now also LG1.3 (B); no longer LG1.6 (C)
- net GND: now also C34.2, C35.2, JC1.6 (Pin_6), M4.4 (VSS), M5.4 (VSS), M6.4 (VSS), C44.2, C45.2, C46.2, C47.2, C56.2, C57.2, ESD1.10 (GND), R34.1, R38.1; no longer C34.1, C35.1, JC1.8 (Pin_8)
- net I2C1_SCL: now also R79.2, R85.1
- net I2C1_SDA: now also R78.2, R84.1
- net I2C2_SCL: now also R81.2, R87.1
- net I2C2_SDA: now also R80.2, R86.1
- net NRST: now also R62.2; no longer JC1.2 (Pin_2)
- net OSC32_IN: now also U3.8 (PC14)
- net OSC32_OUT: now also U3.9 (PC15)
- net OSC_EN: now also U3.24 (PH1)
- net OSC_IN: now also U3.23 (PH0)
- net SW_CLK: now also R63.2, U3.109 (PA14); no longer JC1.5 (Pin_5)
- net SW_DIO: now also R64.2, U3.105 (PA13); no longer JC1.6 (Pin_6)
- net SW_O: now also R65.2, U3.133 (PB3); no longer JC1.7 (Pin_7)
- net UART5_RX: now also R67.2; no longer JC1.3 (Pin_3)
- net UART5_TX: now also R66.2; no longer JC1.4 (Pin_4)
- net at JC1.1 (Pin_1): now also ESD1.5 (VCC), R73.2
- net at C61.1, C62.1, C67.1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: now also Q3.7 (OUT), Q3.8 (OUT), R70.1
- net EF1_out: now reaches C42.2, EF1.4 (OUT), EF1.5 (OUT), EF1.6 (OUT), EF1.7 (OUT), EF1.8 (OUT), R39.1
- net EF1_out: now also Q1.1 (IN), Q1.2 (IN), D3.1 (K), R43.1, R45.2
- net EF2_out: now reaches C43.2, EF2.4 (OUT), EF2.5 (OUT), EF2.6 (OUT), EF2.7 (OUT), EF2.8 (OUT), LG1.5 (VCC), R41.1
- net EF2_out: now also Q2.1 (IN), Q2.2 (IN), D4.1 (K), R44.1, R46.2
- net EF1_en: now reaches EF1.2 (PGOOD), LG1.1 (A)
- net EF1_en: now also R43.2
- net EF2_en: now reaches EF2.2 (PGOOD)
- net EF2_en: now also LG1.6 (C), R44.2; no longer LG1.3 (B)
- net at EF2.18 (dVdT): now also C35.1; no longer C35.2
- net at EF2.17 (ILIM): now also R34.2
- net at Q2.4 (BIAS): now also C45.1, D2.1 (K)
- net at Q2.6 (CT): now also C47.1
- net at Q3.4 (BIAS): now also C56.1, D6.1 (K)
- net at Q3.6 (CT): now also C57.1
- net at EF1.18 (dVdT): now also C34.1; no longer C34.2
- net at Q1.4 (BIAS): now also C44.1, D1.1 (K)
- net at Q1.6 (CT): now also C46.1
- new net: ESD1.1 (A), ESD1.14 (A), JC1.2 (Pin_2), R62.1
- new net: ESD1.13 (B), ESD1.2 (B), JC1.3 (Pin_3), R63.1
- new net: ESD1.12 (C), ESD1.3 (C), JC1.4 (Pin_4), R64.1
- new net: ESD1.11 (D), ESD1.4 (D), JC1.5 (Pin_5), R65.1
- new net: ESD1.6 (E), ESD1.9 (E), JC1.7 (Pin_7), R66.1
- new net: ESD1.7 (F), ESD1.8 (F), JC1.8 (Pin_8), R67.1
- new net: D4.2 (A), R55.2
- new net: D3.2 (A), R54.2
- new net: D1.2 (A), R45.1
- new net: D2.2 (A), R46.1
- new net: D6.2 (A), R68.1
- new net: D7.2 (A), R70.2
- new net: D5.2 (A), R56.2
- new net: D8.2 (A), FB2.2
- new net: FB2.1, R73.1
Other:
- note added: "I2C 1&2 pull-up resistors"
- note added: "SW & UART peripheral with ESD protection"
- note removed: "Abbreviations:\nKS - kill switch\nRBF - remove before flight"
- note removed: "Mounting holes pads"
- note removed: "SW & UART"
- moved on the sheet: AS20, C25, C26, C30, C36, C37, C38, C42, C43, C51, C52, C53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

Commit message: kill me pls
Parts:
- added R66, R67, R68, R69: 4k7, VST104_footprints:R_SMD_0402, symbol Device:R_Small
- renumbered C63 to C61, C64 to C62, C65 to C63, C66 to C64, C61 to C65, C62 to C66, C69 to C67, C70 to C68, C67 to C69, C68 to C70, C79 to C77, C77 to C78, C78 to C79, R15 to R10, R16 to R11, R17 to R12, R18 to R13, R19 to R14, R20 to R15, R21 to R16, R22 to R17, R23 to R18, R24 to R19, R25 to R20, R26 to R21, R27 to R22, R28 to R23, R29 to R24, R30 to R25, R31 to R26, R32 to R27, R33 to R28, R34 to R29, R35 to R30, R36 to R31, R37 to R32, R38 to R33, R39 to R34, R40 to R35, R41 to R36, R42 to R37, R43 to R38, R44 to R39, R45 to R40, R46 to R41, R47 to R42, R48 to R43, R49 to R44, R50 to R45, R51 to R46, R52 to R47, R53 to R48, R54 to R49, R8 to R5, R55 to R50, R56 to R51, R57 to R52, R58 to R53, R59 to R54, R60 to R55, R61 to R56, R62 to R57, R63 to R58, R64 to R59, R9 to R6, R65 to R60, R66 to R61, R67 to R62, R68 to R63, R69 to R64, R70 to R65, R12 to R7, R71 to R70, R72 to R71, R73 to R72, R74 to R73, R75 to R74, R76 to R75, R77 to R76, R78 to R77, R79 to R78, R80 to R79, R13 to R8, R81 to R80, R82 to R81, R83 to R82, R84 to R83, R85 to R84, R86 to R85, R87 to R86, R14 to R9, U3 to U1, U1 to U2, U2 to U3
Connections:
- net CAN1_RX: now also R66.2; no longer U2.4 (RXD)
- net CAN1_TX: now also R67.2; no longer U2.1 (TXD)
- net CAN2_RX: now also R68.2; no longer U3.4 (RXD)
- net CAN2_TX: now also R69.2; no longer U3.1 (TXD)
- net GND: now also U1.107 (VSS), U1.120 (VSS), U1.130 (VSS), U1.143 (VSS), U1.16 (VSS), U1.38 (VSS), U1.51 (VSS), U1.61 (VSS), U1.71 (VSS), U1.83 (VSS), U1.94 (VSS)
- net GNDA: now also U1.30 (VSSA)
- net H12_EN: now also U1.19 (PF7)
- net H1_1: now also AS12.3 (NO3); no longer AS12.11 (NO1)
- net H1_1-4_EN: now also U1.64 (PE11)
- net H1_10: now also AS17.7 (NO4); no longer AS17.15 (NO2)
- net H1_10_IO: now also U1.21 (PF9)
- net H1_1_IO: now also U1.65 (PE12)
- net H1_2: now also AS12.15 (NO2); no longer AS12.3 (NO3)
- net H1_2_IO: now also U1.67 (PE14)
- net H1_3: now also AS12.11 (NO1); no longer AS12.15 (NO2)
- net H1_3_IO: now also U1.66 (PE13)
- net H1_45: now also AS6.15 (NO2); no longer AS6.11 (NO1)
- net H1_46: now also AS6.11 (NO1); no longer AS6.3 (NO3)
- net H1_47: now also AS6.7 (NO4); no longer AS6.15 (NO2)
- net H1_48: now also AS6.3 (NO3); no longer AS6.7 (NO4)
- net H1_49: now also AS7.15 (NO2); no longer AS7.11 (NO1)
- net H1_4_IO: now also U1.68 (PE15)
- net H1_5: now also AS13.3 (NO3); no longer AS13.11 (NO1)
- net H1_5-8_EN: now also U1.142 (PE1)
- net H1_50: now also AS7.11 (NO1); no longer AS7.3 (NO3)
- net H1_51: now also AS7.7 (NO4); no longer AS7.15 (NO2)
- net H1_52: now also AS7.3 (NO3); no longer AS7.7 (NO4)
- net H1_5_IO: now also U1.1 (PE2)
- net H1_6: now also AS13.15 (NO2); no longer AS13.3 (NO3)
- net H1_6_IO: now also U1.3 (PE4)
- net H1_7: now also AS13.11 (NO1); no longer AS13.15 (NO2)
- net H1_7_IO: now also U1.2 (PE3)
- net H1_8_IO: now also U1.4 (PE5)
- net H2_1: now also AS18.15 (NO2); no longer AS18.11 (NO1)
- net H2_1-4_EN: now also U1.5 (PE6)
- net H2_10: now also AS17.3 (NO3); no longer AS17.7 (NO4)
- net H2_10_IO: now also U1.49 (PF11)
- net H2_1_IO: now also U1.58 (PE7)
- net H2_2_IO: now also U1.60 (PE9)
- net H2_3: now also AS18.11 (NO1); no longer AS18.15 (NO2)
- net H2_3_IO: now also U1.59 (PE8)
- net H2_4_IO: now also U1.63 (PE10)
- net H2_5: now also AS19.15 (NO2); no longer AS19.11 (NO1)
- net H2_5-8_EN: now also U1.50 (PF12)
- net H2_5_IO: now also U1.53 (PF13)
- net H2_6_IO: now also U1.55 (PF15)
- net H2_7: now also AS19.11 (NO1); no longer AS19.15 (NO2)
- net H2_7_IO: now also U1.54 (PF14)
- net H2_8_IO: now also U1.141 (PE0)
- net OSC32_IN: no longer U1.8 (PC14)
- net OSC32_OUT: no longer U1.9 (PC15)
- net SPI1_CS2: now also U1.20 (PF8)
- net SPI2_CLK: now also U1.10 (PF0)
- net SPI2_CS1: now also U1.11 (PF1)
- net SPI2_CS2: now also U1.22 (PF10)
- net SPI2_EN: now also U1.128 (PG13)
- net SPI2_MISO: now also U1.132 (PG15)
- net SPI2_MOSI: now also U1.129 (PG14)
- net SPI3_CLK: now also U1.15 (PF5)
- net SPI3_CS1: now also U1.18 (PF6)
- net SPI3_EN: now also U1.12 (PF2)
- net SPI3_MISO: now also U1.14 (PF4)
- net SPI3_MOSI: now also U1.13 (PF3)
- net SPI_1_CS1: now also AS15.3 (NO3); no longer AS15.7 (NO4)
- net SPI_1_MISO: no longer AS15.15 (NO2)
- net SPI_1_MOSI: now also AS15.15 (NO2); no longer AS15.11 (NO1)
- net SPI_1_SCK: now also AS15.7 (NO4); no longer AS15.3 (NO3)
- net SPI_2_CS2: now also AS17.15 (NO2); no longer AS17.3 (NO3)
- net UART3_CTS: now also U1.126 (PG11)
- net UART3_EN: now also U1.93 (PG8)
- net UART3_RST: now also U1.127 (PG12)
- net UART3_RX: now also U1.125 (PG10)
- net UART3_TX: now also U1.124 (PG9)
- net UART_1_CTS: now also AS3.11 (NO1); no longer AS3.3 (NO3)
- net UART_1_RTS: now also AS3.15 (NO2); no longer AS3.7 (NO4)
- net UART_1_RX: now also AS3.3 (NO3); no longer AS3.15 (NO2)
- net UART_1_TX: now also AS3.7 (NO4); no longer AS3.11 (NO1)
- new net: R69.1, U3.1 (TXD)
- new net: R68.1, U3.4 (RXD)
- new net: R67.1, U2.1 (TXD)
- new net: R66.1, U2.4 (RXD)
