File: board_sierra/board_sierra.sch (KiCad schematic (older format))
At the start: 232 parts, among them M1 CY15B102Q, M2 CY15B102Q, M3 CY15B102Q, M4 S25FL256L, M5 S25FL256L, M6 S25FL256L, Q1 TPS22965-Q1, Q2 TPS22965-Q1, Q3 TPS22965-Q1, SW1 nrst_sw, SW2 nrst_sw, U1 STM32L496ZGTx, U2 TCAN1051-Q1, U3 TCAN1051-Q1, Y1 ABS07AIG, Y2 SiT8924

Commit message: rising hope
Parts:
- added C80, C81, C82, C83, C84, C85, C86, C87: 10n, VST104_footprints:C_SMD_0402, symbol Device:C
- added R87, R88: 200k, VST104_footprints:R_SMD_0402, symbol Device:R
Connections:
- net H1_51_IO is gone; now on net H1_48_IO: AS7.16 (COM2)
- net H1_52_IO is gone; now on net H1_50_IO: AS7.8 (COM4)
- net SUP_3V3_REF is gone; now on net GND: H1.34 (Pin_34)
- net CAN_1_H: now also H1.23 (Pin_23); no longer H1.27 (Pin_27)
- net CAN_1_L: now also H1.24 (Pin_24); no longer H1.28 (Pin_28)
- net CAN_2_H: now also H2.23 (Pin_23); no longer H2.28 (Pin_28)
- net CAN_2_L: now also H2.24 (Pin_24); no longer H2.27 (Pin_27)
- net CPU_SELECT: now also H1.29 (Pin_29); no longer H2.34 (Pin_34)
- net CPU_WD_1: now also H1.27 (Pin_27), R87.2; no longer H1.35 (Pin_35)
- net GLO_FAULT: now also H1.26 (Pin_26); no longer H2.36 (Pin_36)
- net GLO_KS_1: now also H1.35 (Pin_35); no longer H1.37 (Pin_37)
- net GLO_SYNC: now also H1.25 (Pin_25); no longer H2.35 (Pin_35)
- net GND: now also H1.33 (Pin_33), H2.29 (Pin_29), H2.30 (Pin_30), H2.32 (Pin_32); no longer H1.19 (Pin_19), H1.20 (Pin_20), H2.19 (Pin_19), H2.20 (Pin_20)
- net GNDA: now also H2.31 (Pin_31); no longer H1.33 (Pin_33)
- net H12_EN: no longer U1.19 (PF7)
- net H1_1: now also AS12.11 (NO1); no longer AS12.3 (NO3)
- net H1_1-4_EN: no longer U1.64 (PE11)
- net H1_10_IO: no longer U1.21 (PF9)
- net H1_1_IO: no longer U1.65 (PE12)
- net H1_2: now also AS12.7 (NO4); no longer AS12.15 (NO2)
- net H1_2_IO: no longer U1.67 (PE14)
- net H1_3: now also AS12.15 (NO2); no longer AS12.11 (NO1)
- net H1_3_IO: no longer U1.66 (PE13)
- net H1_4: now also AS12.3 (NO3); no longer AS12.7 (NO4)
- net H1_41: now also AS5.3 (NO3); no longer AS5.11 (NO1)
- net H1_41_IO: now also AS5.4 (COM3); no longer AS5.12 (COM1)
- net H1_42: now also AS5.7 (NO4); no longer AS5.3 (NO3)
- net H1_42_IO: now also AS5.8 (COM4); no longer AS5.4 (COM3)
- net H1_43: now also AS6.11 (NO1); no longer AS5.15 (NO2)
- net H1_43_IO: now also AS6.12 (COM1); no longer AS5.16 (COM2)
- net H1_44: now also AS6.15 (NO2); no longer AS5.7 (NO4)
- net H1_44_IO: now also AS6.16 (COM2); no longer AS5.8 (COM4)
- net H1_45: now also AS6.3 (NO3); no longer AS6.15 (NO2)
- net H1_45_IO: now also AS6.4 (COM3); no longer AS6.12 (COM1)
- net H1_46: now also AS6.7 (NO4); no longer AS6.11 (NO1)
- net H1_46_IO: now also AS6.8 (COM4); no longer AS6.4 (COM3)
- net H1_47: now also AS7.11 (NO1); no longer AS6.7 (NO4)
- net H1_47_IO: now also AS7.12 (COM1); no longer AS6.16 (COM2)
- net H1_48: now also AS7.15 (NO2); no longer AS6.3 (NO3)
- net H1_48_IO: no longer AS6.8 (COM4)
- net H1_49: now also AS7.3 (NO3); no longer AS7.15 (NO2)
- net H1_49_IO: now also AS7.4 (COM3); no longer AS7.12 (COM1)
- net H1_4_IO: no longer U1.68 (PE15)
- net H1_5: now also AS13.11 (NO1); no longer AS13.3 (NO3)
- net H1_5-8_EN: no longer U1.142 (PE1)
- net H1_50: now also AS7.7 (NO4); no longer AS7.11 (NO1)
- net H1_50_IO: no longer AS7.4 (COM3)
- net H1_51: now also AS17.11 (NO1); no longer AS7.7 (NO4)
- net H1_52: now also AS17.15 (NO2); no longer AS7.3 (NO3)
- net H1_5_IO: no longer U1.1 (PE2)
- net H1_6: now also AS13.7 (NO4); no longer AS13.15 (NO2)
- net H1_6_IO: no longer U1.3 (PE4)
- net H1_7_IO: no longer U1.2 (PE3)
- net H1_8: now also AS13.3 (NO3); no longer AS13.7 (NO4)
- net H1_8_IO: no longer U1.4 (PE5)
- net H2_1: now also AS18.7 (NO4); no longer AS18.15 (NO2)
- net H2_1-4_EN: no longer U1.5 (PE6)
- net H2_10_IO: no longer U1.49 (PF11)
- net H2_1_IO: no longer U1.58 (PE7)
- net H2_2: now also AS18.11 (NO1); no longer AS18.3 (NO3)
- net H2_2_IO: no longer U1.60 (PE9)
- net H2_3: now also AS18.3 (NO3); no longer AS18.11 (NO1)
- net H2_3_IO: no longer U1.59 (PE8)
- net H2_4: now also AS18.15 (NO2); no longer AS18.7 (NO4)
- net H2_43: no longer H2.43 (Pin_43)
- net H2_44: no longer H2.44 (Pin_44)
- net H2_45: no longer H2.45 (Pin_45)
- net H2_46: no longer H2.46 (Pin_46)
- net H2_4_IO: no longer U1.63 (PE10)
- net H2_5: now also AS19.7 (NO4); no longer AS19.15 (NO2)
- net H2_5-8_EN: no longer U1.50 (PF12)
- net H2_51: now also AS17.3 (NO3)
- net H2_52: now also AS17.7 (NO4)
- net H2_5_IO: no longer U1.53 (PF13)
- net H2_6: now also AS19.11 (NO1); no longer AS19.3 (NO3)
- net H2_6_IO: no longer U1.55 (PF15)
- net H2_7_IO: no longer U1.54 (PF14)
- net H2_8: now also AS19.15 (NO2); no longer AS19.7 (NO4)
- net H2_8_IO: no longer U1.141 (PE0)
- net I2C_1_SCL: now also H1.21 (Pin_21); no longer H1.25 (Pin_25)
- net I2C_1_SDA: now also H1.22 (Pin_22); no longer H1.26 (Pin_26)
- net I2C_2_SCL: now also H2.21 (Pin_21); no longer H2.25 (Pin_25)
- net I2C_2_SDA: now also H2.22 (Pin_22); no longer H2.26 (Pin_26)
- net SPI1_CS2: no longer U1.20 (PF8)
- net SPI2_CLK: no longer U1.10 (PF0)
- net SPI2_CS1: no longer U1.11 (PF1)
- net SPI2_CS2: no longer U1.22 (PF10)
- net SPI2_EN: no longer U1.128 (PG13)
- net SPI2_MISO: no longer U1.132 (PG15)
- net SPI2_MOSI: no longer U1.129 (PG14)
- net SPI3_CLK: no longer U1.15 (PF5)
- net SPI3_CS1: no longer U1.18 (PF6)
- net SPI3_EN: no longer U1.12 (PF2)
- net SPI3_MISO: no longer U1.14 (PF4)
- net SPI3_MOSI: no longer U1.13 (PF3)
- net SPI_1_CS1: now also H1.9 (Pin_9); no longer H1.11 (Pin_11)
- net SPI_1_CS2: now also AS13.15 (NO2), H1.7 (Pin_7); no longer AS17.11 (NO1), H1.9 (Pin_9)
- net SPI_1_MISO: now also AS15.11 (NO1), H1.12 (Pin_12); no longer H1.14 (Pin_14)
- net SPI_1_MOSI: now also H1.10 (Pin_10); no longer H1.12 (Pin_12)
- net SPI_1_SCK: now also H1.11 (Pin_11); no longer H1.13 (Pin_13)
- net SPI_2_CS1: now also H2.9 (Pin_9); no longer H2.11 (Pin_11)
- net SPI_2_CS2: now also AS19.3 (NO3), H2.7 (Pin_7); no longer AS17.15 (NO2), H2.9 (Pin_9)
- net SPI_2_MISO: now also H2.12 (Pin_12); no longer H2.14 (Pin_14)
- net SPI_2_MOSI: now also H2.10 (Pin_10); no longer H2.12 (Pin_12)
- net SPI_2_SCK: now also H2.11 (Pin_11); no longer H2.13 (Pin_13)
- net SUP_3V3: now also H2.27 (Pin_27), H2.28 (Pin_28); no longer H1.29 (Pin_29), H1.31 (Pin_31)
- net SUP_5V: now also H2.25 (Pin_25), H2.26 (Pin_26); no longer H1.30 (Pin_30), H1.32 (Pin_32)
- net SUP_BAT_1: now also H2.45 (Pin_45); no longer H2.30 (Pin_30)
- net SUP_BAT_2: now also H2.46 (Pin_46); no longer H2.32 (Pin_32)
- net UART3_CTS: no longer U1.126 (PG11)
- net UART3_EN: no longer U1.93 (PG8)
- net UART3_RST: no longer U1.127 (PG12)
- net UART3_RX: no longer U1.125 (PG10)
- net UART3_TX: no longer U1.124 (PG9)
- net UART5_RX: now also U1.116 (PD2)
- net UART5_TX: now also U1.98 (PC8)
- net UART_1_CTS: now also H1.14 (Pin_14); no longer H1.16 (Pin_16)
- net UART_1_RTS: now also H1.16 (Pin_16); no longer H1.18 (Pin_18)
- net UART_1_RX: now also H1.15 (Pin_15); no longer H1.17 (Pin_17)
- net UART_1_TX: now also H1.13 (Pin_13); no longer H1.15 (Pin_15)
- net UART_2_CTS: now also H2.14 (Pin_14); no longer H2.16 (Pin_16)
- net UART_2_RTS: now also H2.16 (Pin_16); no longer H2.18 (Pin_18)
- net UART_2_RX: now also H2.15 (Pin_15); no longer H2.17 (Pin_17)
- net UART_2_TX: now also H2.13 (Pin_13); no longer H2.15 (Pin_15)
- net UART_RCS_1_CTS: now also H1.18 (Pin_18); no longer H1.22 (Pin_22)
- net UART_RCS_1_RTS: now also H1.20 (Pin_20); no longer H1.24 (Pin_24)
- net UART_RCS_1_RX: now also H1.19 (Pin_19); no longer H1.23 (Pin_23)
- net UART_RCS_1_TX: now also H1.17 (Pin_17); no longer H1.21 (Pin_21)
- net UART_RCS_2_CTS: now also H2.18 (Pin_18); no longer H2.22 (Pin_22)
- net UART_RCS_2_RTS: now also H2.20 (Pin_20); no longer H2.24 (Pin_24)
- net UART_RCS_2_RX: now also H2.19 (Pin_19); no longer H2.23 (Pin_23)
- net UART_RCS_2_TX: now also H2.17 (Pin_17); no longer H2.21 (Pin_21)
- net at H2.37 (Pin_37): now also C82.1
- net at H2.38 (Pin_38): now also C86.2
- net H2_39: now reaches H2.39 (Pin_39)
- net H2_40: now reaches H2.40 (Pin_40)
- net at H1.36 (Pin_36): now also R88.1
- net H1_39: now reaches H1.39 (Pin_39)
- net H1_39: now also AS5.11 (NO1)
- net H1_40: now reaches H1.40 (Pin_40)
- net H1_40: now also AS5.15 (NO2)
- removed net H1_10: AS17.7 (NO4), H1.10 (Pin_10)
- net H1_41-44_EN renamed H1_39-42_EN
- net H1_45-48_EN renamed H1_43-46_EN
- net H1_49-52_EN renamed H1_47-50_EN
- removed net H1_7: AS13.11 (NO1), H1.7 (Pin_7)
- removed net H2_10: AS17.3 (NO3), H2.10 (Pin_10)
- removed net H2_7: AS19.11 (NO1), H2.7 (Pin_7)
- net SUP_5V_REF: no longer names the net of H2.33 (Pin_33)
- net SUP_5V_REF: now also C80.1
- new net: C84.2, H2.34 (Pin_34)
- new net: C81.1, H2.35 (Pin_35)
- new net: C85.2, H2.36 (Pin_36)
- new net: C83.1, H2.43 (Pin_43)
- new net: C87.2, H2.44 (Pin_44)
- new net: H1.28 (Pin_28), R87.1
- new net CPU_MODE: H1.30 (Pin_30)
- new net GLO_KS_2: R88.2
- new net H1_39_IO: AS5.12 (COM1)
- new net H1_40_IO: AS5.16 (COM2)
- no-connect marks 106 -> 100
