File: board_sierra/board_sierra.sch (KiCad schematic (older format))
At the start: 242 parts, among them M1 CY15B102Q, M2 CY15B102Q, M3 CY15B102Q, M4 S25FL256L, M5 S25FL256L, M6 S25FL256L, Q1 TPS22965-Q1, Q2 TPS22965-Q1, Q3 TPS22965-Q1, SW1 nrst_sw, SW2 nrst_sw, U1 STM32L496ZGTx, U2 TCAN1051-Q1, U3 TCAN1051-Q1, Y1 ABS07AIG, Y2 SiT8924

Commit message: brain teaser SOLVED
Parts:
- removed AS10, AS11, AS5, AS6, AS7, AS8: DGQ2788A, VST104_footprints:mini_QFN-16-1.8x2.6mm, symbol VST104:DGQ2788A
- removed C27, C28, C29, C31, C33, C39, C80, C81, C82, C83, C84, C85, C86, C87: 10n, VST104_footprints:C_SMD_0402, symbol Device:C
- removed R10, R11, R13, R24, R25, R8, R82, R87, R88, R9: 200k, VST104_footprints:R_SMD_0402, symbol Device:R
- removed R83, R84, R85, R86: 4k7, VST104_footprints:R_SMD_0402, symbol Device:R_Small
- added AS15: DGQ2788A, VST104_footprints:mini_QFN-16-1.8x2.6mm, symbol VST104:DGQ2788A
- added C74: 10n, VST104_footprints:C_SMD_0402, symbol Device:C
- added R22, R41, R5, R52, R6, R80: 200k, VST104_footprints:R_SMD_0402, symbol Device:R
- renumbered AS17 to AS10, AS16 to AS11, AS15 to AS12, AS18 to AS13, AS19 to AS14, AS9 to AS5, AS20 to AS6, AS12 to AS7, AS13 to AS8, AS14 to AS9, C30 to C27, C32 to C28, C34 to C29, C35 to C30, C36 to C31, C37 to C32, C38 to C33, C77 to C34, C40 to C35, C41 to C36, C42 to C37, C43 to C38, C44 to C39, C45 to C40, C46 to C41, C47 to C42, C48 to C43, C58 to C44, C50 to C45, C51 to C46, C52 to C47, C53 to C48, C54 to C49, C55 to C50, C56 to C51, C57 to C52, C49 to C53, C59 to C54, C60 to C55, C61 to C56, C62 to C57, C63 to C58, C64 to C59, C65 to C60, C66 to C61, C67 to C62, C68 to C63, C69 to C64, C70 to C65, C71 to C66, C72 to C67, C73 to C68, C74 to C69, C75 to C70, C76 to C71, C78 to C72, C79 to C73, R12 to R10, R14 to R11, R15 to R12, R16 to R13, R17 to R14, R18 to R15, R19 to R16, R20 to R17, R21 to R18, R22 to R19, R23 to R20, R81 to R21, R26 to R23, R27 to R24, R28 to R25, R29 to R26, R30 to R27, R31 to R28, R32 to R29, R33 to R30, R34 to R31, R35 to R32, R36 to R33, R37 to R34, R38 to R35, R39 to R36, R40 to R37, R41 to R38, R42 to R39, R43 to R40, R53 to R42, R45 to R43, R46 to R44, R47 to R45, R48 to R46, R49 to R47, R50 to R48, R51 to R49, R52 to R50, R44 to R51, R54 to R53, R55 to R54, R56 to R55, R57 to R56, R58 to R57, R59 to R58, R60 to R59, R61 to R60, R62 to R61, R63 to R62, R64 to R63, R65 to R64, R66 to R65, R67 to R66, R68 to R67, R69 to R68, R70 to R69, R5 to R7, R71 to R70, R72 to R71, R73 to R72, R74 to R73, R75 to R74, R76 to R75, R77 to R76, R78 to R77, R79 to R78, R80 to R79, R6 to R8, R7 to R9
Connections:
- net labels added: CAN1_H, CAN1_L, CAN2_H, CAN2_L, CPU_EN, GLO_EN, MODE, SPI1_CS1, SPI1_EN, SPI2_SCK, SUP_3V3_REF, SUP_5V_REF, UART_1_RST, UART_2_RST, UART_RCS_1_RST, UART_RCS_2_RST, USER1_1, USER1_2, USER1_4, USER1_EN, USER2_1, USER2_2, USER2_4, USER2_EN, USER3_1, USER3_2, USER3_3, USER3_4, USER3_EN, USER4_1, USER4_2, USER4_3, USER4_4, USER4_EN, USER5_1, USER5_2, USER5_3, USER5_4, USER5_EN, USER6_1, USER6_2, USER6_3, USER6_4, USER6_EN, USER_1_1, USER_1_2, USER_1_4, USER_2_1, USER_2_2, USER_2_4, USER_3_1, USER_3_2, USER_3_3, USER_3_4, USER_4_1, USER_4_2, USER_4_3, USER_4_4, USER_5_1, USER_5_2, USER_5_3, USER_5_4, USER_6_1, USER_6_2, USER_6_3, USER_6_4, USER_SPI1_EN, USER_SPI2_EN, WATCHDOG
- net labels removed: CPU_SELECT, GLO_EN_OU, GLO_KS_2, H12_EN, H1_1, H1_1-4_EN, H1_10_IO, H1_1_IO, H1_2, H1_2_IO, H1_3, H1_39, H1_39-42_EN, H1_39_IO, H1_3_IO, H1_4, H1_40, H1_40_IO, H1_41, H1_41_IO, H1_42, H1_42_IO, H1_43, H1_43-46_EN, H1_43_IO, H1_44, H1_44_IO, H1_45, H1_45_IO, H1_46, H1_46_IO, H1_47, H1_47-50_EN, H1_47_IO, H1_48, H1_48_IO, H1_49, H1_49_IO, H1_4_IO, H1_5, H1_5-8_EN, H1_50, H1_50_IO, H1_51, H1_52, H1_5_IO, H1_6, H1_6_IO, H1_7_IO, H1_8, H1_8_IO, H2_1, H2_1-4_EN, H2_10_IO, H2_1_IO, H2_2, H2_2_IO, H2_3, H2_39, H2_3_IO, H2_4, H2_40, H2_41, H2_41-44_EN, H2_41_IO, H2_42, H2_42_IO, H2_43, H2_43_IO, H2_44, H2_44_IO, H2_45, H2_45-48_EN, H2_45_IO, H2_46, H2_46_IO, H2_47, H2_47_IO, H2_48, H2_48_IO, H2_49, H2_49-52_EN, H2_49_IO, H2_4_IO, H2_5, H2_5-8_EN, H2_50, H2_50_IO, H2_51, H2_51_IO, H2_52, H2_52_IO, H2_5_IO, H2_6, H2_6_IO, H2_7_IO, H2_8, H2_8_IO, SELECT, SPI2_CLK, SPI3_CLK, SPI3_CS1, SPI3_EN, SPI3_MISO, SPI3_MOSI, SUP_BAT_1, SUP_BAT_2, UART4_CTS, UART4_RST, UART_1_RTS, UART_2_RTS, UART_RCS_1_RTS, UART_RCS_2_RTS
- wire segments 1294 -> 1106
- no-connect marks 100 -> 105
Other:
- note added: "CAN FD transceiver\n"
- note added: "I2C 1&2 pull-up"
- note removed: "CAN FD transceiver and isolator"
- note removed: "I2C 1&2 pull-up resistors"
- note removed: "User IO bottom H1 isolators"
- moved on the sheet: AS10, AS12, AS6

Commit message: weekend
Changed lines of the file:
@@
 Connection ~ 4650 12750
-$Comp
-L Device:R R5
-U 1 1 7B488437
-P 4650 12950
-F 0 "R5" H 4600 13100 50  0000 R CNN
-F 1 "200k" V 4750 13050 50  0000 R CNN
-F 2 "VST104_footprints:R_SMD_0402" V 4580 12950 50  0001 C CNN
-F 3 "~" H 4650 12950 50  0001 C CNN
-	1    4650 12950
-	1    0    0    -1
-$EndComp
 $Comp
 L power:GND #PWR017
@@
 Text Label 4400 14750 2    50   ~ 0
 CPU_EN
-Text GLabel 3050 12450 2    50   Input ~ 0
+Text GLabel 3050 12650 2    50   Input ~ 0
 USER_3_4
 Text GLabel 3050 12350 2    50   Input ~ 0
-USER_3_2
-Text GLabel 3050 12550 2    50   Input ~ 0
 USER_3_3
-Text GLabel 3050 12650 2    50   Input ~ 0
-USER_3_1
-Text GLabel 3050 14450 2    50   Input ~ 0
-USER_4_4
 Text GLabel 3050 14350 2    50   Input ~ 0
 USER_4_2
 Text GLabel 3050 14550 2    50   Input ~ 0
-USER_4_3
-Text GLabel 3050 14650 2    50   Input ~ 0
 USER_4_1
 Wire Wire Line
@@
 Text Label 1450 14600 2    50   ~ 0
 USER4_4
-Text GLabel 9050 12450 2    50   Input ~ 0
+Text GLabel 9050 12350 2    50   Input ~ 0
 USER_5_4
-Text GLabel 9050 12350 2    50   Input ~ 0
+Text GLabel 9050 12650 2    50   Input ~ 0
 USER_5_2
 Text GLabel 9050 12550 2    50   Input ~ 0
 USER_5_3
-Text GLabel 9050 12650 2    50   Input ~ 0
+Text GLabel 9050 12450 2    50   Input ~ 0
 USER_5_1
 Text Label 7450 12100 2    50   ~ 0
@@
 	-1   0    0    1
 $EndComp
-Text GLabel 9050 14550 2    50   Input ~ 0
+Text GLabel 9050 14750 2    50   Input ~ 0
 USER_6_4
-Text GLabel 9050 14450 2    50   Input ~ 0
+Text GLabel 9050 14650 2    50   Input ~ 0
 USER_6_2
-Text GLabel 9050 14650 2    50   Input ~ 0
-USER_6_3
-Text GLabel 9050 14750 2    50   Input ~ 0
-USER_6_1
 Text Label 7450 14200 2    50   ~ 0
 USER6_EN
@@
 Text Label 5000 4650 0    50   ~ 0
 CPU_EN
+$Comp
+L Device:R R5
+U 1 1 7B488437
+P 4650 12950
+F 0 "R5" H 4600 13100 50  0000 R CNN
+F 1 "200k" V 4750 13050 50  0000 R CNN
+F 2 "VST104_footprints:R_SMD_0402" V 4580 12950 50  0001 C CNN
+F 3 "~" H 4650 12950 50  0001 C CNN
+	1    4650 12950
+	1    0    0    -1
+$EndComp
+Text Label 5000 5850 0    50   ~ 0
+USER6_EN
+Text Label 5000 5750 0    50   ~ 0
+USER6_1
+Text Label 5000 5650 0    50   ~ 0
+USER6_2
+Text Label 5000 5450 0    50   ~ 0
+USER6_3
+Text Label 5000 4550 0    50   ~ 0
+USER6_4
+Text GLabel 9050 14550 2    50   Input ~ 0
+USER_6_1
+Text GLabel 9050 14450 2    50   Input ~ 0
+USER_6_3
+Text GLabel 3050 14450 2    50   Input ~ 0
+USER_4_4
+Text GLabel 3050 14650 2    50   Input ~ 0
+USER_4_3
 Wire Bus Line
 	11800 7350 11800 8350
@@
 Wire Bus Line
 	14100 7350 15300 7350
+Text GLabel 3050 12450 2    50   Input ~ 0
+USER_3_1
+Text GLabel 3050 12550 2    50   Input ~ 0
+USER_3_2
 $EndSCHEMATC

Commit message: a bit of wiring
Parts:
- removed C2, C3: 100n, VST104_footprints:C_SMD_0402, symbol Device:C
- removed C22: 1u, VST104_footprints:C_SMD_0402, symbol Device:C
- removed R1: 1k, VST104_footprints:R_SMD_0402, symbol Device:R
- removed R4: 10k, VST104_footprints:R_SMD_0402, symbol Device:R
- removed SW1, SW2: nrst_sw, VST104_footprints:tactileSW_EVPBB_2.6x1.6mm, symbol Switch:SW_Push_Dual
- added C16, C7: 100n, VST104_footprints:C_SMD_0402, symbol Device:C
- added R10, R11, R5, R6, R7: 10k, VST104_footprints:R_SMD_0402, symbol Device:R_Small
- C17: value 100n -> 1u
- C18, C20: value 1u -> 100n
- C19: value 100n -> 4u7
- C21: value 10n -> 4u7
- renumbered AS9 to AS1, AS7 to AS10, AS13 to AS11, AS10 to AS12, AS11 to AS13, AS8 to AS14, AS14 to AS15, AS6 to AS2, AS1 to AS3, AS2 to AS4, AS15 to AS6, AS4 to AS7, AS12 to AS8, AS3 to AS9, C11 to C10, C12 to C11, C13 to C12, C14 to C13, C15 to C14, C16 to C15, C43 to C2, C7 to C24, C8 to C25, C28 to C26, C74 to C27, C51 to C28, C24 to C29, C34 to C3, C53 to C30, C23 to C31, C52 to C32, C35 to C33, C54 to C34, C60 to C35, C61 to C36, C64 to C37, C65 to C38, C31 to C39, C32 to C40, C70 to C41, C33 to C42, C71 to C43, C48 to C44, C49 to C45, C50 to C46, C44 to C47, C45 to C48, C72 to C49, C73 to C50, C25 to C51, C26 to C52, C36 to C53, C55 to C54, C29 to C55, C30 to C56, C27 to C57, C37 to C58, C38 to C59, C56 to C60, C57 to C61, C39 to C62, C40 to C63, C58 to C64, C59 to C65, C62 to C66, C63 to C67, C41 to C68, C42 to C69, C66 to C70, C67 to C71, C46 to C72, C47 to C73, C68 to C74, C69 to C75, C9 to C8, C10 to C9, D6 to D1, D7 to D2, D8 to D3, D1 to D4, D2 to D5, D3 to D6, D4 to D7, D5 to D8, Q3 to Q1, Q1 to Q2, Q2 to Q3, R40 to R1, R10 to R12, R80 to R13, R6 to R14, R51 to R15, R5 to R16, R8 to R17, R52 to R18, R7 to R19, R22 to R2, R50 to R20, R55 to R21, R62 to R22, R63 to R23, R64 to R24, R23 to R25, R53 to R26, R12 to R27, R13 to R28, R14 to R29, R41 to R3, R44 to R30, R45 to R31, R46 to R32, R42 to R33, R43 to R34, R27 to R35, R28 to R36, R76 to R37, R77 to R38, R78 to R39, R21 to R4, R79 to R40, R56 to R41, R57 to R42, R58 to R43, R59 to R44, R60 to R45, R61 to R46, R9 to R47, R24 to R48, R54 to R49, R15 to R50, R16 to R51, R17 to R52, R18 to R53, R19 to R54, R20 to R55, R11 to R56, R71 to R57, R25 to R58, R26 to R59, R29 to R60, R30 to R61, R31 to R62, R32 to R63, R33 to R64, R34 to R65, R35 to R66, R36 to R67, R65 to R68, R66 to R69, R67 to R70, R68 to R71, R69 to R72, R70 to R73, R37 to R74, R38 to R75, R39 to R76, R47 to R77, R48 to R78, R72 to R79, R2 to R8, R73 to R80, R74 to R81, R75 to R82, R49 to R83, R3 to R9
Connections:
- net labels added: CLK, HD, Q0, Q1, Q2, Q3, QSPI_~CS~_1, QSPI_~CS~_2, QSPI_~CS~_3, SI, SO, SPI1_~CS~_1, SPI1_~CS~_2, SPI1_~CS~_3, SPI3_CS1, SPI3_CS2, SPI3_EN, SPI3_MISO, SPI3_MOSI, SPI3_SCK, UART4_CTS, UART4_RST, VDDA, WP
- net labels removed: 0, 1, 2, 3, GNDPWR, OPAMP1, OPAMP2, QSPI_BK1_RST, QSPI_~CS~_A, QSPI_~CS~_B, QSPI_~CS~_C, RS, SC, SPI1_CS1, SPI1_CS2, SPI1_EN, SPI1_~CS~_A, SPI1_~CS~_B, SPI1_~CS~_C, VREF+
- wire segments 1106 -> 1174
Other:
- note added: "CAN & I2C isolators"
- note added: "GLOBAL & CPU isolators"
- note added: "I2C 1 & 2 pull-up"
- note added: "RCS UART isolators"
- note added: "USER 1 & 2 isolators"
- note added: "USER 3 & 4 isolators"
- note added: "USER 5 & 6 isolators"
- note removed: "Global signals isolator"
- note removed: "I2C 1&2 pull-up"
- note removed: "I2C isolator"
- note removed: "Radio subs. UART isolators"
- note removed: "User IO H1&H2 isolators"
- note removed: "User IO bottom H2 isolators"
- note removed: "User IO top H1 isolators"
- note removed: "User IO top H2 isolators"
- moved on the sheet: AS1, AS10, AS11, AS12, AS13, AS14, AS15, AS2, AS3, AS4, AS5, AS6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

Commit message: almost there
Parts:
- removed C37: 100n, VST104_footprints:C_SMD_0402, symbol Device:C
- removed TS3: MCP9804, VST104_footprints:DFN-8_3.0x2.0mm_EP, symbol VST104:MCP9804
- added R8, R9: 10k, VST104_footprints:R_SMD_0402, symbol Device:R_Small
- renumbered C24 to C22, C25 to C23, C26 to C24, C27 to C25, C28 to C26, C29 to C27, C30 to C28, C31 to C29, C32 to C30, C33 to C31, C34 to C32, C35 to C33, C36 to C34, C38 to C35, C39 to C36, C40 to C37, C41 to C38, C42 to C39, C43 to C40, C44 to C41, C45 to C42, C46 to C43, C47 to C44, C48 to C45, C49 to C46, C50 to C47, C51 to C48, C52 to C49, C53 to C50, C54 to C51, C55 to C52, C56 to C53, C57 to C54, C58 to C55, C59 to C56, C60 to C57, C61 to C58, C62 to C59, C63 to C60, C64 to C61, C65 to C62, C66 to C63, C67 to C64, C68 to C65, C69 to C66, C70 to C67, C71 to C68, C72 to C69, C73 to C70, C74 to C71, C75 to C72, R8 to R10, R9 to R11, R10 to R12, R11 to R13, R12 to R14, R13 to R15, R14 to R16, R15 to R17, R16 to R18, R17 to R19, R18 to R20, R19 to R21, R20 to R22, R21 to R23, R22 to R24, R23 to R25, R24 to R26, R25 to R27, R26 to R28, R27 to R29, R28 to R30, R29 to R31, R30 to R32, R31 to R33, R32 to R34, R33 to R35, R34 to R36, R35 to R37, R36 to R38, R37 to R39, R38 to R40, R39 to R41, R40 to R42, R41 to R43, R42 to R44, R43 to R45, R44 to R46, R45 to R47, R46 to R48, R47 to R49, R48 to R50, R49 to R51, R50 to R52, R51 to R53, R52 to R54, R53 to R55, R54 to R56, R55 to R57, R56 to R58, R57 to R59, R58 to R60, R59 to R61, R60 to R62, R61 to R63, R62 to R64, R63 to R65, R64 to R66, R65 to R67, R66 to R68, R67 to R69, R68 to R70, R69 to R71, R70 to R72, R71 to R73, R72 to R74, R73 to R75, R74 to R76, R75 to R77, R76 to R78, R77 to R79, R78 to R80, R79 to R81, R80 to R82, R81 to R83, R82 to R84, R83 to R85, TS4 to TS3, TS5 to TS4, TS6 to TS5, TS7 to TS6, TS8 to TS7
Connections:
- net labels added: EF1_CUR, EF2_CUR, I2C3_EN, I2C3_SCL, I2C3_SDA
- net labels removed: EFSE_3_VOUT, EFSE_5_VOUT, I2C1_EN
- wire segments 1174 -> 1183
- no-connect marks 105 -> 104
Other:
- note added: "*RESERVED"

Commit message: train jurney update
Connections:
- wire segments 1183 -> 1210
- no-connect marks 104 -> 106
Changed lines of the file:
@@
 Text Label 6050 9550 0    50   ~ 0
 I2C2_EN
+Text Label 1550 8650 2    50   ~ 0
+USER1_4
+Text Label 1550 8450 2    50   ~ 0
+SPI2_CS2
+Text Label 1550 8550 2    50   ~ 0
+USER1_2
+Text Label 1550 5550 2    50   ~ 0
+USER2_4
+Text Label 1550 9550 2    50   ~ 0
+SPI3_CS2
+Text Label 1550 9750 2    50   ~ 0
+USER2_2
+Text Label 1550 9650 2    50   ~ 0
+USER2_1
+Wire Wire Line
+	2800 8650 1550 8650
+Wire Wire Line
+	1550 8550 2800 8550
+Wire Wire Line
+	2800 8450 1550 8450
+Wire Wire Line
+	2800 9750 1550 9750
+Wire Wire Line
+	1550 9650 2800 9650
+Wire Wire Line
+	2800 9550 1550 9550
+Wire Wire Line
+	2800 5550 1550 5550
+Wire Wire Line
+	1550 5450 2800 5450
+Text Label 1550 8250 2    50   ~ 0
+USER3_1
+Text Label 1550 8350 2    50   ~ 0
+USER3_2
+Text Label 6450 5550 0    50   ~ 0
+USER3_3
+Text Label 6450 5650 0    50   ~ 0
+USER3_4
+Wire Wire Line
+	6450 5550 5200 5550
+Wire Wire Line
+	5200 5450 6450 5450
+Wire Wire Line
+	5200 5650 6450 5650
+Wire Wire Line
+	1550 8250 2800 8250
+Text Label 6050 7650 0    50   ~ 0
+USER4_2
+Text Label 1550 7550 2    50   ~ 0
+USER4_3
+Text Label 1550 7650 2    50   ~ 0
+USER4_4
+Wire Wire Line
+	2800 8350 1550 8350
+Wire Wire Line
+	5200 7650 6050 7650
+Wire Wire Line
+	1550 7550 2800 7550
+Wire Wire Line
+	2800 7650 1550 7650
+Wire Wire Line
+	2800 7450 1550 7450
+Text Label 1550 7450 2    50   ~ 0
+USER5_1
+NoConn ~ 2800 7350
+NoConn ~ 5200 8450
+Text Label 1550 9050 2    50   ~ 0
+USER5_2
+Text Label 1550 9150 2    50   ~ 0
+USER5_3
+Text Label 1550 9250 2    50   ~ 0
+USER5_4
+Wire Wire Line
+	2800 9350 1550 9350
+Wire Wire Line
+	1550 9250 2800 9250
+Wire Wire Line
+	2800 9150 1550 9150
+Wire Wire Line
+	2800 9050 1550 9050
+Wire Wire Line
+	2800 9450 1550 9450
+Text Label 1550 9350 2    50   ~ 0
+USER6_1
+Text Label 1550 9450 2    50   ~ 0
+USER6_2
+Text Label 1550 8850 2    50   ~ 0
+USER6_3
+Text Label 1550 8950 2    50   ~ 0
+USER6_4
+Wire Wire Line
+	2800 8950 1550 8950
+Wire Wire Line
+	2800 8850 1550 8850
+Wire Wire Line
+	5200 7950 6450 7950
+Text Label 6450 7950 0    50   ~ 0
+USER1_EN
+Wire Wire Line
+	5200 8050 6450 8050
+Text Label 6450 8050 0    50   ~ 0
+USER_SPI1_EN
+Text Label 6600 4550 0    50   ~ 0
+USER2_EN
+Wire Wire Line
+	6600 4550 5200 4550
+Text Label 1550 5450 2    50   ~ 0
+USER1_1
+Text Label 6450 5450 0    50   ~ 0
+USER4_1
 Wire Bus Line
 	14300 9850 14300 10850

Commit message: review
Parts:
- C1, C10, C11, C12, C13, C14, C15, C16, C17, C18, C19, C2, C20, C21, C22, C23, C24, C25, C26, C27, C28, C29, C3, C31, C32, C33, C34, C35, C38, C4, C40, C44, C45, C46, C47, C48, C49, C5, C50, C51, C52, C53, C54, C55, C56, C57, C58, C59, C6, C60, C61, C62, C63, C64, C67, C68, C69, C7, C70, C71, C72, C8, C9: symbol Device:C -> board_sierra-rescue:C-Device
- C30, C36, C37, C39, C41, C42, C43, C65, C66: symbol Device:C_Small -> board_sierra-rescue:C_Small-Device
- D1, D2, D3, D4, D5, D6, D7: symbol Device:D_Schottky -> board_sierra-rescue:D_Schottky-Device
- D8: symbol Device:D_Zener -> board_sierra-rescue:D_Zener-Device
- FB1, FB2: symbol Device:Ferrite_Bead_Small -> board_sierra-rescue:Ferrite_Bead_Small-Device
- H1, H2: symbol Connector_Generic:Conn_02x26_Odd_Even -> board_sierra-rescue:Conn_02x26_Odd_Even-Connector_Generic
- JC1: symbol Connector_Generic:Conn_01x08 -> board_sierra-rescue:Conn_01x08-Connector_Generic
- L1: symbol Device:L -> board_sierra-rescue:L-Device
- MH1, MH2, MH3, MH4: symbol Mechanical:MountingHole_Pad -> board_sierra-rescue:MountingHole_Pad-Mechanical
- NT1: symbol Device:Net-Tie_2 -> board_sierra-rescue:Net-Tie_2-Device
- R1, R10, R11, R14, R15, R16, R17, R18, R19, R2, R20, R21, R22, R23, R24, R25, R26, R27, R28, R29, R3, R30, R31, R32, R33, R34, R35, R36, R37, R38, R4, R49, R50, R51, R58, R60, R61, R62, R63, R68, R69, R74, R75, R76, R77, R78, R79, R80, R81, R82, R83, R84, R85: symbol Device:R -> board_sierra-rescue:R-Device
- R12, R13, R39, R40, R41, R42, R43, R44, R45, R46, R47, R48, R5, R52, R53, R54, R55, R56, R57, R59, R6, R64, R65, R66, R67, R7, R70, R71, R72, R73, R8, R9: symbol Device:R_Small -> board_sierra-rescue:R_Small-Device
- U1: symbol MCU_ST_STM32L4:STM32L496ZGTx -> board_sierra-rescue:STM32L496ZGTx-MCU_ST_STM32L4
- Y1: symbol Device:Crystal -> board_sierra-rescue:Crystal-Device
Connections:
- wire segments 1210 -> 1215

Commit message: almost done
Parts:
- removed NT1: Ground, VST104_footprints:R_SMD_0402, symbol board_sierra-rescue:Net-Tie_2-Device
- added TP1, TP10, TP11, TP12, TP13, TP14, TP15, TP16, TP17, TP2, TP3, TP4, TP5, TP6, TP7, TP8, TP9: test_point, VST104_footprints:scope_PAD, symbol Connector:TestPoint
- added TP18, TP19: GND, VST104_footprints:scope_GND, symbol Connector:TestPoint
- JC1: footprint VST104_footprints:MOLEX_501461-0891 -> VST104_footprints:CLP-104-02-x-D
- L1: footprint VST104_footprints:L_SMD_1212_3.0x3.0x1.1mm_muRata -> VST104_footprints:L_SMD_0402
- U1: footprint Package_QFP:LQFP-144_20x20mm_P0.5mm -> VST104_footprints:LQFP-144_20x20mm_P0.5mm
- renumbered C38 to C36, C40 to C37, C36 to C38, C37 to C39, C41 to C40, C42 to C41, C43 to C42, C39 to C43, M4 to M1, M5 to M2, M6 to M3, M1 to M4, M2 to M5, M3 to M6, R23 to R22, R22 to R23, R26 to R25, R25 to R26, R32 to R29, R33 to R30, R34 to R31, R29 to R32, R30 to R33, R31 to R34
Connections:
- net CAN1_RX: now also TP14.1
- net CAN1_TX: now also TP15.1
- net CAN2_RX: now also TP16.1
- net CAN2_TX: now also TP17.1
- net CL: now also TP9.1
- net CLK: now also TP4.1
- net GND: now also C1.1, C4.1, U1.30 (VSSA), U1.31 (VREF-), TP18.1, TP19.1
- net HD: now also TP13.1
- net I2C2_SCL: now also TP1.1
- net I2C2_SDA: now also TP2.1
- net Q0: now also TP5.1
- net Q1: now also TP6.1
- net Q2: now also TP7.1
- net Q3: now also TP8.1
- net SI: now also TP10.1
- net SO: now also TP11.1
- net SPI1_~WP: now also TP12.1
- net at C33.1, C34.1, C35.1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: now also TP3.1
- removed net GNDA: C1.1, C4.1, H2.31 (Pin_31), U1.30 (VSSA), U1.31 (VREF-)
- net I2C1_SCL: no longer names the net of U1.129 (PG14)
- net I2C1_SDA: no longer names the net of U1.128 (PG13)
- net SUP_3V3_REF: no longer names the net of H1.31 (Pin_31)
- net SUP_5V_REF: no longer names the net of H1.32 (Pin_32)
- no-connect marks 106 -> 111
Other:
- moved on the sheet: C38, C39, C43, M4, M5, M6, R23, R26, R32, R33, R34, R37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

Commit message: capacitors size fixed
Parts:
- removed TP3: test_point, VST104_footprints:scope_PAD, symbol Connector:TestPoint
- added C26: 10u, VST104_footprints:C_SMD_0805, symbol board_sierra-rescue:C-Device
- added R86, R87: 0, VST104_footprints:R_SMD_1206, symbol board_sierra-rescue:R_Small-Device
- added UA1: Conn_01x03, VST104_footprints:PC104_universal_OBC&FPGA, symbol Connector_Generic:Conn_01x03
- C15: footprint VST104_footprints:C_SMD_0402 -> VST104_footprints:C_SMD_0805
- C17, C19, C21, C4: footprint VST104_footprints:C_SMD_0402 -> VST104_footprints:C_SMD_0603
- C27: renamed from C26; value 1n -> 100n
- C28: renamed from C30; value 100u -> 1n
- C3: value 100n -> 10n
- C49: renamed from C48; value 17p -> 17p 1%
- C50: renamed from C49; value 17p -> 17p 1%
- C51: renamed from C52; value C -> 22n 1%
- C52: renamed from C53; value C -> 15n 1%
- C56: renamed from C55; value 100n -> 10u; footprint VST104_footprints:C_SMD_0402 -> VST104_footprints:C_SMD_0805
- C57: renamed from C56; value 100n -> 10u; footprint VST104_footprints:C_SMD_0402 -> VST104_footprints:C_SMD_0805
- C60: renamed from C59; value 1n -> 100n
- C61: renamed from C60; value 1n -> 100n
- C66: renamed from C65; value 100u -> 1n
- C67: renamed from C66; value 100u -> 1n
- C70: renamed from C69; value 100u -> 1u; footprint VST104_footprints:C_SMD_0402 -> VST104_footprints:C_SMD_0603
- C71: renamed from C70; value 100u -> 1u; footprint VST104_footprints:C_SMD_0402 -> VST104_footprints:C_SMD_0603
- R1, R10, R11, R14, R15, R16, R17, R18, R19, R2, R20, R21, R22, R27, R28, R3, R35, R36, R4, R50, R51: value 200k -> 100k
- R12, R13, R5, R6, R7, R8, R9: value 10k -> 22
- R24, R25: value 30 -> 8.1
- R52, R55: value R -> 210k 1%
- R53: value R -> 16k9 1%
- R54: value R -> 86k6 1%
- R56: value R -> 6k49 1%
- R57: value R -> 48k7 1%
- R59: renamed from R60; value R -> 75k 1%
- R60: renamed from R61; value R -> 75k 1%
- R62: value R -> 33k2 1%
- R63: value R -> 32k2 1%
- R64: value 4 -> 110k 1%
- R65: value 1 -> 60k4 1%
- R66: value 1 -> 110k 1%
- R67: value 4 -> 31k6 1%
- R68, R69: value R -> 10k
- R70, R71, R72, R73: value 4k7 -> 22
- R74, R75: value 200K -> 10k
- R76, R79: value 43 -> 8.1
- R77, R80: value 30 -> 12
- R85: value R -> 330
- renumbered C27 to C29, C28 to C30, C29 to C31, C33 to C32, C34 to C33, C31 to C34, C32 to C35, C35 to C36, C36 to C37, C37 to C38, C38 to C39, C39 to C40, C40 to C41, C41 to C42, C42 to C43, C43 to C44, C46 to C45, C47 to C46, C44 to C47, C45 to C48, C50 to C53, C51 to C54, C54 to C55, C57 to C58, C58 to C59, C61 to C62, C62 to C63, C63 to C64, C64 to C65, C67 to C68, C68 to C69, C71 to C72, C72 to C73, R59 to R61, TP11 to TP10, TP12 to TP11, TP13 to TP12, TP14 to TP13, TP15 to TP14, TP16 to TP15, TP17 to TP16, TP18 to TP17, TP19 to TP18, TP4 to TP3, TP5 to TP4, TP6 to TP5, TP7 to TP6, TP8 to TP7, TP9 to TP8, TP10 to TP9
Connections:
- net +3V3: now also C26.2
- net GND: now also C26.1, UA1.1 (Pin_1)
- net SUP_3V3: now also R86.2
- net SUP_5V: now also R87.2
- new net: R86.1, UA1.2 (Pin_2)
- new net: R87.1, UA1.3 (Pin_3)
Other:
- moved on the sheet: C27, C28, C32, C33, C36, C37, C38, C45, C46, C51, C52, C56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
