File: board_whiskey/board_whiskey.kicad_pcb (KiCad board)
At the start: 4 copper layers, 90.2 x 95.9 mm, 103 parts, among them J1 Conn_01x08, M1 CY15B102Q, M2 CY15B102Q, M3 CY15B102Q, M4 S25FLxL, M5 S25FLxL, M6 S25FLxL, SW2 SW_Push_Dual, U1 TCAN1051, U2 TCAN1051, U3 STM32L496QGIx, U4 ADuM142E, U5 ADuM142E, U6 ADuM142E, U7 ADuM142E, U8 LSF0102-Q1, U9 LSF0102-Q1, Y1 ABS07AIG, Y2 SiT8924

Commit message: night update
Parts:
- removed C1, C11, C12, C13, C14, C15, C17, C18, C2, C24, C25, C26, C27, C28, C29, C3, C30, C31, C32, C33, C34, C35, C36, C37, C38, C39, C4, C41, C42, C43, C45, C8: 100n, Capacitor_SMD:C_0603_1608Metric
- removed C10, C9: 17p, Capacitor_SMD:C_0603_1608Metric
- removed C16, C21: 4n7, Capacitor_SMD:C_0603_1608Metric
- removed C19, C20, C22, C23: 100p, Capacitor_SMD:C_0603_1608Metric
- removed C40, C44, C46, C6: 1u, Capacitor_SMD:C_0603_1608Metric
- removed C5: 10n, Capacitor_SMD:C_0603_1608Metric
- removed C7: 10u, Capacitor_SMD:C_0603_1608Metric
- removed D1, D2: VCAN16A2, Package_TO_SOT_SMD:SOT-323_SC-70
- removed FB1: ???, Inductor_SMD:L_0603_1608Metric
- removed the J1 at (64.8, 54.6)
- removed L1: 10u, Inductor_SMD:L_0603_1608Metric
- removed L2, L3: L, VST104_footprints:CMCH_1210
- removed M1, M2, M3: CY15B102Q, Package_SO:SOIC-8_5.275x5.275mm_P1.27mm
- removed M4, M5, M6: S25FLxL, VST104_footprints:WSON-8-EP-6.0x8.0mm
- removed R1, R13, R14, R15, R16, R17, R18, R5, R6: 10k, Resistor_SMD:R_0603_1608Metric
- removed R10: 470, Resistor_SMD:R_0603_1608Metric
- removed R11, R12, R7, R8: 60, Resistor_SMD:R_0603_1608Metric
- removed R2, R3: 280k, Resistor_SMD:R_0603_1608Metric
- removed R4: 1k, Resistor_SMD:R_0603_1608Metric
- removed the REF** at (115.6, 129.5)
- removed SW2: SW_Push_Dual, VST104_footprints:EVPBB0AAB000
- removed TS1, TS2, TS3, TS4, TS5, TS6, TS7, TS8: MCP9804, Package_DFN_QFN:DFN-8-1EP_3x2mm_P0.5mm_EP1.75x1.45mm
- removed U1, U2: TCAN1051, Package_SON:WSON-8-1EP_3x3mm_P0.5mm_EP1.6x2.0mm
- removed U3: STM32L496QGIx, Package_BGA:UFBGA-132_7x7mm_Layout12x12_P0.5mm
- removed U4, U5, U6, U7: ADuM142E, Package_SO:QSOP-16_3.9x4.9mm_P0.635mm
- removed U8, U9: LSF0102-Q1, Package_SO:VSSOP-8_2.3x2mm_P0.5mm
- removed Y1: ABS07AIG, Crystal:Crystal_SMD_3215-2Pin_3.2x1.5mm
- removed Y2: SiT8924, Crystal:Crystal_SMD_2016-4Pin_2.0x1.6mm
- added REF**: OSHW-Logo2_7.3x6mm_SilkScreen, Symbol:OSHW-Logo2_7.3x6mm_SilkScreen, F.Cu at (96.2, 131.8)
- renumbered MH1 to H1, MH2 to H2, MH3 to H3, MH4 to H4, H1 to J1, H2 to J2
Connections:
- J1 pad 1: (no net) -> /CAN_A_L
- J1 pad 10: (no net) -> Net-(J1-Pad10)
- J1 pad 11: (no net) -> Net-(J1-Pad11)
- J1 pad 12: (no net) -> Net-(J1-Pad12)
- J1 pad 13: (no net) -> Net-(J1-Pad13)
- J1 pad 14: (no net) -> Net-(J1-Pad14)
- J1 pad 15: UART_1_TX -> Net-(J1-Pad15)
- J1 pad 16: UART_1_CTS -> Net-(J1-Pad16)
- J1 pad 17: UART_1_RX -> Net-(J1-Pad17)
- J1 pad 18: UART_1_RTS -> Net-(J1-Pad18)
- J1 pad 19: GND -> Net-(J1-Pad19)
- J1 pad 2: (no net) -> /CAN_A_H
- J1 pad 20: GND -> Net-(J1-Pad20)
- J1 pad 21: UART_RCS_1_TX -> Net-(J1-Pad21)
- J1 pad 22: UART_RCS_1_CTS -> Net-(J1-Pad22)
- J1 pad 23: UART_RCS_1_RX -> Net-(J1-Pad23)
- J1 pad 24: UART_RCS_1_RTS -> Net-(J1-Pad24)
- J1 pad 25: I2C_1_SCL -> Net-(J1-Pad25)
- J1 pad 26: I2C_1_SDA -> Net-(J1-Pad26)
- J1 pad 27: CAN_1_H -> Net-(J1-Pad27)
- J1 pad 28: CAN_1_L -> Net-(J1-Pad28)
- J1 pad 29: SUP_3V3 -> Net-(J1-Pad29)
- J1 pad 3: (no net) -> Net-(J1-Pad3)
- J1 pad 30: SUP_5V -> Net-(J1-Pad30)
- J1 pad 31: SUP_3V3 -> /CHARGE
- J1 pad 32: SUP_5V -> /CHARGE
- J1 pad 33: GNDA -> /GND
- J1 pad 34: (no net) -> /GND
- J1 pad 35: (no net) -> Net-(J1-Pad35)
- J1 pad 36: (no net) -> Net-(J1-Pad36)
- J1 pad 37: (no net) -> Net-(J1-Pad37)
- J1 pad 38: (no net) -> Net-(J1-Pad38)
- J1 pad 39: (no net) -> Net-(J1-Pad39)
- J1 pad 4: (no net) -> Net-(J1-Pad4)
- J1 pad 40: (no net) -> Net-(J1-Pad40)
- J1 pad 41: (no net) -> Net-(J1-Pad41)
- J1 pad 42: (no net) -> Net-(J1-Pad42)
- J1 pad 43: (no net) -> Net-(J1-Pad43)
- J1 pad 44: (no net) -> Net-(J1-Pad44)
- J1 pad 45: (no net) -> Net-(J1-Pad45)
- J1 pad 46: (no net) -> Net-(J1-Pad46)
- J1 pad 47: (no net) -> Net-(J1-Pad47)
- J1 pad 48: (no net) -> Net-(J1-Pad48)
- J1 pad 49: (no net) -> Net-(J1-Pad49)
- J1 pad 5: (no net) -> Net-(J1-Pad5)
- J1 pad 50: (no net) -> Net-(J1-Pad50)
- J1 pad 51: (no net) -> Net-(J1-Pad51)
- J1 pad 52: (no net) -> Net-(J1-Pad52)
- J1 pad 6: (no net) -> Net-(J1-Pad6)
- J1 pad 7: (no net) -> Net-(J1-Pad7)
- J1 pad 8: (no net) -> Net-(J1-Pad8)
- J1 pad 9: (no net) -> Net-(J1-Pad9)
- J2 pad 1: (no net) -> /CAN_B_L
- J2 pad 10: (no net) -> Net-(J2-Pad10)
- J2 pad 11: (no net) -> Net-(J2-Pad11)
- J2 pad 12: (no net) -> Net-(J2-Pad12)
- J2 pad 13: (no net) -> Net-(J2-Pad13)
- J2 pad 14: (no net) -> Net-(J2-Pad14)
- J2 pad 15: UART_2_TX -> Net-(J2-Pad15)
- J2 pad 16: UART_2_CTS -> Net-(J2-Pad16)
- J2 pad 17: UART_2_RX -> Net-(J2-Pad17)
- J2 pad 18: UART_2_RTS -> Net-(J2-Pad18)
- J2 pad 19: GND -> Net-(J2-Pad19)
- J2 pad 2: (no net) -> /CAN_B_H
- J2 pad 20: GND -> Net-(J2-Pad20)
- J2 pad 21: UART_RCS_2_TX -> Net-(J2-Pad21)
- J2 pad 22: UART_RCS_2_CTS -> Net-(J2-Pad22)
- J2 pad 23: UART_RCS_2_RX -> Net-(J2-Pad23)
- J2 pad 24: UART_RCS_2_RTS -> Net-(J2-Pad24)
- J2 pad 25: I2C_2_SCL -> /5V
- J2 pad 26: I2C_2_SDA -> /5V
- J2 pad 27: CAN_2_L -> Net-(J2-Pad27)
- J2 pad 28: CAN_2_H -> Net-(J2-Pad28)
- J2 pad 29: SUP_UNREG -> /GND
- J2 pad 3: (no net) -> Net-(J2-Pad3)
- J2 pad 30: (no net) -> /GND
- J2 pad 31: SUP_UNREG -> /GND
- J2 pad 32: (no net) -> /GND
- J2 pad 33: (no net) -> Net-(J2-Pad33)
- J2 pad 34: (no net) -> Net-(J2-Pad34)
- J2 pad 35: (no net) -> Net-(J2-Pad35)
- J2 pad 36: (no net) -> Net-(J2-Pad36)
- J2 pad 37: (no net) -> Net-(J2-Pad37)
- J2 pad 38: (no net) -> Net-(J2-Pad38)
- J2 pad 39: (no net) -> Net-(J2-Pad39)
- J2 pad 4: (no net) -> Net-(J2-Pad4)
- J2 pad 40: (no net) -> Net-(J2-Pad40)
- J2 pad 41: (no net) -> Net-(J2-Pad41)
- J2 pad 42: (no net) -> Net-(J2-Pad42)
- J2 pad 43: (no net) -> Net-(J2-Pad43)
- J2 pad 44: (no net) -> Net-(J2-Pad44)
- J2 pad 45: (no net) -> /VBAT
- J2 pad 46: (no net) -> /VBAT
- J2 pad 47: (no net) -> Net-(J2-Pad47)
- J2 pad 48: (no net) -> Net-(J2-Pad48)
- J2 pad 49: (no net) -> Net-(J2-Pad49)
- J2 pad 5: (no net) -> Net-(J2-Pad5)
- J2 pad 50: (no net) -> Net-(J2-Pad50)
- J2 pad 51: (no net) -> Net-(J2-Pad51)
- J2 pad 52: (no net) -> Net-(J2-Pad52)
- J2 pad 6: (no net) -> Net-(J2-Pad6)
- J2 pad 7: (no net) -> Net-(J2-Pad7)
- J2 pad 8: (no net) -> Net-(J2-Pad8)
- J2 pad 9: (no net) -> Net-(J2-Pad9)
Routing:
- added copper zone on F.Cu, net (none)
- removed copper zone on F.Cu, net Net-(TS1-Pad3)
