File: element_foxtrot/element_foxtrot/element_foxtrot.kicad_pcb (KiCad board)
At the start: 2 copper layers, 15 parts, among them J1 Conn_02x26_Top_Bottom, J2 Conn_02x26_Top_Bottom, U1 STUSB4500QTR, U3 USBLC6

Commit message: switches and connectors
Parts:
- added J8: Battery, VST104_footprints:PXC_1935187, F.Cu at (246.2, -13.2)
- added SW2: 300DP3J1BLKM6QE, VST104_footprints:300DP3J1BLKM6QE, F.Cu at (218.8, -4.00)
- added SW3: SW_SPST, VST104_footprints:300SP1J1BLKM2QE, F.Cu at (242.6, -1.51)
- added SW4: SW_SPST, VST104_footprints:300SP1J1BLKM2QE, F.Cu at (264.6, -13.6)
- added TP1: TestPoint, VST104_footprints:scope_PAD, F.Cu at (229.5, -22.4)
- added TP10: TestPoint_Alt, VST104_footprints:KSE_PN6095, F.Cu at (241.1, 28.8)
- added TP2: TestPoint, VST104_footprints:scope_PAD, F.Cu at (232.1, -22.4)
- added TP4: TestPoint_Alt, VST104_footprints:KSE_PN6095, F.Cu at (215.0, 28.8)
- added TP7: TestPoint_Alt, VST104_footprints:KSE_PN6095, F.Cu at (215.0, 41.8)
- added TP8: TestPoint_Alt, VST104_footprints:KSE_PN6095, F.Cu at (228.0, 28.8)
- added TP9: TestPoint_Alt, VST104_footprints:KSE_PN6095, F.Cu at (228.0, 41.8)
- added U7: TL432DBZ, Package_TO_SOT_SMD:SOT-23, F.Cu at (240.1, -26.1)
- added U8: USBLC6, Package_TO_SOT_SMD:SOT-23-6, F.Cu at (230.6, -26.0)
- added U9: USBLC6, Package_TO_SOT_SMD:SOT-23-6, F.Cu at (235.4, -26.0)
Connections:
- net /+BATT_1 renamed /SUP_BAT_1
- net /+BATT_2 renamed /SUP_BAT_2
- net /+UNREG renamed /SUP_UNREG
- TP3 pad 1: (no net) -> /VSINK
- U1 pad 11: (no net) -> /ATTACH
- U1 pad 19: (no net) -> /ALTER
- U1 pad 22: (no net) -> VDD
- U1 pad 7: (no net) -> /SCL
- U1 pad 8: (no net) -> /SDA
- U3 pad 5: (no net) -> +5V

Commit message: professor check needed
Parts:
- added U5: OKR-T6-W12, VST104_footprints:OKR-T6-W12, F.Cu at (251.6, -51.6)
- added U6: OKR-T6-W12, VST104_footprints:OKR-T6-W12, F.Cu at (263.8, -51.6)
- moved SW2 105.5 mm to (309.4, -58.0)
- moved SW3 69.0 mm to (311.0, -10.0)
- moved SW4 58.7 mm to (313.4, 19.0)
- moved TP9 33.8 mm to (259.6, 53.8)
- moved TP10 20.4 mm to (261.4, 30.2)
- moved TP7 19.2 mm to (215.6, 61.0)
- moved TP8 17.2 mm to (237.8, 43.0)
