File: element_foxtrot/element_foxtrot/element_foxtrot.sch (KiCad schematic (older format))
At the start: 93 parts

Commit message: switches and connectors
Parts:
- removed D?: ESDA25P35, symbol Device:D_Schottky
- removed D? (x3): LED, symbol Device:LED
- removed Q? (x3): STR2N2VH5, symbol Device:Q_NMOS_DGS
- removed R? (x3): 100k, symbol Device:R
- removed R? (x3): 1k, symbol Device:R_Small
- removed R?: 100k, symbol Device:R_Small
- removed TP? (x4): TestPoint, VST104_footprints:scope_PAD, symbol Connector:TestPoint
- added C17: 100p, symbol Device:C
- added C18: 100n, symbol Device:C_Small
- added C19: 1n, symbol Device:C_Small
- added C20, C21, C22, C23, C24, C25, C26: 10u, symbol Device:C
- added D13, D14, D8, D9: D, symbol Device:D
- added D15, D16: ESDA25P35, symbol Device:D_Schottky
- added D6: D_TVS, symbol Device:D_TVS
- added F1: 6, symbol Device:Fuse
- added F2, F3, F4, F5: 5A, symbol Device:Fuse
- added J6: Ext_power, symbol Connector:Barrel_Jack
- added J8: Battery, VST104_footprints:PXC_1935187, symbol Connector_Generic:Conn_01x04
- added Q6, Q9: SQD40N06-14L, symbol Device:Q_NMOS_DGS
- added Q7: BSS127S-7, symbol Device:Q_NMOS_DGS
- added R16: 47k, symbol Device:R_Small
- added R17: 5k23, symbol Device:R_Small
- added R19, R31: 100k, symbol Device:R_Small
- added R20: 20k, symbol Device:R_Small
- added R32: 268, symbol Device:R_Small
- added R33: 436, symbol Device:R_Small
- added R34: 150k, symbol Device:R_Small
- added SW2: 300DP3J1BLKM6QE, VST104_footprints:300DP3J1BLKM6QE, symbol Switch:SW_Push_DPDT
- added SW3, SW4: SW_SPST, VST104_footprints:300SP1J1BLKM2QE, symbol Switch:SW_SPST
- added TP1, TP2: TestPoint, VST104_footprints:scope_PAD, symbol Connector:TestPoint
- added TP10, TP4, TP7, TP8, TP9: TestPoint_Alt, VST104_footprints:KSE_PN6095, symbol Connector:TestPoint_Alt
- added U4: LM74700, symbol VST104:LM74700
- added U5, U6: OKR-T6-W12, symbol VST104:OKR-T6-W12
- added U7: TL432DBZ, Package_TO_SOT_SMD:SOT-23, symbol Reference_Voltage:TL432DBZ
- added U8, U9: USBLC6, Package_TO_SOT_SMD:SOT-23-6, symbol Power_Protection:USBLC6-4SC6
- D12: renamed from D?; value ESDA25P35 -> ESDA7P120
- gave numbers to parts that had none: 69
Connections:
- net +5V: now also U8.5 (VBUS)
- net AB_side: now also U8.4 (I/O3)
- net ALTER: now also U9.4 (I/O3)
- net CC1: now also TP1.1
- net CC2: now also TP2.1
- net GND: now also C17.1, C19.2, C20.2, C21.2, C22.2, C23.2, C24.2, C25.2, C26.2, D15.2 (A), D16.2 (A), D6.2 (A2), J6.2, J8.2 (Pin_2), J8.4 (Pin_4), Q7.3 (S), R17.2, R31.2, R32.2, R33.2, TP9.1, U4.2 (GND), U5.3 (GND), U6.3 (GND), U7.3 (A), U8.2 (GND), U9.2 (GND)
- net GNDA: now also TP10.1
- net GPIO: now also U8.1 (I/O1)
- net PDO2: now also Q3.1 (G), R8.1
- net PDO3: now also U8.3 (I/O2); no longer Q3.1 (G), R8.1
- net SCL: now also U9.3 (I/O2)
- net SDA: now also U9.1 (I/O1)
- net SUP_3V3: now also C25.1, D14.1 (K), D16.1 (K), TP8.1
- net SUP_5V: now also D5.1 (K), C26.1, D8.1 (K), D9.1 (K), TP7.1
- net VBUS: no longer J3.A4 (VBUS), J3.A9 (VBUS), J3.B4 (VBUS), J3.B9 (VBUS), Q1.1 (D), R3.2
- net VDD: now also U9.5 (VBUS)
- net VSINK: now also SW2.1 (A)
- net ATTACH: now reaches U1.11 (ATTACH)
- net ATTACH: now also U8.6 (I/O4)
- net at Q3.4 (D): now also R13.2
- net +BATT_1 renamed SUP_BAT_1
- net SUP_BAT_1: now also SW3.1 (A)
- net +BATT_2 renamed SUP_BAT_2
- net SUP_BAT_2: now also SW4.1 (A)
- net +UNREG renamed SUP_UNREG
- net SUP_UNREG: now also C24.1, D13.1 (K), D15.1 (K), TP4.1
- net V_HIGH: no longer names the net of C7.1, Q5.1 (D)
- net V_HIGH: now also F3.2
- net V_LOW: no longer names the net of C6.1, Q4.1 (D)
- net V_LOW: now also SW2.4 (A); no longer D5.1 (K)
- new net: F1.2, J3.A4 (VBUS), J3.A9 (VBUS), J3.B4 (VBUS), J3.B9 (VBUS)
- new net: F1.1, Q1.1 (D), R3.2
- new net: C20.1, F2.1, U5.2 (VIN)
- new net: D8.2 (A), U5.4 (VOUT)
- new net: R32.1, U5.5 (TRIM)
- new net: C23.1, F5.1, U6.2 (VIN)
- new net: D14.2 (A), U6.4 (VOUT)
- new net: R33.1, U6.5 (TRIM)
- new net: J8.1 (Pin_1), SW3.2 (B)
- new net: J8.3 (Pin_3), SW4.2 (B)
- new net: C17.2, C18.1, D6.1 (A1), J6.1, Q6.3 (S), U4.3 (EN), U4.6 (Anode)
- new net: C21.1, D9.2 (A), F3.1
- new net: C22.1, D13.2 (A), F4.1
- new net: F4.2, F5.2, SW2.2 (B)
- new net: F2.2, SW2.5 (B)
- new net: Q6.1 (D), Q9.1 (D), R16.1, R19.1, R20.1, U4.4 (Cathode)
- new net: Q6.2 (G), U4.5 (Gate)
- new net: C18.2, U4.1 (Vcap)
- new net: C19.1, R16.2, R17.1, U7.1 (REF)
- new net: Q7.2 (G), R20.2, R31.1, U7.2 (K)
- new net: Q7.1 (D), R34.2
- new net: Q9.2 (G), R19.2, R34.1
- new net VEXT: Q9.3 (S), SW2.3 (C), SW2.6 (C)
- no-connect marks 13 -> 14
Other:
- moved on the sheet: C1, C10, C11, C12, C13, C14, C15, C2, C3, C4, C5, C6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

Commit message: professor check needed
Parts:
- removed C17: 100p, symbol Device:C
- removed C18: 100n, symbol Device:C_Small
- removed C19: 1n, symbol Device:C_Small
- removed D13, D14: D, symbol Device:D
- removed D6: D_TVS, symbol Device:D_TVS
- removed J6: Ext_power, symbol Connector:Barrel_Jack
- removed J8: Battery, VST104_footprints:PXC_1935187, symbol Connector_Generic:Conn_01x04
- removed Q6, Q9: SQD40N06-14L, symbol Device:Q_NMOS_DGS
- removed Q7: BSS127S-7, symbol Device:Q_NMOS_DGS
- removed R16: 47k, symbol Device:R_Small
- removed R17: 5k23, symbol Device:R_Small
- removed R19, R31: 100k, symbol Device:R_Small
- removed R20: 20k, symbol Device:R_Small
- removed R3: NC, symbol Device:R_Small
- removed R32: 268, symbol Device:R_Small
- removed R34: 150k, symbol Device:R_Small
- removed SW1: SW_Push, symbol Switch:SW_Push
- removed SW3, SW4: SW_SPST, VST104_footprints:300SP1J1BLKM2QE, symbol Switch:SW_SPST
- removed U4: LM74700, symbol VST104:LM74700
- removed U5, U6: OKR-T6-W12, symbol VST104:OKR-T6-W12
- removed U7: TL432DBZ, Package_TO_SOT_SMD:SOT-23, symbol Reference_Voltage:TL432DBZ
- added C?: 100p, symbol Device:C
- added C?: 100n, symbol Device:C_Small
- added C?: 1n, symbol Device:C_Small
- added D?: D_TVS, symbol Device:D_TVS
- added D? (x4): D, symbol Device:D
- added J?: Ext_power, symbol Connector:Barrel_Jack
- added Q?: DMT68M8LSS, symbol Device:Q_NMOS_DGS
- added Q?: 2N7002BK, symbol Device:Q_NMOS_DGS
- added Q?: SI4447ADY, symbol Device:Q_PMOS_DGS
- added R?: 5k23, symbol Device:R_Small
- added R?: 47k, symbol Device:R_Small
- added R?: 20k, symbol Device:R_Small
- added R? (x3): 100k, symbol Device:R_Small
- added R?: 150k, symbol Device:R_Small
- added R? (x2): 436, symbol Device:R_Small
- added R? (x3): 0, VST104_footprints:R_SMD_1206, symbol Device:R
- added R?: NC, VST104_footprints:R_SMD_1206, symbol Device:R
- added TP? (x6): TestPoint_Alt, VST104_footprints:scope_PAD, symbol Connector:TestPoint_Alt
- added U? (x3): OKL-T6-W12, VST104_footprints:OKL-T6-W12, symbol VST104:OKL-T6-W12
- added U?: TL432DBZ, Package_TO_SOT_SMD:SOT-23, symbol Reference_Voltage:TL432DBZ
- added U?: LM74700, symbol VST104:LM74700
- Q1, Q2, Q4, Q5: value STL6P3LLH6 -> SI4447ADY
- Q8: value STR2N2VH5 -> 2N7002BKS
Connections:
- net GND: now also C?.1, C?.2, D?.2 (A2), J?.2, Q?.3 (S), R?.1, R?.2, R?.2, R?.2, R?.2, U?.2 (GND), U?.3 (A), U?.3 (GND), U?.3 (GND), U?.3 (GND), U?.7 (GND), U?.7 (GND), U?.7 (GND)
- net RST: now also R?.2
- net SUP_3V3: now also R?.1, TP?.1; no longer C25.1, D16.1 (K)
- net SUP_5V: now also R?.1, TP?.1; no longer C26.1, D5.1 (K), D8.1 (K), D9.1 (K)
- net SUP_UNREG: now also R?.1, TP?.1; no longer C24.1, D15.1 (K)
- net VBUS: now also F1.1, Q1.1 (D)
- net VSINK: now also D?.2 (A); no longer SW2.1 (A)
- net at C6.1, Q4.1 (D): now also D?.2 (A); no longer SW2.4 (A)
- net at C20.1, F2.1: now also U?.2 (VIN)
- net at D8.2 (A): now also U?.4 (VOUT), U?.5 (Sense)
- net at C23.1, F5.1: now also U?.2 (VIN)
- net at R33.1: now also U?.6 (Trim)
- net at C22.1, F4.1: now also R?.2, U?.2 (VIN)
- net at F4.2, F5.2: now also D?.1 (K), D?.1 (K); no longer SW2.2 (B)
- net at F2.2: now also D?.1 (K), D?.1 (K); no longer SW2.5 (B)
- net VEXT: no longer names the net of SW2.3 (C)
- net VEXT: no longer SW2.6 (C)
- new net: C25.1, D16.1 (K), R?.2, TP?.1, U?.4 (VOUT), U?.5 (Sense)
- new net: C?.1, C?.2, D?.1 (A1), J?.1, Q?.3 (S), U?.3 (EN), U?.6 (Anode)
- new net: Q?.1 (D), Q?.3 (S), R?.1, R?.1, R?.1, U?.4 (Cathode)
- new net: Q?.2 (G), U?.5 (Gate)
- new net: C?.2, U?.1 (Vcap)
- new net: C?.1, R?.1, R?.2, U?.1 (REF)
- new net: Q?.2 (G), R?.1, R?.2, U?.2 (K)
- new net: Q?.1 (D), R?.2
- new net: Q?.2 (G), R?.1, R?.2
- new net: D?.2 (A), D?.2 (A), Q?.1 (D)
- new net: R?.1, U?.6 (Trim) (x2)
- new net: C24.1, D15.1 (K), R?.1, R?.2, TP?.1, U?.4 (VOUT), U?.5 (Sense)
- new net: C26.1, D5.1 (K), D8.1 (K), D9.1 (K), R?.2, TP?.1
- no-connect marks 14 -> 18
Other:
- moved on the sheet: C20, C21, C23, C24, C25, C26, D15, D16, D5, D8, D9, F1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
