File: element_foxtrot/element_foxtrot.kicad_pcb (KiCad board)
At the start: 2 copper layers, 31 parts, among them J1 Conn_02x26_Top_Bottom, J2 Conn_02x26_Top_Bottom, J8 Battery, SW2 300DP3J1BLKM6QE, SW3 SW_SPST, SW4 SW_SPST, U1 STUSB4500QTR, U3 USBLC6, U5 OKR-T6-W12, U6 OKR-T6-W12, U7 TL432DBZ, U8 USBLC6, U9 USBLC6

Commit message: libraries for foxtrot
Parts:
- removed J1, J2: Conn_02x26_Top_Bottom, VST104_footprints:CES-126-01-x-D
- removed J8: Battery, VST104_footprints:PXC_1935187
- removed SW2: 300DP3J1BLKM6QE, VST104_footprints:300DP3J1BLKM6QE
- removed SW3, SW4: SW_SPST, VST104_footprints:300SP1J1BLKM2QE
- removed the TP1 at (229.5, -22.4)
- removed the TP1 at (97.7, -6.66)
- removed the TP2 at (232.1, -22.4)
- removed the TP2 at (100.3, -6.66)
- removed the TP4 at (215.0, 28.8)
- removed the TP4 at (105.6, -6.66)
- removed the TP7 at (215.6, 61.0)
- removed the TP7 at (113.4, -6.66)
- removed U8, U9: USBLC6, Package_TO_SOT_SMD:SOT-23-6
- added J3: Conn_02x26_Top_Bottom, VST104_footprints:CES-126-01-x-D, F.Cu at (184.3, -128.8)
- added J4: Conn_02x26_Top_Bottom, VST104_footprints:CES-126-01-x-D, F.Cu at (184.3, -121.8)
- added J5: Ext_Power, VST104_footprints:PJ-063AH, F.Cu at (183.6, -96.7)
- added J6: Program, VST104_footprints:TSW-105-07-x-S, F.Cu at (203.6, -101.0)
- added J7: USB, VST104_footprints:TSW-104-07-x-S, F.Cu at (202.3, -88.4)
- added P1: USB_C_Plug, VST104_footprints:CX90M-16P, F.Cu at (203.4, -93.6)
- added R34: 0, VST104_footprints:R_SMD_1206, F.Cu at (190.4, -88.7)
- added R35: 0, VST104_footprints:R_SMD_1206, F.Cu at (213.5, -101.4)
- added R36: 0, VST104_footprints:R_SMD_1206, F.Cu at (219.0, -101.4)
- added SW1: switch_3P3T, VST104_footprints:G-168S-3011, F.Cu at (197.9, -111.3)
- added TP1: TestPoint, VST104_footprints:scope_PAD, F.Cu at (194.5, -89.1)
- added TP11: TestPoint_Alt, VST104_footprints:scope_PAD, F.Cu at (261.5, -115.7)
- added TP12: TestPoint_Alt, VST104_footprints:scope_PAD, F.Cu at (232.8, -89.5)
- added TP13: TestPoint_Alt, VST104_footprints:scope_PAD, F.Cu at (235.4, -89.6)
- added TP14: TestPoint_Alt, VST104_footprints:scope_PAD, F.Cu at (232.8, -92.1)
- added TP15: TestPoint_Alt, VST104_footprints:scope_PAD, F.Cu at (194.5, -86.4)
- added TP2: TestPoint, VST104_footprints:scope_PAD, F.Cu at (191.6, -85.8)
- added TP4: TestPoint, VST104_footprints:scope_PAD, F.Cu at (229.2, -101.7)
- added TP7: TestPoint_Alt, VST104_footprints:KSE_PN6095, F.Cu at (250.1, -110.5)
- added U2: TL432DBZ, Package_TO_SOT_SMD:SOT-23, F.Cu at (225.6, -100.8)
- added U4: OKL-T6-W12, VST104_footprints:OKL-T6-W12, F.Cu at (222.2, -111.3)
- TP10: footprint VST104_footprints:KSE_PN6095 -> VST104_footprints:scope_PAD
- TP5, TP6: value TestPoint -> TestPoint_Alt; footprint VST104_footprints:scope_PAD -> VST104_footprints:KSE_PN6095
- U1: value STUSB4500QTR -> L7985; footprint Package_DFN_QFN:QFN-24-1EP_4x4mm_P0.5mm_EP2.7x2.7mm -> VST104_footprints:HSOP8_3.9x4.9mm_EP
- U3: value USBLC6 -> STUSB4500QTR; footprint Package_TO_SOT_SMD:SOT-666 -> VST104_footprints:QFN-24_4.0x4.0mm_EP
- U5: value OKR-T6-W12 -> OKL-T6-W12; footprint VST104_footprints:OKR-T6-W12 -> VST104_footprints:OKL-T6-W12
- U6: value OKR-T6-W12 -> USBLC6; footprint VST104_footprints:OKR-T6-W12 -> VST104_footprints:SOT-363_TSSOP-6_2.0x1.25mm
- U7: value TL432DBZ -> USBLC6; footprint Package_TO_SOT_SMD:SOT-23 -> VST104_footprints:SOT-363_TSSOP-6_2.0x1.25mm
- moved TP5 167.0 mm to (237.0, -113.0)
- moved U1 162.5 mm to (227.4, -90.2)
- moved TP3 154.7 mm to (228.4, -97.2)
- moved TP9 151.6 mm to (250.1, -97.5)
- moved TP8 143.0 mm to (237.0, -100.0)
- moved TP10 136.7 mm to (189.0, -85.8)
- moved TP6 136.4 mm to (216.9, -92.4)
- moved U3 121.4 mm to (184.7, -87.4)
- moved U5 74.0 mm to (258.6, -125.3)
- moved U7 72.1 mm to (225.2, -96.6)
- moved U6 63.8 mm to (258.4, -115.2)
Connections:
- TP10 pad 1: GNDA -> Net-(C20-Pad1)
- TP3 pad 1: /VSINK -> /GPIO
- TP5 pad 1: /GPIO -> /SUP_UNREG
- TP6 pad 1: /PDO2 -> /SUP_5V
- TP8 pad 1: /SUP_3V3 -> GND
- TP9 pad 1: GND -> GNDA
- U1 pad 1: /CC1 -> (no net)
- U1 pad 2: /CC1 -> (no net)
- U1 pad 3: (no net) -> /VSINK
- U1 pad 4: /CC2 -> (no net)
- U1 pad 5: /CC2 -> (no net)
- U1 pad 7: /SCL -> GND
- U1 pad 8: /SDA -> /VSINK
- U3 pad 1: (no net) -> /CC1
- U3 pad 2: GND -> /CC1
- U3 pad 4: (no net) -> /CC2
- U3 pad 5: +5V -> /CC2
- U5 pad 1: (no net) -> Net-(R28-Pad1)
- U5 pad 2: (no net) -> Net-(C18-Pad1)
- U5 pad 4: (no net) -> Net-(C22-Pad1)
- U5 pad 5: (no net) -> Net-(C22-Pad1)
- U6 pad 1: (no net) -> /SDA
- U6 pad 2: (no net) -> GND
- U6 pad 3: GND -> /SCL
- U6 pad 4: (no net) -> /ALTER
- U6 pad 5: (no net) -> VDD
- U7 pad 1: (no net) -> /USB_N
- U7 pad 2: (no net) -> GND
- U7 pad 3: GND -> /USB_P

Commit message: ready for wiring
Parts:
- added 2A1: Fuse, VST104_footprints:R_SMD_0603, F.Cu at (90.0, 332.2)
- added C1: 10u, VST104_footprints:C_SMD_0805, F.Cu at (77.4, 328.5)
- added C10: 2n2, VST104_footprints:C_SMD_0603, F.Cu at (51.2, 332.4)
- added C11: 1n, VST104_footprints:C_SMD_0603, F.Cu at (98.4, 335.6)
- added C12: 1u, VST104_footprints:C_SMD_0603, F.Cu at (97.0, 339.4)
- added C13: 1u, VST104_footprints:C_SMD_0603, F.Cu at (102.8, 332.7)
- added C14: 1u, VST104_footprints:C_SMD_0603, F.Cu at (107.2, 329.7)
- added C15: 470u, VST104_footprints:CP_Radial_D8.0mm_P3.50mm_L11.5mm, F.Cu at (45.7, 348.6)
- added C16: 470u, VST104_footprints:CP_Radial_D8.0mm_P3.50mm_L11.5mm, F.Cu at (55.2, 348.6)
- added C17: 22u, VST104_footprints:C_SMD_0805, F.Cu at (88.4, 342.5)
- added C18: 22u, VST104_footprints:C_SMD_0805, F.Cu at (98.6, 332.9)
- added C19: 1u, VST104_footprints:C_SMD_0603, F.Cu at (92.2, 345.2)
- added C2: 220n, VST104_footprints:C_SMD_0603, F.Cu at (47.2, 332.4)
- added C20: 10u, VST104_footprints:C_SMD_0805, F.Cu at (103.0, 330.0)
- added C21: 10u, VST104_footprints:C_SMD_0805, F.Cu at (88.4, 339.6)
- added C22: 10u, VST104_footprints:C_SMD_0805, F.Cu at (92.8, 339.6)
- added C3: 100p, VST104_footprints:C_SMD_0603, F.Cu at (88.2, 345.2)
- added C4: 22n, VST104_footprints:C_SMD_0603, F.Cu at (43.3, 334.1)
- added C5: 1n, VST104_footprints:C_SMD_0603, F.Cu at (81.6, 331.2)
- added C6: 1u, VST104_footprints:C_SMD_0603, F.Cu at (92.6, 342.3)
- added C7: 4u7, VST104_footprints:C_SMD_0805, F.Cu at (98.6, 330.0)
- added C8: 10u, VST104_footprints:C_SMD_0805, F.Cu at (81.8, 328.5)
- added C9: 220u, VST104_footprints:CP_Radial_D6.3mm_P2.50mm_L11.2mm, F.Cu at (69.6, 350.7)
- added D1: SMAJ15CA, VST104_footprints:D_SMA_DO-214AC_4.3x2.6mm, F.Cu at (48.0, 338.6)
- added D10: BAV199, VST104_footprints:SOT-23-3_2.9x1.3mm, F.Cu at (51.2, 355.5)
- added D11: DDZ15CSF, VST104_footprints:D_SOD-323-F_1.25x1.7mm, F.Cu at (125.2, 357.7)
- added D12: BAV199, VST104_footprints:SOT-23-3_2.9x1.3mm, F.Cu at (62.2, 346.0)
- added D13: LED, VST104_footprints:D_SMD_0603_LED, F.Cu at (129.3, 357.5)
- added D14: LED, VST104_footprints:D_SMD_0603_LED, F.Cu at (120.8, 365.6)
- added D15: LED, VST104_footprints:D_SMD_0603_LED, F.Cu at (124.8, 363.1)
- added D16: FM4004W, VST104_footprints:D_SMA_DO-214AC_4.3x2.6mm, F.Cu at (44.9, 355.5)
- added D2: STPS3L60UFN, VST104_footprints:D_SMB-FN_DO-214AA-FN, F.Cu at (184.6, 344.6)
- added D3: SMAJ15CA, VST104_footprints:D_SMA_DO-214AC_4.3x2.6mm, F.Cu at (45.3, 329.1)
- added D4: ESDA25W5, VST104_footprints:SOT-323-5L_2.0x1.25mm, F.Cu at (73.0, 328.8)
- added D5: BAT54JFILM, VST104_footprints:D_SOD-323_1.65x1.28mm, F.Cu at (75.8, 348.2)
- added D6: DDZ15CSF, VST104_footprints:D_SOD-323-F_1.25x1.7mm, F.Cu at (120.9, 357.7)
- added D7: LED, VST104_footprints:D_SMD_0603_LED, F.Cu at (120.8, 363.1)
- added D8: LED, VST104_footprints:D_SMD_0603_LED, F.Cu at (125.0, 360.3)
- added D9: DDZ15CSF, VST104_footprints:D_SOD-323-F_1.25x1.7mm, F.Cu at (120.9, 360.5)
- added F1: 10A, VST104_footprints:FUSE_2AG_01110501Z, F.Cu at (90.7, 352.6)
- added F2: 10A, VST104_footprints:FUSE_2AG_01110501Z, F.Cu at (90.7, 362.3)
- added F3: 5A, VST104_footprints:FUSE_2AG_01110501Z, F.Cu at (109.4, 352.6)
- added F4: 5A, VST104_footprints:FUSE_2AG_01110501Z, F.Cu at (90.7, 371.9)
- added F5: 5A, VST104_footprints:FUSE_2AG_01110501Z, F.Cu at (109.4, 362.3)
- added F6: 5A, VST104_footprints:FUSE_2AG_01110501Z, F.Cu at (109.4, 371.9)
- added J1: Conn_02x26_Top_Bottom, VST104_footprints:CES-126-01-x-D, F.Cu at (38.6, 236.5)
- added J2: Conn_02x26_Top_Bottom, VST104_footprints:CES-126-01-x-D, F.Cu at (38.6, 231.4)
- added J8: TSW-102-07-T-D, VST104_footprints:TSW-102-07-x-D, F.Cu at (200.8, 316.3)
- added L1: 22u, VST104_footprints:L_SMD_8040_8.0x8.0x4.2mm, F.Cu at (91.3, 333.3)
- added Q1: SQD40061EL, VST104_footprints:TO-252AA_6.5x6.1mm, F.Cu at (45.4, 325.1)
- added Q10: 2N7002BK, VST104_footprints:SOT-23-3_2.9x1.3mm, F.Cu at (68.5, 329.1)
- added Q2: SQD40061EL, VST104_footprints:TO-252AA_6.5x6.1mm, F.Cu at (53.5, 325.1)
- added Q3: SQD40061EL, VST104_footprints:TO-252AA_6.5x6.1mm, F.Cu at (61.6, 325.1)
- added Q4: SQD40061EL, VST104_footprints:TO-252AA_6.5x6.1mm, F.Cu at (69.7, 325.1)
- added Q5: 2N7002BK, VST104_footprints:SOT-23-3_2.9x1.3mm, F.Cu at (64.1, 329.1)
- added Q6: SQD40061EL, VST104_footprints:TO-252AA_6.5x6.1mm, F.Cu at (77.8, 325.1)
- added Q7: 2N7002BK, VST104_footprints:SOT-23-3_2.9x1.3mm, F.Cu at (59.6, 329.1)
- added Q8: SQD40061EL, VST104_footprints:TO-252AA_6.5x6.1mm, F.Cu at (86.0, 325.1)
- added Q9: SQD40061EL, VST104_footprints:TO-252AA_6.5x6.1mm, F.Cu at (94.1, 325.1)
- added R1: 1k, VST104_footprints:R_SMD_0603, F.Cu at (102.8, 335.2)
- added R10: 5k23, VST104_footprints:R_SMD_0603, F.Cu at (111.1, 332.2)
- added R11: 5k1, VST104_footprints:R_SMD_0603, F.Cu at (47.2, 334.9)
- added R12: 698, VST104_footprints:R_SMD_0603, F.Cu at (51.2, 334.9)
- added R13: 100k, VST104_footprints:R_SMD_0603, F.Cu at (115.1, 329.7)
- added R14: 20k, VST104_footprints:R_SMD_0603, F.Cu at (100.1, 344.8)
- added R15: 100k, VST104_footprints:R_SMD_0603, F.Cu at (104.5, 340.6)
- added R16: 100k, VST104_footprints:R_SMD_0603, F.Cu at (110.7, 334.7)
- added R17: 22k, VST104_footprints:R_SMD_0603, F.Cu at (108.9, 337.2)
- added R18: 100k, VST104_footprints:R_SMD_0603, F.Cu at (115.1, 332.2)
- added R19: 22k, VST104_footprints:R_SMD_0603, F.Cu at (108.9, 339.7)
- added R2: 470, VST104_footprints:R_SMD_0603, F.Cu at (101.0, 338.1)
- added R20: 1k, VST104_footprints:R_SMD_0603, F.Cu at (104.5, 343.1)
- added R21: 1k2, VST104_footprints:R_SMD_0603, F.Cu at (114.6, 334.7)
- added R22: 250, VST104_footprints:R_SMD_0603, F.Cu at (112.8, 337.2)
- added R23: 100k, VST104_footprints:R_SMD_0603, F.Cu at (104.9, 337.7)
- added R24: 100k, VST104_footprints:R_SMD_0603, F.Cu at (108.4, 342.2)
- added R25: 100k, VST104_footprints:R_SMD_0603, F.Cu at (112.8, 339.7)
- added R26: 100k, VST104_footprints:R_SMD_0603, F.Cu at (108.4, 344.7)
- added R27: 250, VST104_footprints:R_SMD_0603, F.Cu at (116.8, 337.2)
- added R28: 100, VST104_footprints:R_SMD_0603, F.Cu at (112.4, 342.2)
- added R29: 10k, VST104_footprints:R_SMD_0603, F.Cu at (116.8, 339.7)
- added R3: 1k, VST104_footprints:R_SMD_0603, F.Cu at (107.2, 332.2)
- added R30: 10k, VST104_footprints:R_SMD_0603, F.Cu at (112.4, 344.7)
- added R31: 10k, VST104_footprints:R_SMD_0603, F.Cu at (116.3, 342.2)
- added R32: 2k18, VST104_footprints:R_SMD_0603, F.Cu at (116.3, 344.7)
- added R33: 1k34, VST104_footprints:R_SMD_0603, F.Cu at (104.0, 345.6)
- added R4: 100k, VST104_footprints:R_SMD_0603, F.Cu at (111.1, 329.7)
- added R5: 10k, VST104_footprints:R_SMD_0603, F.Cu at (96.1, 344.8)
- added R6: 100, VST104_footprints:R_SMD_0603, F.Cu at (55.1, 332.4)
- added R7: 1k2, VST104_footprints:R_SMD_0603, F.Cu at (100.5, 341.9)
- added R8: 1k2, VST104_footprints:R_SMD_0603, F.Cu at (106.7, 334.7)
- added R9: 47k, VST104_footprints:R_SMD_0603, F.Cu at (96.6, 342.3)
- J3: value Conn_02x26_Top_Bottom -> Ext_Power; footprint VST104_footprints:CES-126-01-x-D -> VST104_footprints:PJ-063AH
- J4: value Conn_02x26_Top_Bottom -> Program; footprint VST104_footprints:CES-126-01-x-D -> VST104_footprints:TSW-105-07-x-S
- J5: value Ext_Power -> USB; footprint VST104_footprints:PJ-063AH -> VST104_footprints:TSW-104-07-x-S
- J6: value Program -> TSW-102-07-T-D; footprint VST104_footprints:TSW-105-07-x-S -> VST104_footprints:TSW-102-07-x-D
- J7: value USB -> TSW-102-07-T-D; footprint VST104_footprints:TSW-104-07-x-S -> VST104_footprints:TSW-102-07-x-D
- P1: value USB_C_Plug -> CX90M-16P
- U6: value USBLC6 -> USBLC6-4; footprint VST104_footprints:SOT-363_TSSOP-6_2.0x1.25mm -> VST104_footprints:SOT-23-6L_2.9x1.6mm
- U7: value USBLC6 -> USBLC6-2; footprint VST104_footprints:SOT-363_TSSOP-6_2.0x1.25mm -> VST104_footprints:SOT-23-6L_2.9x1.6mm
- moved P1 453.4 mm to (125.8, 353.1)
- moved J3 431.9 mm to (163.7, 302.7)
- moved R34 404.1 mm to (52.5, 291.1)
- moved TP11 404.1 mm to (123.6, 264.1)
- moved TP4 404.1 mm to (91.2, 278.1)
- moved U4 404.1 mm to (84.3, 268.5)
- moved J4 404.1 mm to (46.3, 258.1)
- moved J5 404.1 mm to (45.7, 283.1)
- moved R35 404.1 mm to (75.5, 278.4)
- moved R36 404.1 mm to (81.1, 278.4)
- moved SW1 404.1 mm to (59.9, 268.5)
- moved TP1 404.1 mm to (56.6, 290.8)
- moved TP10 404.1 mm to (51.0, 294.1)
- moved TP12 404.1 mm to (94.8, 290.3)
- moved TP13 404.1 mm to (97.4, 290.2)
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Connections:
- J3 pad 1: /H1-1 -> Net-(F1-Pad2)
- J3 pad 2: /H1-2 -> GND
- J4 pad 1: /H2-1 -> VDD
- J4 pad 2: /H2-2 -> GND
- J4 pad 3: /H2-3 -> /ALTER
- J4 pad 4: /H2-4 -> /SCL
- J4 pad 5: /H2-5 -> /SDA
- J5 pad 1: (no net) -> +5V
- J5 pad 2: GND -> /USB_P
- J6 pad 1: VDD -> Net-(J6-Pad1)
- J6 pad 2: GND -> Net-(J6-Pad1)
- J6 pad 3: /ALTER -> /SUP_UNREG
- J6 pad 4: /SCL -> /SUP_UNREG
- J7 pad 1: +5V -> Net-(J7-Pad1)
- J7 pad 2: /USB_P -> Net-(J7-Pad1)
- J7 pad 3: /USB_N -> /SUP_3V3
- J7 pad 4: GND -> /SUP_3V3
- P1 pad B6: (no net) -> /USB_P
- P1 pad B7: (no net) -> /USB_N
- P1 pad MH: (no net) -> Net-(P1-PadMH)
- R34 pad 1: /SUP_UNREG -> Net-(J6-Pad1)
- R35 pad 1: /SUP_3V3 -> Net-(J7-Pad1)
- R36 pad 1: /SUP_5V -> Net-(J8-Pad1)
- SW1 pad 2: Net-(SW1-Pad2) -> (no net)
- SW1 pad 3: Net-(SW1-Pad3) -> (no net)
- SW1 pad 5: (no net) -> Net-(R19-Pad2)
- SW1 pad 6: (no net) -> Net-(Q5-Pad3)
- TP13 pad 1: /SUP_UNREG -> Net-(J6-Pad1)
- TP14 pad 1: /SUP_3V3 -> Net-(J7-Pad1)
- TP15 pad 1: /SUP_5V -> Net-(J8-Pad1)
- U1 pad 1: (no net) -> Net-(D2-Pad1)
- U1 pad 4: (no net) -> Net-(C4-Pad1)
- U1 pad 5: (no net) -> Net-(C5-Pad2)
- U2 pad 1: (no net) -> Net-(C11-Pad1)
- U2 pad 2: (no net) -> Net-(R14-Pad2)
- U3 pad 18: (no net) -> Net-(R1-Pad2)
- U3 pad 21: (no net) -> Net-(C13-Pad2)
- U3 pad 23: (no net) -> Net-(C14-Pad2)
- U3 pad 24: (no net) -> Net-(C12-Pad2)
- U3 pad 6: (no net) -> /RST
- U3 pad 9: (no net) -> Net-(R20-Pad1)

Commit message: tracing foxtrot
Parts:
- removed the D1 at (48.0, 338.6)
- removed the D3 at (45.3, 329.1)
- removed the D7 at (120.8, 363.1)
- removed the Q1 at (45.4, 325.1)
- removed the R11 at (47.2, 334.9)
- removed the R16 at (110.7, 334.7)
- removed the R26 at (108.4, 344.7)
- removed the R29 at (116.8, 339.7)
- removed the R34 at (52.5, 291.1)
- removed the R4 at (111.1, 329.7)
- removed the R5 at (96.1, 344.8)
- removed the R6 at (55.1, 332.4)
- removed TP15: TestPoint_Alt, VST104_footprints:scope_PAD
- removed the TP2 at (53.7, 294.1)
- removed the TP3 at (90.4, 282.6)
- added D13: BAV199, VST104_footprints:SOT-23-3_2.9x1.3mm, F.Cu at (172.0, 82.1)
- added D14: DDZ15CSF, VST104_footprints:D_SOD-323-F_1.25x1.7mm, F.Cu at (184.5, 84.2)
- added D15: BAV199, VST104_footprints:SOT-23-3_2.9x1.3mm, F.Cu at (172.0, 78.4)
- added D5: SMAJ15CA, VST104_footprints:D_SMA_DO-214AC_4.3x2.6mm, F.Cu at (141.2, 71.5)
- added H1: MountingHole_Pad, VST104_footprints:MountingHole_3.2mm_M3_Pad_Via, F.Cu at (222.5, 62.5)
- added H10: MountingHole_Pad, VST104_footprints:MountingHole_3.2mm_M3_Pad_Via, F.Cu at (222.5, 223.8)
- added H11: MountingHole_Pad, VST104_footprints:MountingHole_3.2mm_M3_Pad_Via, F.Cu at (126.2, 223.8)
- added H12: MountingHole_Pad, VST104_footprints:MountingHole_3.2mm_M3_Pad_Via, F.Cu at (30.0, 223.8)
- added H13: MountingHole_Pad, VST104_footprints:MountingHole_3.2mm_M3_Pad_Via, F.Cu at (222.5, 332.5)
- added H14: MountingHole_Pad, VST104_footprints:MountingHole_3.2mm_M3_Pad_Via, F.Cu at (127.5, 332.5)
- added H15: MountingHole_Pad, VST104_footprints:MountingHole_3.2mm_M3_Pad_Via, F.Cu at (30.0, 332.5)
- added H2: MountingHole_Pad, VST104_footprints:MountingHole_3.2mm_M3_Pad_Via, F.Cu at (222.5, 97.5)
- added H3: MountingHole_Pad, VST104_footprints:MountingHole_3.2mm_M3_Pad_Via, F.Cu at (126.2, 62.5)
- added H4: MountingHole_Pad, VST104_footprints:MountingHole_3.2mm_M3_Pad_Via, F.Cu at (126.2, 97.5)
- added H5: MountingHole_Pad, VST104_footprints:MountingHole_3.2mm_M3_Pad_Via, F.Cu at (30.0, 62.5)
- added H6: MountingHole_Pad, VST104_footprints:MountingHole_3.2mm_M3_Pad_Via, F.Cu at (30.0, 97.5)
- added H7: MountingHole_Pad, VST104_footprints:MountingHole_3.2mm_M3_Pad_Via, F.Cu at (222.5, 109.5)
- added H8: MountingHole_Pad, VST104_footprints:MountingHole_3.2mm_M3_Pad_Via, F.Cu at (126.2, 109.5)
- added H9: MountingHole_Pad, VST104_footprints:MountingHole_3.2mm_M3_Pad_Via, F.Cu at (30.0, 109.5)
- added Q7: SQD40061EL, VST104_footprints:TO-252AA_6.5x6.1mm, F.Cu at (187.2, 92.4)
- added R12: 1k2, VST104_footprints:R_SMD_0805, F.Cu at (198.5, 81.2)
- added R21: 100k, VST104_footprints:R_SMD_0805, F.Cu at (178.8, 74.8)
- added R22: 22k, VST104_footprints:R_SMD_0805, F.Cu at (157.0, 92.2)
- added R23: 100k, VST104_footprints:R_SMD_0805, F.Cu at (182.5, 84.2)
- added R24: 22k, VST104_footprints:R_SMD_0805, F.Cu at (183.5, 81.2)
- added R25: 1k, VST104_footprints:R_SMD_0805, F.Cu at (166.2, 86.0)
- added R32: 10k, VST104_footprints:R_SMD_0805, F.Cu at (173.8, 89.8)
- added R37: 0, VST104_footprints:R_SMD_1206, F.Cu at (51.5, 90.5)
- added R7: 1k, VST104_footprints:R_SMD_0805, F.Cu at (206.8, 87.0)
- added TP4: TestPoint, VST104_footprints:scope_PAD, F.Cu at (161.5, 71.0)
- 2A1: footprint VST104_footprints:R_SMD_0603 -> VST104_footprints:C_SMD_0805
- C10, C11, C12, C13, C14, C19, C2, C3, C4, C5, C6: footprint VST104_footprints:C_SMD_0603 -> VST104_footprints:C_SMD_0805
- D1: renamed from D14; footprint VST104_footprints:D_SMD_0603_LED -> VST104_footprints:D_SMD_0805_LED
- D10, D12: value BAV199 -> LED; footprint VST104_footprints:SOT-23-3_2.9x1.3mm -> VST104_footprints:D_SMD_0805_LED
- D16: renamed from D13; footprint VST104_footprints:D_SMD_0603_LED -> VST104_footprints:D_SMD_0805_LED
- D2: value STPS3L60UFN -> SMAJ15CA; footprint VST104_footprints:D_SMB-FN_DO-214AA-FN -> VST104_footprints:D_SMA_DO-214AC_4.3x2.6mm
- D3: renamed from D15; footprint VST104_footprints:D_SMD_0603_LED -> VST104_footprints:D_SMD_0805_LED
- D4: value ESDA25W5 -> STPS3L60UFN; footprint VST104_footprints:SOT-323-5L_2.0x1.25mm -> VST104_footprints:D_SMB-FN_DO-214AA-FN
- D6: value DDZ15CSF -> ESDA25W5; footprint VST104_footprints:D_SOD-323-F_1.25x1.7mm -> VST104_footprints:SOT-323-5L_2.0x1.25mm
- D8: value LED -> DDZ15CSF; footprint VST104_footprints:D_SMD_0603_LED -> VST104_footprints:D_SOD-323-F_1.25x1.7mm
- D9: value DDZ15CSF -> LED; footprint VST104_footprints:D_SOD-323-F_1.25x1.7mm -> VST104_footprints:D_SMD_0805_LED
- P1: value CX90M-16P -> Val**
- Q5: value 2N7002BK -> SQD40061EL; footprint VST104_footprints:SOT-23-3_2.9x1.3mm -> VST104_footprints:TO-252AA_6.5x6.1mm
- Q6: value SQD40061EL -> 2N7002BK; footprint VST104_footprints:TO-252AA_6.5x6.1mm -> VST104_footprints:SOT-23-3_2.9x1.3mm
- R1: renamed from R22; footprint VST104_footprints:R_SMD_0603 -> VST104_footprints:R_SMD_0805
- R10: value 5k23 -> 100; footprint VST104_footprints:R_SMD_0603 -> VST104_footprints:R_SMD_0805
- R11: renamed from R7; footprint VST104_footprints:R_SMD_0603 -> VST104_footprints:R_SMD_0805
- R13: value 100k -> 47k; footprint VST104_footprints:R_SMD_0603 -> VST104_footprints:R_SMD_0805
- R14: value 20k -> 5k23; footprint VST104_footprints:R_SMD_0603 -> VST104_footprints:R_SMD_0805
- R15: value 100k -> 5k1; footprint VST104_footprints:R_SMD_0603 -> VST104_footprints:R_SMD_0805
- R16: renamed from R12; footprint VST104_footprints:R_SMD_0603 -> VST104_footprints:R_SMD_0805
- R17: value 22k -> 100k; footprint VST104_footprints:R_SMD_0603 -> VST104_footprints:R_SMD_0805
- R18: value 100k -> 20k; footprint VST104_footprints:R_SMD_0603 -> VST104_footprints:R_SMD_0805
- R19: value 22k -> 1k2; footprint VST104_footprints:R_SMD_0603 -> VST104_footprints:R_SMD_0805
- R2: renamed from R25; footprint VST104_footprints:R_SMD_0603 -> VST104_footprints:R_SMD_0805
- R20, R3: value 1k -> 100k; footprint VST104_footprints:R_SMD_0603 -> VST104_footprints:R_SMD_0805
- R26: renamed from R21; footprint VST104_footprints:R_SMD_0603 -> VST104_footprints:R_SMD_0805
- R27: renamed from R23; footprint VST104_footprints:R_SMD_0603 -> VST104_footprints:R_SMD_0805
- R28: renamed from R24; footprint VST104_footprints:R_SMD_0603 -> VST104_footprints:R_SMD_0805
- R29: renamed from R28; footprint VST104_footprints:R_SMD_0603 -> VST104_footprints:R_SMD_0805
- R30, R31: footprint VST104_footprints:R_SMD_0603 -> VST104_footprints:R_SMD_0805
- R33: renamed from R32; footprint VST104_footprints:R_SMD_0603 -> VST104_footprints:R_SMD_0805
- R34: renamed from R33; footprint VST104_footprints:R_SMD_0603 -> VST104_footprints:R_SMD_0805
- R4: renamed from R27; footprint VST104_footprints:R_SMD_0603 -> VST104_footprints:R_SMD_0805
- R5: renamed from R1; footprint VST104_footprints:R_SMD_0603 -> VST104_footprints:R_SMD_0805
- R6: renamed from R2; footprint VST104_footprints:R_SMD_0603 -> VST104_footprints:R_SMD_0805
- R8: value 1k2 -> 100k; footprint VST104_footprints:R_SMD_0603 -> VST104_footprints:R_SMD_0805
- R9: value 47k -> 10k; footprint VST104_footprints:R_SMD_0603 -> VST104_footprints:R_SMD_0805
- SW1: footprint VST104_footprints:G-168S-3011 -> VST104_footprints:EG4319
- TP9: footprint VST104_footprints:KSE_PN6095 -> VST104_footprints:scope_PAD
- U2: value TL432DBZ -> TL432AIDBZR; footprint Package_TO_SOT_SMD:SOT-23 -> VST104_footprints:SOT-23-3_2.9x1.3mm
- U4, U5: value OKL-T6-W12 -> Val**
- moved F1 309.1 mm to (212.5, 68.5), turned to 90 degrees
- moved D10 308.0 mm to (198.5, 85.0), turned to 90 degrees
- moved C9 307.3 mm to (221.5, 83.5)
- moved D12 304.3 mm to (208.2, 79.0)
- moved F2 299.2 mm to (147.5, 68.5), turned to 90 degrees
- moved F6 297.9 mm to (92.5, 74.5)
- moved F5 297.2 mm to (92.5, 65.5)
- moved C10 296.2 mm to (208.2, 81.2), turned to 180 degrees
- moved P1 294.9 mm to (159.5, 60.1), turned to 180 degrees
- moved C4 293.2 mm to (206.8, 90.8), turned to 90 degrees
- moved D8 291.2 mm to (193.0, 77.1), turned to 90 degrees
- moved D9 290.4 mm to (157.8, 72.4), turned to 180 degrees
- moved D1 288.7 mm to (175.8, 82.2)
- moved R16 287.3 mm to (202.2, 90.5), turned to 270 degrees
- moved Q2 286.9 mm to (195.8, 75.9), turned to 270 degrees
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- renumbered D16 to D17, D5 to D7, Module_4 to Module_1, Module_1 to Module_4, Q10 to Q1, Q9 to Q10, Q7 to Q8, Q8 to Q9, TP4 to TP2, TP1 to TP3
Connections:
- D10 pad 2: Net-(C12-Pad2) -> Net-(D10-Pad2)
- D11 pad 1: Net-(D11-Pad1) -> Net-(C12-Pad2)
- D12 pad 2: Net-(C12-Pad2) -> Net-(D12-Pad2)
- D2 pad 1: Net-(D2-Pad1) -> GND
- D2 pad 2: GND -> Net-(C3-Pad2)
- D4 pad 1: /CC1 -> Net-(D4-Pad1)
- D6 pad 1: Net-(D6-Pad1) -> /CC2
- D6 pad 2: Net-(D6-Pad2) -> GND
- D8 pad 1: GND -> Net-(D8-Pad1)
- D9 pad 1: Net-(C12-Pad2) -> GND
- J4 pad 2: GND -> /SDA
- J4 pad 3: /ALTER -> /SCL
- J4 pad 4: /SCL -> /ALTER
- J4 pad 5: /SDA -> GND
- L1 pad 1: Net-(D2-Pad1) -> Net-(D4-Pad1)
- Q1 pad 1: Net-(Q10-Pad1) (its old number) -> Net-(Q1-Pad1)
- Q2 pad 1: Net-(D9-Pad2) -> Net-(D8-Pad2)
- Q2 pad 2: Net-(C12-Pad2) -> Net-(D8-Pad1)
- Q2 pad 3: VBUS -> Net-(C3-Pad2)
- Q3 pad 2: Net-(D11-Pad1) -> Net-(C12-Pad2)
- Q3 pad 3: Net-(D6-Pad1) -> VBUS
- Q4 pad 1: Net-(D9-Pad2) -> Net-(D14-Pad2)
- Q4 pad 2: Net-(C12-Pad2) -> Net-(D14-Pad1)
- Q4 pad 3: /VSINK -> Net-(D8-Pad1)
- Q5 pad 1: Net-(Q5-Pad1) -> Net-(D11-Pad2)
- Q5 pad 2: GND -> Net-(C12-Pad2)
- Q5 pad 3: Net-(Q5-Pad3) -> /VSINK
- Q6 pad 1: Net-(D11-Pad2) -> Net-(Q6-Pad1)
- Q6 pad 2: Net-(D11-Pad1) -> GND
- Q6 pad 3: /VSINK -> Net-(Q6-Pad3)
- Q8 pad 1: Net-(Q7-Pad1) -> Net-(Q8-Pad1)
- Q9 pad 1: Net-(Q7-Pad1) -> Net-(Q8-Pad1)
- R10 pad 1: Net-(C11-Pad1) -> Net-(C5-Pad2)
- R10 pad 2: GND -> Net-(C10-Pad2)
- R11 pad 2: Net-(D7-Pad2) -> Net-(D9-Pad2)
- R13 pad 1: Net-(C12-Pad2) -> Net-(D8-Pad1)
- R13 pad 2: Net-(D9-Pad2) -> Net-(C11-Pad1)
- R14 pad 1: Net-(D6-Pad1) -> Net-(C11-Pad1)
- R14 pad 2: Net-(R14-Pad2) -> GND
- R15 pad 1: Net-(R14-Pad2) -> Net-(C5-Pad2)
- R15 pad 2: Net-(Q5-Pad1) -> Net-(2A1-Pad2)
- R17 pad 1: Net-(D9-Pad2) -> Net-(C12-Pad2)
- R17 pad 2: Net-(R17-Pad2) -> Net-(D11-Pad2)
- R18 pad 1: Net-(D11-Pad1) -> Net-(D8-Pad1)
- R18 pad 2: Net-(D11-Pad2) -> Net-(R18-Pad2)
- R19 pad 1: Net-(D11-Pad2) -> Net-(2A1-Pad2)
- R19 pad 2: Net-(R19-Pad2) -> Net-(D12-Pad2)
- R2 pad 1: Net-(Q10-Pad1) (its old number) -> Net-(Q1-Pad1)
- R20 pad 1: Net-(R20-Pad1) -> Net-(R18-Pad2)
- R20 pad 2: /VSINK -> Net-(Q6-Pad1)
- R27 pad 2: Net-(Q7-Pad1) -> Net-(Q8-Pad1)
- R3 pad 1: Net-(C5-Pad2) -> Net-(Q1-Pad1)
- R3 pad 2: Net-(C4-Pad2) -> GND
- R30 pad 2: /SCL -> /ALTER
- R31 pad 2: /ALTER -> /SCL
- R35 pad 1: Net-(J7-Pad1) -> Net-(J6-Pad1)
- R35 pad 2: Net-(C21-Pad1) -> Net-(C20-Pad1)
- R36 pad 1: Net-(J8-Pad1) -> Net-(J7-Pad1)
- R36 pad 2: Net-(C22-Pad1) -> Net-(C21-Pad1)
- R8 pad 1: Net-(D6-Pad1) -> GND
- R8 pad 2: Net-(D8-Pad2) -> /RST
- R9 pad 1: Net-(D6-Pad1) -> Net-(D8-Pad2)
- R9 pad 2: Net-(C11-Pad1) -> GND
- SW1 pad 1: Net-(R17-Pad2) -> (no net)
- SW1 pad 10: GND -> Net-(Q8-Pad1)
- SW1 pad 2: (no net) -> Net-(R22-Pad2)
- SW1 pad 4: Net-(D10-Pad3) -> Net-(D13-Pad3)
- SW1 pad 5: Net-(R19-Pad2) -> Net-(Q6-Pad3)
- SW1 pad 6: Net-(Q5-Pad3) -> Net-(R24-Pad2)
- SW1 pad 9: Net-(Q7-Pad1) -> GND
- TP10 pad 1: Net-(C20-Pad1) -> Net-(C21-Pad1)
- TP11 pad 1: Net-(C21-Pad1) -> Net-(C22-Pad1)
- TP12 pad 1: Net-(C22-Pad1) -> Net-(J6-Pad1)
- TP13 pad 1: Net-(J6-Pad1) -> Net-(J7-Pad1)
- TP14 pad 1: Net-(J7-Pad1) -> Net-(J8-Pad1)
- TP9 pad 1: GNDA -> Net-(C20-Pad1)
- U1 pad 1: Net-(D2-Pad1) -> Net-(D4-Pad1)
- U2 pad 2: Net-(R14-Pad2) -> Net-(R18-Pad2)
- U3 pad 16: Net-(D10-Pad3) -> Net-(D13-Pad3)
- U3 pad 9: Net-(R20-Pad1) -> Net-(R25-Pad1)
Routing:
- net GND: track 0.00 -> 32.8 mm, vias 0 -> 39
- net VDD: track 0.00 -> 31.4 mm, vias 0 -> 2
- net /CC2: track 0.00 -> 27.0 mm, vias 0 -> 2
- net /ALTER: track 0.00 -> 25.3 mm, vias 0 -> 2
- net Net-(C12-Pad2): track 0.00 -> 23.6 mm, vias 0 -> 20
- net /VSINK: track 0.00 -> 23.5 mm, vias 0 -> 2
- net /SCL: track 0.00 -> 22.6 mm, vias 0 -> 1
- net /PDO2: track 0.00 -> 22.0 mm
- net /CC1: track 0.00 -> 21.0 mm, vias 0 -> 2
- net /SDA: track 0.00 -> 20.9 mm, vias 0 -> 1
- net /USB_P: track 0.00 -> 20.2 mm, vias 0 -> 2
- net /USB_N: track 0.00 -> 19.0 mm, vias 0 -> 1
- net Net-(D14-Pad2): track 0.00 -> 18.8 mm, vias 0 -> 2
- net Net-(D11-Pad2): track 0.00 -> 18.7 mm, vias 0 -> 2
- net Net-(R5-Pad2): track 0.00 -> 14.4 mm, vias 0 -> 2
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- added copper zone on B.Cu, net +5V
- added copper zone on F.Cu, net +5V
- added copper zone on F.Cu, net /VSINK
- added copper zone on F.Cu, net GND
- added copper zone on In2.Cu, net GND
- added copper zone on F.Cu, net Net-(2A1-Pad2)
- added copper zone on F.Cu, net Net-(C12-Pad2)
- added copper zone on In1.Cu, net Net-(C12-Pad2)
- added copper zone on F.Cu, net Net-(C3-Pad2)
- added copper zone on In1.Cu, net Net-(C3-Pad2)
- added copper zone on F.Cu, net Net-(C4-Pad1)
- added copper zone on F.Cu, net Net-(C5-Pad2)
- added copper zone on F.Cu, net Net-(D14-Pad1)
- added copper zone on In1.Cu, net Net-(D14-Pad1)
- added copper zone on F.Cu, net Net-(D4-Pad1)
- added copper zone on F.Cu, net Net-(D8-Pad1)
- added copper zone on In1.Cu, net Net-(D8-Pad1)
- added copper zone on F.Cu, net Net-(F1-Pad2)
- added copper zone on In1.Cu, net Net-(F1-Pad2)
- added copper zone on F.Cu, net Net-(F2-Pad2)
- added copper zone on In1.Cu, net Net-(F2-Pad2)
- added copper zone on F.Cu, net VBUS
- added copper zone on In1.Cu, net VBUS
Other:
- board outline added: 202.5 x 280 mm
- copper layers 2 -> 4
- net class Default: clearance 0.2 -> 0.127; trace_width 0.25 -> 0.127; via_dia 0.8 -> 0.6; via_drill 0.4 -> 0.3
- rule trace_clearance: 0.2 -> 0.127
- rule trace_min: 0.2 -> 0
- rule via_min_size: 0.4 -> 0.6

Commit message: ready for check
Parts:
- removed the J1 at (145.2, 116.0)
- removed the J2 at (145.2, 110.0)
- removed Module_3: PC104_module, VST104_footprints:PC104_footprint
- removed the Q9 at (112.5, 65.5)
- removed the R27 at (115.2, 67.0)
- removed TP14: TestPoint_Alt, VST104_footprints:scope_PAD
- removed the TP4 at (161.5, 71.0)
- added G***: LOGO, VST104_logos:VST_logo_vertical_12.5mm, F.Cu at (33.0, 85.0)
- added G***: LOGO, VST104_logos:OSH_logo_9mm, F.Cu at (33.0, 75.0)
- added G***: LOGO, VST104_logos:VST_logo_vertical_174.5mm, F.Cu at (127.5, 350.0)
- added H16: MountingHole_Pad, VST104_footprints:MountingHole_3.2mm_M3_Pad_Via, F.Cu at (30.0, 367.5)
- added H17: MountingHole_Pad, VST104_footprints:MountingHole_3.2mm_M3_Pad_Via, F.Cu at (127.5, 367.5)
- added H18: MountingHole_Pad, VST104_footprints:MountingHole_3.2mm_M3_Pad_Via, F.Cu at (222.5, 367.5)
- added J4: TSW-103-07-x-D, VST104_footprints:TSW-103-07-x-D, F.Cu at (86.5, 97.5)
- added J5: TSW-103-07-x-D, VST104_footprints:TSW-103-07-x-D, F.Cu at (69.0, 97.5)
- added Module 2: PC104_module, VST104_footprints:PC104_footprint, F.Cu at (31.1, 324.7)
- added Q10: SQD40061EL, VST104_footprints:TO-252AA_6.5x6.1mm, F.Cu at (127.0, 81.4)
- added R28: 100k, VST104_footprints:R_SMD_0805, F.Cu at (132.5, 77.8)
- added TP13: TestPoint_Alt, VST104_footprints:scope_PAD_2mm, F.Cu at (45.5, 94.2)
- added TP2: TestPoint, VST104_footprints:scope_PAD_1mm, F.Cu at (164.2, 72.8)
- F7: renamed from 2A1; value Fuse -> 2A1
- J6: value TSW-102-07-T-D -> TSW-103-07-x-D; footprint VST104_footprints:TSW-102-07-x-D -> VST104_footprints:TSW-103-07-x-D
- J7, J8: value TSW-102-07-T-D -> Conn_01x45; footprint VST104_footprints:TSW-102-07-x-D -> VST104_footprints:conn_FPC_45x0.5_505110-4591
- Module 1: renamed from Module_2
- Module 3: renamed from Module_4
- Module 4: renamed from Module_1
- P1: value Val** -> CX90M-16P
- TP1: renamed from TP2; footprint VST104_footprints:scope_PAD -> VST104_footprints:scope_PAD_1mm
- TP10: renamed from TP11; footprint VST104_footprints:scope_PAD -> VST104_footprints:scope_PAD_2mm
- TP11: renamed from TP12; footprint VST104_footprints:scope_PAD -> VST104_footprints:scope_PAD_2mm
- TP12: renamed from TP13; footprint VST104_footprints:scope_PAD -> VST104_footprints:scope_PAD_2mm
- TP3: footprint VST104_footprints:scope_PAD -> VST104_footprints:scope_PAD_1mm
- TP8: renamed from TP9; footprint VST104_footprints:scope_PAD -> VST104_footprints:scope_PAD_2mm
- TP9: renamed from TP10; footprint VST104_footprints:scope_PAD -> VST104_footprints:scope_PAD_2mm
- U4, U5: value Val** -> OKL-T6-W12
- moved J8 262.3 mm to (212.0, 305.0), turned to 90 degrees
- moved J7 224.8 mm to (212.0, 271.0), turned to 90 degrees
- moved J6 35.0 mm to (51.5, 97.5), turned to 180 degrees
- moved Q8 19.8 mm to (136.8, 73.2), turned to 180 degrees
- moved R27 17.3 mm to (132.5, 75.5), turned to 0 degrees
- moved R29 16.2 mm to (60.5, 74.2), turned to 90 degrees
- moved C17 15.2 mm to (85.5, 78.0), turned to 90 degrees
- moved C18 14.2 mm to (60.5, 78.0), turned to 90 degrees
- moved F5 13.2 mm to (105.5, 76.5)
- moved F6 13.2 mm to (105.5, 67.5)
- moved R33 13.0 mm to (67.5, 72.2), turned to 270 degrees
- moved R34 12.3 mm to (42.5, 72.2), turned to 270 degrees
- moved U7 10.2 mm to (172.0, 75.0), turned to 0 degrees
- moved Q9 10.0 mm to (119.8, 81.4), turned to 0 degrees
- moved U4 8.54 mm to (76.5, 76.5), turned to 180 degrees
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- renumbered D12 to D11, D11 to D12, F6 to F5, F5 to F6, J3 to J1, J4 to J2, J5 to J3, Q10 to Q9, R19 to R16, R16 to R17, R17 to R18, R18 to R19, R28 to R27, TP5 to TP4, TP6 to TP5, TP7 to TP6, TP8 to TP7
Connections:
- F5 pad 1: Net-(C22-Pad1) -> Net-(C18-Pad1)
- F6 pad 1: Net-(C18-Pad1) -> Net-(C22-Pad1)
- J6 pad 2: Net-(J6-Pad1) -> /SUP_5V
- J6 pad 3: /SUP_UNREG -> Net-(J6-Pad1)
- J6 pad 4: /SUP_UNREG -> /SUP_5V
- J7 pad 1: Net-(J7-Pad1) -> /H1-24
- J7 pad 2: Net-(J7-Pad1) -> /H2-24
- J7 pad 3: /SUP_3V3 -> /H1-23
- J7 pad 4: /SUP_3V3 -> /H1-26
- J8 pad 1: Net-(J8-Pad1) -> /H2-1
- J8 pad 2: Net-(J8-Pad1) -> /H1-2
- J8 pad 3: /SUP_5V -> /H2-2
- J8 pad 4: /SUP_5V -> /H1-1
- Module 1 pad H2_31: GNDA -> GND
- Module 3 pad H2_31: GNDA -> GND
- Module 4 pad H2_31: GNDA -> GND
- P1 pad MH: Net-(P1-PadMH) -> GND
- Q9 pad 1: Net-(Q10-Pad1) -> Net-(Q8-Pad1)
- R27 pad 2: Net-(Q10-Pad1) -> Net-(Q8-Pad1)
- R35 pad 1: Net-(J6-Pad1) -> Net-(J4-Pad1)
- R36 pad 1: Net-(J7-Pad1) -> Net-(J5-Pad1)
- R37 pad 1: Net-(J8-Pad1) -> Net-(J6-Pad1)
- SW1 pad 1: (no net) -> Net-(D13-Pad3)
- SW1 pad 10: Net-(Q8-Pad1) -> Net-(R24-Pad2)
- SW1 pad 12: /PDO2 -> (no net)
- SW1 pad 13: (no net) -> /PDO2
- SW1 pad 14: (no net) -> Net-(Q8-Pad1)
- SW1 pad 16: (no net) -> GND
- SW1 pad 4: Net-(D13-Pad3) -> (no net)
- SW1 pad 5: Net-(Q6-Pad3) -> (no net)
- SW1 pad 6: Net-(R24-Pad2) -> (no net)
- SW1 pad 9: GND -> Net-(Q6-Pad3)
- TP11 pad 1: Net-(J6-Pad1) -> Net-(J4-Pad1)
- TP12 pad 1: Net-(J7-Pad1) -> Net-(J5-Pad1)
- TP3 pad 1: /CC1 -> /CC2
Routing:
- net /H2-2: track 0.00 -> 513.3 mm, vias 0 -> 4
- net /H2-1: track 0.00 -> 512.3 mm, vias 0 -> 3
- net /H2-4: track 0.00 -> 505.9 mm, vias 0 -> 4
- net /H1-2: track 0.00 -> 505.2 mm, vias 0 -> 2
- net /H2-3: track 0.00 -> 503.4 mm, vias 0 -> 2
- net /H2-6: track 0.00 -> 498.5 mm, vias 0 -> 4
- net /H1-4: track 0.00 -> 497.8 mm, vias 0 -> 2
- net /H2-5: track 0.00 -> 496.0 mm, vias 0 -> 2
- net /H1-1: track 0.00 -> 495.0 mm, vias 0 -> 2
- net /H2-8: track 0.00 -> 491.6 mm, vias 0 -> 4
- net /H1-6: track 0.00 -> 490.4 mm, vias 0 -> 2
- net /H2-7: track 0.00 -> 488.6 mm, vias 0 -> 2
- net /H1-3: track 0.00 -> 487.6 mm, vias 0 -> 2
- net /H1-8: track 0.00 -> 484.0 mm, vias 0 -> 2
- net /H2-10: track 0.00 -> 483.7 mm, vias 0 -> 4
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- added copper zone on B.Cu, net /SUP_3V3
- added copper zone on F.Cu, net /SUP_3V3
- added copper zone on In1.Cu, net /SUP_3V3
- added copper zone on B.Cu, net /SUP_5V
- added copper zone on F.Cu, net /SUP_5V
- added copper zone on In1.Cu, net /SUP_5V
- added copper zone on B.Cu, net /SUP_UNREG
- added copper zone on F.Cu, net /SUP_UNREG
- added copper zone on In1.Cu, net /SUP_UNREG
- added copper zone on In1.Cu, net /VSINK
- added copper zone on In1.Cu, net GND
- added copper zone on F.Cu, net Net-(C17-Pad1)
- added copper zone on In1.Cu, net Net-(C17-Pad1)
- added copper zone on F.Cu, net Net-(C18-Pad1)
- added copper zone on In1.Cu, net Net-(C18-Pad1)
- added copper zone on F.Cu, net Net-(C20-Pad1)
- added copper zone on In1.Cu, net Net-(C20-Pad1)
- added copper zone on F.Cu, net Net-(C21-Pad1)
- added copper zone on In1.Cu, net Net-(C21-Pad1)
- added copper zone on F.Cu, net Net-(C22-Pad1)
- added copper zone on In1.Cu, net Net-(C22-Pad1)
- added copper zone on F.Cu, net Net-(F5-Pad2)
- added copper zone on In1.Cu, net Net-(F5-Pad2)
- added copper zone on F.Cu, net Net-(F6-Pad2)
- added copper zone on In1.Cu, net Net-(F6-Pad2)
- added copper zone on F.Cu, net Net-(J4-Pad1)
- added copper zone on In1.Cu, net Net-(J4-Pad1)
- added copper zone on F.Cu, net Net-(J5-Pad1)
- added copper zone on In1.Cu, net Net-(J5-Pad1)
- added copper zone on F.Cu, net Net-(J6-Pad1)
- added copper zone on In1.Cu, net Net-(J6-Pad1)
Other:
- board size 202.5 x 280 mm -> 202.5 x 315 mm
- rule trace_min: 0 -> 0.127
- board text added: "3.3V 6A"
- board text added: "3V3 DCDC"
- board text added: "5V"
- board text added: "5V 6A"
- board text added: "5V DCDC"
- board text added: "5V direct"
- board text added: "7-14V"
- board text added: "8-12V"
- board text added: "ALT"
- board text added: "D+"
- board text added: "D-"
- board text added: "EXT."
- board text added: "EXT. input"
- board text added: "GN"
- board text added: "GND"
- board text added: "GROUND"
- board text added: "SCL"
- board text added: "SDA"
- board text added: "UNREG dir."
- board text added: "UNREG. 6A"
- board text added: "USB vbus"
- board text added: "USBC"
- board text added: "VDD"
- board text added: "VST104-Foxtrot"
- board text added: "max 6A"
- board text added: "max 8A"
- board text added: "v1.0"

Commit message: CUBEmx updated
Parts:
- added G***: LOGO, VST104_logos:OSH_logo_9mm, F.Cu at (212.0, 110.0)
