File: element_foxtrot/element_foxtrot.kicad_pcb (KiCad board)
At the start: 4 copper layers, 202.5 x 315 mm, 150 parts, among them J1 Ext_Power, J2 Program, J3 USB, J4 TSW-103-07-x-D, J5 TSW-103-07-x-D, J6 TSW-103-07-x-D, J7 Conn_01x45, J8 Conn_01x45, P1 CX90M-16P, Q1 2N7002BK, Q10 SQD40061EL, Q2 SQD40061EL, Q3 SQD40061EL, Q4 SQD40061EL, Q5 SQD40061EL, Q6 2N7002BK, Q7 SQD40061EL, Q8 2N7002BK, Q9 SQD40061EL, SW1 switch_3P3T, U1 L7985, U2 TL432AIDBZR, U3 STUSB4500QTR, U4 OKL-T6-W12, U5 OKL-T6-W12, U6 USBLC6-4, U7 USBLC6-2

Commit message: small updates
Parts:
- removed G*** (x2): LOGO, VST104_logos:OSH_logo_9mm
- removed G***: LOGO, VST104_logos:VST_logo_vertical_12.5mm
- removed G***: LOGO, VST104_logos:VST_logo_vertical_174.5mm
- removed H16, H17, H18: MountingHole_Pad, VST104_footprints:MountingHole_3.2mm_M3_Pad_Via
- removed Module 1: PC104_module, VST104_footprints:PC104_footprint
- removed Module 2: PC104_module, VST104_footprints:PC104_footprint
- removed Module 3: PC104_module, VST104_footprints:PC104_footprint
- removed Module 4: PC104_module, VST104_footprints:PC104_footprint
- removed R37: 0, VST104_footprints:R_SMD_1206
- removed U3: STUSB4500QTR, VST104_footprints:QFN-24_4.0x4.0mm_EP
- removed U4: OKL-T6-W12, VST104_footprints:OKL-T6-W12
- added DC/DC1: OKL-T6-W12, VST104_footprints:OKL-T6-W12, F.Cu at (76.5, 51.5)
- added DC/DC2: OKL-T6-W12, VST104_footprints:OKL-T6-W12, F.Cu at (51.5, 51.5)
- added LD1: AL5809, VST104_footprints:Power-DI-123_2.8x1.8x1mm, F.Cu at (154.5, 47.2)
- added LD2: AL5809, VST104_footprints:Power-DI-123_2.8x1.8x1mm, F.Cu at (198.5, 56.8)
- added LD3: AL5809, VST104_footprints:Power-DI-123_2.8x1.8x1mm, F.Cu at (133.0, 48.2)
- added Module_1: PC104_module, VST104_footprints:PC104_footprint, F.Cu at (131.3, 193.8)
- added Module_2: PC104_module, VST104_footprints:PC104_footprint, F.Cu at (31.1, 193.8)
- added Module_3: PC104_module, VST104_footprints:PC104_footprint, F.Cu at (31.1, 299.7)
- added Module_4: PC104_module, VST104_footprints:PC104_footprint, F.Cu at (131.3, 299.7)
- C1: value 10u -> 100p
- C10: value 2n2 -> 22u
- C11: value 1n -> 22u
- C12, C13, C14: value 1u -> 10u
- C15: value 470u -> 1u; footprint VST104_footprints:CP_Radial_D8.0mm_P3.50mm_L11.5mm -> VST104_footprints:C_SMD_0805
- C16: value 470u -> 10u; footprint VST104_footprints:CP_Radial_D8.0mm_P3.50mm_L11.5mm -> VST104_footprints:C_SMD_0805
- C17: value 22u -> 220n
- C18: value 22u -> 22n
- C19: value 1u -> 1n
- C2: value 220n -> 1u
- C21: value 10u -> 220u; footprint VST104_footprints:C_SMD_0805 -> VST104_footprints:CP_Radial_D6.3mm_P2.50mm_L11.2mm
- C22: value 10u -> 2n2
- C3: value 100p -> 4u7
- C4: value 22n -> 1n
- C5: value 1n -> 1u
- C7: value 4u7 -> 1u
- C8: value 10u -> 470u; footprint VST104_footprints:C_SMD_0805 -> VST104_footprints:CP_Radial_D8.0mm_P3.50mm_L11.5mm
- C9: value 220u -> 470u; footprint VST104_footprints:CP_Radial_D6.3mm_P2.50mm_L11.2mm -> VST104_footprints:CP_Radial_D8.0mm_P3.50mm_L11.5mm
- D1: value LED -> SMAJ15CA; footprint VST104_footprints:D_SMD_0805_LED -> VST104_footprints:D_SMA_DO-214AC_4.3x2.6mm
- D10: value LED -> DDZ15CSF; footprint VST104_footprints:D_SMD_0805_LED -> VST104_footprints:D_SOD-323-F_1.25x1.7mm
- D11, D9: value LED -> BAV199; footprint VST104_footprints:D_SMD_0805_LED -> VST104_footprints:SOT-23-3_2.9x1.3mm
- D12: value DDZ15CSF -> green; footprint VST104_footprints:D_SOD-323-F_1.25x1.7mm -> VST104_footprints:D_SMD_0805_LED
- D13: value BAV199 -> FM4004W; footprint VST104_footprints:SOT-23-3_2.9x1.3mm -> VST104_footprints:D_SMA_DO-214AC_4.3x2.6mm
- D14: value DDZ15CSF -> yellow; footprint VST104_footprints:D_SOD-323-F_1.25x1.7mm -> VST104_footprints:D_SMD_0805_LED
- D15: value BAV199 -> blue; footprint VST104_footprints:SOT-23-3_2.9x1.3mm -> VST104_footprints:D_SMD_0805_LED
- D16: value LED -> STPS3L60UFN; footprint VST104_footprints:D_SMD_0805_LED -> VST104_footprints:D_SMB-FN_DO-214AA-FN
- D17: value FM4004W -> green; footprint VST104_footprints:D_SMA_DO-214AC_4.3x2.6mm -> VST104_footprints:D_SMD_0805_LED
- D3: value LED -> ESDA25W5; footprint VST104_footprints:D_SMD_0805_LED -> VST104_footprints:SOT-323-5L_2.0x1.25mm
- D4: value STPS3L60UFN -> BAT54JFILM; footprint VST104_footprints:D_SMB-FN_DO-214AA-FN -> VST104_footprints:D_SOD-323_1.65x1.28mm
- D5: value SMAJ15CA -> DDZ15CSF; footprint VST104_footprints:D_SMA_DO-214AC_4.3x2.6mm -> VST104_footprints:D_SOD-323-F_1.25x1.7mm
- D6: value ESDA25W5 -> red; footprint VST104_footprints:SOT-323-5L_2.0x1.25mm -> VST104_footprints:D_SMD_0805_LED
- D7: value BAT54JFILM -> red; footprint VST104_footprints:D_SOD-323_1.65x1.28mm -> VST104_footprints:D_SMD_0805_LED
- J2: value Program -> TSW-103-07-x-D; footprint VST104_footprints:TSW-105-07-x-S -> VST104_footprints:TSW-103-07-x-D
- J3: value USB -> TSW-103-07-x-D; footprint VST104_footprints:TSW-104-07-x-S -> VST104_footprints:TSW-103-07-x-D
- J5: value TSW-103-07-x-D -> Program; footprint VST104_footprints:TSW-103-07-x-D -> VST104_footprints:TSW-105-07-x-S
- J6: value TSW-103-07-x-D -> Conn_01x45; footprint VST104_footprints:TSW-103-07-x-D -> VST104_footprints:conn_FPC_45x0.5_505110-4591
- J7: value Conn_01x45 -> USB; footprint VST104_footprints:conn_FPC_45x0.5_505110-4591 -> VST104_footprints:TSW-104-07-x-S
- Q1, Q6, Q8: value 2N7002BK -> SQD40061EL; footprint VST104_footprints:SOT-23-3_2.9x1.3mm -> VST104_footprints:TO-252AA_6.5x6.1mm
- Q10, Q5, Q7: value SQD40061EL -> 2N7002BK; footprint VST104_footprints:TO-252AA_6.5x6.1mm -> VST104_footprints:SOT-23-3_2.9x1.3mm
- R1: value 250 -> 1k
- R10, R29: value 100 -> 100k
- R11: value 1k2 -> 22k
- R12, R16: value 1k2 -> 100k
- R13: value 47k -> 22k
- R14: value 5k23 -> 1k
- R15: value 5k1 -> 100k
- R17: value 698 -> 100
- R18: value 100k -> 1k05
- R19: value 20k -> 1k65
- R2: value 100k -> 470
- R20: value 100k -> 1k69
- R21, R23: value 100k -> 0; footprint VST104_footprints:R_SMD_0805 -> VST104_footprints:R_SMD_1206
- R22: value 22k -> 0; footprint VST104_footprints:R_SMD_0805 -> VST104_footprints:R_SMD_1206
- R24: value 22k -> 10k
- R25: value 1k -> 10k
- R26: value 1k2 -> 10k
- R27: value 100k -> 150
- R30, R32: value 10k -> 100
- R31: value 10k -> 1k
- R33: value 2k18 -> 5k1
- R34: value 1k34 -> 1k2
- R35: value 0 -> 698; footprint VST104_footprints:R_SMD_1206 -> VST104_footprints:R_SMD_0805
- R36: value 0 -> 1k13; footprint VST104_footprints:R_SMD_1206 -> VST104_footprints:R_SMD_0805
- R4: value 250 -> 10k
- R5: value 1k -> 47k
- R6: value 470 -> 5k23
- R7: value 1k -> 100k
- R8: value 100k -> 20k
- R9: value 10k -> 100k
- TP10, TP11, TP12, TP9: footprint VST104_footprints:scope_PAD_2mm -> VST104_footprints:KSE_PN6095
- TP13: value TestPoint_Alt -> TestPoint; footprint VST104_footprints:scope_PAD_2mm -> VST104_footprints:scope_PAD_1mm
- TP3: value TestPoint -> TestPoint_Alt; footprint VST104_footprints:scope_PAD_1mm -> VST104_footprints:scope_PAD_2mm
- TP4, TP5, TP6, TP7: footprint VST104_footprints:KSE_PN6095 -> VST104_footprints:scope_PAD_2mm
- U1: value L7985 -> TL432AIDBZR; footprint VST104_footprints:HSOP8_3.9x4.9mm_EP -> VST104_footprints:SOT-23-3_2.9x1.3mm
- U2: value TL432AIDBZR -> STUSB4500QTR; footprint VST104_footprints:SOT-23-3_2.9x1.3mm -> VST104_footprints:QFN-24_4.0x4.0mm_EP
- U5: value OKL-T6-W12 -> USBLC6-4; footprint VST104_footprints:OKL-T6-W12 -> VST104_footprints:SOT-23-6L_2.9x1.6mm
- U7: value USBLC6-2 -> L7985; footprint VST104_footprints:SOT-23-6L_2.9x1.6mm -> VST104_footprints:HSOP8_3.9x4.9mm_EP
- moved J7 228.6 mm to (172.8, 45.8), turned to 180 degrees
- moved J6 218.7 mm to (212.0, 246.0), turned to 90 degrees
- moved H13 192.5 mm to (30.0, 335.0), turned to 0 degrees
- moved H15 192.5 mm to (222.5, 335.0), turned to 0 degrees
- moved R34 169.8 mm to (211.5, 56.2), turned to 90 degrees
- moved C22 164.1 mm to (208.2, 56.2)
- moved C21 159.4 mm to (221.5, 58.5), turned to 0 degrees
- moved D17 158.0 mm to (208.2, 54.0), turned to 0 degrees
- moved R19 151.0 mm to (42.5, 45.6), turned to 270 degrees
- moved R17 147.6 mm to (60.5, 49.2), turned to 90 degrees
- moved C18 146.8 mm to (206.8, 65.8)
- moved R20 142.3 mm to (42.5, 49.0), turned to 270 degrees
- moved R33 141.4 mm to (208.2, 58.5), turned to 0 degrees
- moved TP13 137.7 mm to (178.7, 59.5)
- moved C20 137.5 mm to (216.0, 56.2), turned to 90 degrees
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Connections:
- C1 pad 1: /VSINK -> GND
- C1 pad 2: GND -> Net-(C1-Pad2)
- C10 pad 2: Net-(C10-Pad2) -> GND
- C12 pad 1: GND -> /VOUT_UNREG
- C12 pad 2: Net-(C12-Pad2) -> GND
- C13 pad 1: GND -> /VOUT_3V3
- C13 pad 2: Net-(C13-Pad2) -> GND
- C14 pad 1: GND -> /VOUT_5V
- C14 pad 2: Net-(C14-Pad2) -> GND
- C15 pad 1: /VSINK -> VDD
- C17 pad 1: Net-(C17-Pad1) -> /VSINK
- C18 pad 2: GND -> Net-(C18-Pad2)
- C19 pad 1: VDD -> Net-(C18-Pad1)
- C19 pad 2: GND -> Net-(C19-Pad2)
- C2 pad 1: /VSINK -> GND
- C2 pad 2: GND -> Net-(C2-Pad2)
- C21 pad 1: Net-(C21-Pad1) -> Net-(C20-Pad1)
- C22 pad 1: Net-(C22-Pad1) -> Net-(C20-Pad1)
- C22 pad 2: GND -> Net-(C22-Pad2)
- C3 pad 2: Net-(C3-Pad2) -> VBUS
- C4 pad 2: Net-(C4-Pad2) -> GND
- C5 pad 1: Net-(C4-Pad1) -> GND
- C7 pad 2: VBUS -> Net-(C7-Pad2)
- C8 pad 1: Net-(C10-Pad1) -> /VSINK
- C9 pad 1: Net-(C10-Pad1) -> /VSINK
- D1 pad 1: /GPIO -> GND
- D1 pad 2: Net-(D1-Pad2) -> Net-(C1-Pad2)
- D10 pad 1: GND -> Net-(D10-Pad1)
- D11 pad 2: Net-(D11-Pad2) -> Net-(C5-Pad2)
- D12 pad 1: Net-(C12-Pad2) -> GND
- D13 pad 1: GND -> Net-(C11-Pad1)
- D13 pad 2: Net-(C12-Pad2) -> /VOUT_5V
- D14 pad 1: Net-(D14-Pad1) -> /GPIO
- D15 pad 1: GND -> Net-(D15-Pad1)
- D15 pad 2: Net-(C12-Pad2) -> Net-(D15-Pad2)
- D16 pad 1: GND -> Net-(D16-Pad1)
- D16 pad 2: Net-(D16-Pad2) -> GND
- D17 pad 1: Net-(C18-Pad1) -> GND
- D17 pad 2: Net-(C22-Pad1) -> Net-(D17-Pad2)
- D2 pad 2: Net-(C3-Pad2) -> VBUS
- D3 pad 1: Net-(D3-Pad1) -> /CC2
- D3 pad 2: Net-(D3-Pad2) -> GND
- D4 pad 1: Net-(D4-Pad1) -> Net-(C2-Pad2)
- D4 pad 2: GND -> VBUS
- D5 pad 1: GND -> Net-(D5-Pad1)
- D5 pad 2: VBUS -> Net-(D5-Pad2)
- D6 pad 1: /CC2 -> GND
- D6 pad 2: GND -> Net-(D6-Pad2)
- D7 pad 1: Net-(C6-Pad2) -> GND
- D7 pad 2: VBUS -> Net-(D7-Pad2)
- D8 pad 1: Net-(D8-Pad1) -> Net-(C5-Pad2)
- D9 pad 2: Net-(D9-Pad2) -> Net-(C5-Pad2)
- F1 pad 1: Net-(C3-Pad2) -> Net-(C1-Pad2)
- F3 pad 1: Net-(C20-Pad1) -> /VOUT_UNREG
- F4 pad 1: Net-(C17-Pad1) -> Net-(C10-Pad1)
- F5 pad 1: Net-(C18-Pad1) -> Net-(C11-Pad1)
- F6 pad 1: Net-(C22-Pad1) -> /VOUT_5V
- F7 pad 2: Net-(C10-Pad1) -> Net-(C20-Pad1)
- J2 pad 1: VDD -> Net-(J2-Pad1)
- J2 pad 2: /SDA -> /SUP_UNREG
- J2 pad 3: /SCL -> Net-(J2-Pad1)
- J2 pad 4: /ALTER -> /SUP_UNREG
- J2 pad 5: GND -> Net-(J2-Pad1)
- J3 pad 1: +5V -> Net-(J3-Pad1)
- J3 pad 2: /USB_P -> /SUP_3V3
- J3 pad 3: /USB_N -> Net-(J3-Pad1)
- J3 pad 4: GND -> /SUP_3V3
- J4 pad 2: /SUP_UNREG -> /SUP_5V
- J4 pad 4: /SUP_UNREG -> /SUP_5V
- J4 pad 6: /SUP_UNREG -> /SUP_5V
- J5 pad 1: Net-(J5-Pad1) -> VDD
- J5 pad 2: /SUP_3V3 -> /SDA
- J5 pad 3: Net-(J5-Pad1) -> /SCL
- J5 pad 4: /SUP_3V3 -> /ALTER
- J5 pad 5: Net-(J5-Pad1) -> GND
- J6 pad 1: Net-(J6-Pad1) -> /H1-24
- J6 pad 2: /SUP_5V -> /H2-24
- J6 pad 3: Net-(J6-Pad1) -> /H1-23
- J6 pad 4: /SUP_5V -> /H1-26
- J6 pad 5: Net-(J6-Pad1) -> /H1-25
- J6 pad 6: /SUP_5V -> /H1-28
- J7 pad 1: /H1-24 -> +5V
- J7 pad 2: /H2-24 -> /USB_P
- J7 pad 3: /H1-23 -> /USB_N
- J7 pad 4: /H1-26 -> GND
- L1 pad 1: Net-(D4-Pad1) -> Net-(D16-Pad1)
- L1 pad 2: Net-(C10-Pad1) -> Net-(C20-Pad1)
- Q1 pad 1: Net-(Q1-Pad1) -> Net-(D5-Pad2)
- Q1 pad 2: GND -> Net-(D5-Pad1)
- Q1 pad 3: Net-(D3-Pad1) -> Net-(C1-Pad2)
- Q10 pad 2: /VSINK -> GND
- Q10 pad 3: Net-(F6-Pad2) -> Net-(D15-Pad1)
- Q2 pad 2: Net-(D8-Pad1) -> Net-(C5-Pad2)
- Q2 pad 3: Net-(C3-Pad2) -> VBUS
- Q3 pad 1: Net-(D12-Pad2) -> Net-(D10-Pad2)
- Q3 pad 2: Net-(C12-Pad2) -> Net-(D10-Pad1)
- Q3 pad 3: VBUS -> Net-(D5-Pad1)
- Q4 pad 1: Net-(D14-Pad2) -> Net-(D8-Pad2)
- Q4 pad 2: Net-(D14-Pad1) -> Net-(C5-Pad2)
- Q4 pad 3: Net-(D8-Pad1) -> /VSINK
- Q5 pad 1: Net-(D12-Pad2) -> Net-(Q5-Pad1)
- Q5 pad 2: Net-(C12-Pad2) -> GND
- Q5 pad 3: /VSINK -> Net-(Q5-Pad3)
- Q6 pad 1: Net-(Q6-Pad1) -> Net-(D10-Pad2)
- Q6 pad 2: GND -> Net-(D10-Pad1)
- Q6 pad 3: Net-(Q6-Pad3) -> /VSINK
- Q7 pad 1: Net-(D14-Pad2) -> Net-(Q7-Pad1)
- Q7 pad 2: Net-(D14-Pad1) -> GND
- Q7 pad 3: /VSINK -> Net-(Q7-Pad3)
- Q8 pad 1: Net-(Q8-Pad1) -> Net-(Q7-Pad1)
- Q8 pad 2: GND -> /VSINK
- Q8 pad 3: Net-(Q10-Pad1) -> Net-(F5-Pad2)
- Q9 pad 1: Net-(Q8-Pad1) -> Net-(Q7-Pad3)
- Q9 pad 3: Net-(F5-Pad2) -> Net-(F6-Pad2)
- R1 pad 1: +5V -> Net-(C2-Pad2)
- R1 pad 2: Net-(D1-Pad2) -> Net-(R1-Pad2)
- R10 pad 1: Net-(C5-Pad2) -> Net-(Q5-Pad1)
- R10 pad 2: Net-(C10-Pad2) -> GND
- R11 pad 1: VBUS -> Net-(D8-Pad2)
- R11 pad 2: Net-(D9-Pad2) -> Net-(R11-Pad2)
- R12 pad 1: Net-(D8-Pad1) -> Net-(D10-Pad1)
- R13 pad 1: Net-(D8-Pad1) -> Net-(D10-Pad2)
- R13 pad 2: Net-(C11-Pad1) -> Net-(R13-Pad2)
- R14 pad 1: Net-(C11-Pad1) -> Net-(R14-Pad1)
- R14 pad 2: GND -> /VSINK
- R15 pad 1: Net-(C5-Pad2) -> /VSINK
- R15 pad 2: Net-(C10-Pad1) -> Net-(Q7-Pad1)
- R16 pad 1: Net-(C10-Pad1) -> /VSINK
- R16 pad 2: Net-(D11-Pad2) -> Net-(Q7-Pad3)
- R17 pad 1: GND -> Net-(DC/DC2-Pad1)
- R17 pad 2: Net-(C5-Pad2) -> Net-(Q7-Pad3)
- R18 pad 1: Net-(C12-Pad2) -> Net-(DC/DC1-Pad6)
- R18 pad 2: Net-(D12-Pad2) -> Net-(R18-Pad2)
- R19 pad 1: Net-(D8-Pad1) -> Net-(DC/DC2-Pad6)
- R2 pad 1: Net-(Q1-Pad1) -> VBUS
- R2 pad 2: /PDO2 -> Net-(C2-Pad2)
- R20 pad 2: Net-(Q6-Pad1) -> GND
- R21 pad 1: Net-(Q6-Pad1) -> Net-(J2-Pad1)
- R21 pad 2: GND -> /VOUT_UNREG
- R22 pad 1: Net-(D12-Pad2) -> Net-(J3-Pad1)
- R22 pad 2: Net-(R22-Pad2) -> /VOUT_3V3
- R23 pad 1: Net-(D14-Pad1) -> Net-(J4-Pad1)
- R23 pad 2: Net-(D14-Pad2) -> /VOUT_5V
- R24 pad 1: Net-(D14-Pad2) -> VDD
- R24 pad 2: Net-(R24-Pad2) -> /ALTER
- R25 pad 1: Net-(R25-Pad1) -> VDD
- R25 pad 2: /VSINK -> /SCL
- R26 pad 1: /VSINK -> VDD
- R26 pad 2: Net-(D16-Pad2) -> /SDA
- R27 pad 1: /VSINK -> +5V
- R27 pad 2: Net-(Q8-Pad1) -> Net-(D14-Pad2)
- R28 pad 1: /VSINK -> Net-(Q10-Pad1)
- R28 pad 2: Net-(Q10-Pad1) -> /PDO2
- R29 pad 1: Net-(R29-Pad1) -> Net-(Q10-Pad1)
- R29 pad 2: Net-(Q10-Pad1) -> GND
- R3 pad 1: Net-(Q1-Pad1) -> GND
- R3 pad 2: GND -> /RST
- R30 pad 1: VDD -> +5V
- R30 pad 2: /ALTER -> Net-(D15-Pad2)
- R31 pad 1: VDD -> Net-(C19-Pad2)
- R31 pad 2: /SCL -> Net-(C18-Pad2)
- R32 pad 1: VDD -> Net-(C19-Pad2)
- R32 pad 2: /SDA -> Net-(C22-Pad2)
- R33 pad 1: Net-(R33-Pad1) -> Net-(C19-Pad2)
- R33 pad 2: GND -> Net-(C20-Pad1)
- R34 pad 1: Net-(R34-Pad1) -> Net-(C20-Pad1)
- R34 pad 2: GND -> Net-(D17-Pad2)
- R35 pad 1: Net-(J4-Pad1) -> GND
- R35 pad 2: Net-(C20-Pad1) -> Net-(C19-Pad2)
- R36 pad 1: Net-(J5-Pad1) -> Net-(R18-Pad2)
- R36 pad 2: Net-(C21-Pad1) -> GND
- R4 pad 1: +5V -> Net-(D5-Pad2)
- R4 pad 2: Net-(D3-Pad2) -> GND
- R5 pad 1: Net-(C6-Pad2) -> Net-(D5-Pad1)
- R5 pad 2: Net-(R5-Pad2) -> Net-(C4-Pad1)
- R6 pad 1: VBUS -> Net-(C4-Pad1)
- R6 pad 2: Net-(C6-Pad2) -> GND
- R7 pad 2: Net-(C4-Pad2) -> Net-(D8-Pad2)
- R8 pad 1: GND -> Net-(D5-Pad1)
- R8 pad 2: /RST -> Net-(R8-Pad2)
- R9 pad 1: Net-(D8-Pad2) -> Net-(R8-Pad2)
- R9 pad 2: GND -> Net-(Q5-Pad1)
- SW1 pad 1: Net-(D13-Pad3) -> Net-(D9-Pad3)
- SW1 pad 10: Net-(R24-Pad2) -> Net-(R13-Pad2)
- SW1 pad 14: Net-(Q8-Pad1) -> Net-(Q7-Pad1)
- SW1 pad 2: Net-(R22-Pad2) -> Net-(R11-Pad2)
- SW1 pad 9: Net-(Q6-Pad3) -> Net-(Q5-Pad3)
- TP1 pad 1: /PDO2 -> /CC1
- TP10 pad 1: Net-(C22-Pad1) -> /SUP_5V
- TP11 pad 1: Net-(J4-Pad1) -> /SUP_3V3
- TP12 pad 1: Net-(J5-Pad1) -> GND
- TP13 pad 1: Net-(J6-Pad1) -> /PDO2
- TP2 pad 1: /CC1 -> /CC2
- TP3 pad 1: /CC2 -> /VOUT_UNREG
- TP4 pad 1: /SUP_UNREG -> /VOUT_3V3
- TP5 pad 1: /SUP_5V -> /VOUT_5V
- TP6 pad 1: /SUP_3V3 -> Net-(J2-Pad1)
- TP7 pad 1: GND -> Net-(J3-Pad1)
- TP8 pad 1: Net-(C20-Pad1) -> Net-(J4-Pad1)
- TP9 pad 1: Net-(C21-Pad1) -> /SUP_UNREG
- U1 pad 1: Net-(D4-Pad1) -> Net-(C4-Pad1)
- U1 pad 2: (no net) -> Net-(R8-Pad2)
- U1 pad 3: /VSINK -> GND
- U2 pad 1: Net-(C11-Pad1) -> /CC1
- U2 pad 2: Net-(R19-Pad2) -> /CC1
- U2 pad 3: GND -> (no net)
- U5 pad 1: Net-(R29-Pad1) -> /SDA
- U5 pad 2: Net-(C18-Pad1) -> GND
- U5 pad 3: GND -> /SCL
- U5 pad 4: Net-(C22-Pad1) -> /ALTER
- U5 pad 5: Net-(C22-Pad1) -> VDD
- U5 pad 6: Net-(R34-Pad1) -> (no net)
- U6 pad 1: /SDA -> /USB_N
- U6 pad 3: /SCL -> (no net)
- U6 pad 4: /ALTER -> /USB_P
- U6 pad 5: VDD -> +5V
- U7 pad 1: /USB_N -> Net-(D16-Pad1)
- U7 pad 2: GND -> (no net)
- U7 pad 3: /USB_P -> /VSINK
- U7 pad 4: /USB_P -> Net-(C18-Pad1)
- U7 pad 5: +5V -> Net-(C19-Pad2)
- U7 pad 6: /USB_N -> (no net)
Routing:
- net Net-(Q7-Pad3): track 0.00 -> 91.9 mm, vias 0 -> 3
- net Net-(Q10-Pad1): track 91.6 -> 6.74 mm, vias 3 -> 0
- net Net-(Q8-Pad1): track 78.9 -> 0.00 mm, vias 4 -> 0
- net Net-(Q7-Pad1): track 0.00 -> 78.8 mm, vias 0 -> 4
- net Net-(R22-Pad2): track 50.7 -> 0.00 mm
- net Net-(R11-Pad2): track 0.00 -> 50.7 mm
- net Net-(D9-Pad3): track 0.00 -> 33.7 mm, vias 0 -> 1
- net Net-(D13-Pad3): track 33.7 -> 0.00 mm, vias 1 -> 0
- net Net-(C12-Pad2): track 23.6 -> 0.00 mm, vias 20 -> 0
- net Net-(R24-Pad2): track 21.2 -> 0.00 mm
- net Net-(R13-Pad2): track 0.00 -> 21.2 mm
- net Net-(D10-Pad2): track 2.00 -> 18.3 mm, vias 0 -> 2
- net Net-(D14-Pad2): track 18.3 -> 2.25 mm, vias 2 -> 0
- net Net-(D12-Pad2): track 18.2 -> 2.73 mm, vias 2 -> 0
- net Net-(R1-Pad2): track 0.00 -> 14.4 mm, vias 0 -> 2
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- added copper zone on F.Cu, net /VOUT_3V3
- added copper zone on In1.Cu, net /VOUT_3V3
- added copper zone on F.Cu, net /VOUT_5V
- added copper zone on In1.Cu, net /VOUT_5V
- added copper zone on F.Cu, net /VOUT_UNREG
- added copper zone on In1.Cu, net /VOUT_UNREG
- added copper zone on F.Cu, net Net-(C1-Pad2)
- added copper zone on In1.Cu, net Net-(C1-Pad2)
- added copper zone on In1.Cu, net Net-(C10-Pad1)
- added copper zone on F.Cu, net Net-(C11-Pad1)
- added copper zone on In1.Cu, net Net-(C11-Pad1)
- added copper zone on In1.Cu, net Net-(C5-Pad2)
- added copper zone on F.Cu, net Net-(D10-Pad1)
- added copper zone on In1.Cu, net Net-(D10-Pad1)
- added copper zone on F.Cu, net Net-(D16-Pad1)
- added copper zone on F.Cu, net Net-(D5-Pad1)
- added copper zone on In1.Cu, net Net-(D5-Pad1)
- added copper zone on F.Cu, net Net-(J2-Pad1)
- added copper zone on In1.Cu, net Net-(J2-Pad1)
- added copper zone on F.Cu, net Net-(J3-Pad1)
- added copper zone on In1.Cu, net Net-(J3-Pad1)
- removed copper zone on F.Cu, net Net-(C12-Pad2)
- removed copper zone on In1.Cu, net Net-(C12-Pad2)
- removed copper zone on F.Cu, net Net-(C17-Pad1)
- removed copper zone on In1.Cu, net Net-(C17-Pad1)
- removed copper zone on F.Cu, net Net-(C18-Pad1)
- removed copper zone on In1.Cu, net Net-(C18-Pad1)
- removed copper zone on In1.Cu, net Net-(C20-Pad1)
- removed copper zone on F.Cu, net Net-(C21-Pad1)
- removed copper zone on In1.Cu, net Net-(C21-Pad1)
- removed copper zone on F.Cu, net Net-(C22-Pad1)
- removed copper zone on In1.Cu, net Net-(C22-Pad1)
- removed copper zone on F.Cu, net Net-(C3-Pad2)
- removed copper zone on In1.Cu, net Net-(C3-Pad2)
- removed copper zone on F.Cu, net Net-(D14-Pad1)
- removed copper zone on In1.Cu, net Net-(D14-Pad1)
- removed copper zone on F.Cu, net Net-(D4-Pad1)
- removed copper zone on F.Cu, net Net-(D8-Pad1)
- removed copper zone on In1.Cu, net Net-(D8-Pad1)
- removed copper zone on F.Cu, net Net-(J5-Pad1)
- removed copper zone on In1.Cu, net Net-(J5-Pad1)
- removed copper zone on F.Cu, net Net-(J6-Pad1)
- removed copper zone on In1.Cu, net Net-(J6-Pad1)
Other:
- board size 202.5 x 315 mm -> 202.5 x 307.5 mm

Commit message: ready to manufacture
Parts:
- removed R18: 1k05, VST104_footprints:R_SMD_0805
- removed R19: 1k65, VST104_footprints:R_SMD_0805
- removed R20: 1k69, VST104_footprints:R_SMD_0805
- removed R36: 1k13, VST104_footprints:R_SMD_0805
- added RV1: 3k3, VST104_footprints:trimer_3296W_10.0x9.5x10.0, F.Cu at (66.0, 49.0)
- added RV2: 3k3, VST104_footprints:trimer_3296W_10.0x9.5x10.0, F.Cu at (40.5, 49.0)
- DC/DC1, DC/DC2: value OKL-T6-W12 -> Val**
- J2, J3, J4: value TSW-103-07-x-D -> Val**
- P1: value CX90M-16P -> Val**
- moved C11 0.56 mm to (59.9, 53.0)
- moved DC/DC2 0.56 mm to (50.9, 51.5)
- moved R17 0.56 mm to (59.9, 49.2)
Routing:
- net /SUP_UNREG: track 233.3 -> 131.0 mm, vias 6 -> 16
- net Net-(Q7-Pad3): track 91.9 -> 102.5 mm
- net Net-(Q7-Pad1): track 78.8 -> 68.7 mm
- net /H1-49: track 332.1 -> 337.4 mm
- net /H2-36: track 398.6 -> 401.9 mm
- net Net-(DC/DC1-Pad6): track 8.04 -> 11.2 mm
- net /SUP_5V: track 174.1 -> 170.9 mm, vias 6 -> 16
- net /H1-15: track 444.2 -> 441.2 mm
- net /H1-5: track 480.7 -> 478.2 mm
- net GND: track 68.0 -> 65.5 mm, vias 79 -> 77
- net /H1-7: track 472.9 -> 470.8 mm
- net /H1-9: track 465.5 -> 463.4 mm
- net /H1-19: track 428.5 -> 426.4 mm
- net /H1-1: track 495.0 -> 493.0 mm
- net /H1-11: track 458.1 -> 456.0 mm
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Other:
- rule trace_min: 0.127 -> 0
- board text added: "3.3V 5A"
- board text added: "5V 5A"
- board text added: "UNREG. 5A"
- board text removed: "3.3V 6A"
- board text removed: "5V 6A"
- board text removed: "UNREG. 6A"

Commit message: manufacture order
Parts:
- added G***: LOGO, VST104_logos:VST_logo_vertical_174.5mm, F.Cu at (126.2, 317.5)
- DC/DC1, DC/DC2: value Val** -> OKL-T6-W12
- J2, J3, J4: value Val** -> TSW-103-07-x-D
- P1: value Val** -> CX90M-16P
- SW1: value switch_3P3T -> EG4319A
Connections:
- SW1 pad 1: Net-(D9-Pad3) -> (no net)
- SW1 pad 13: /PDO2 -> GND
- SW1 pad 15: (no net) -> GND
- SW1 pad 16: GND -> /PDO2
- SW1 pad 4: (no net) -> Net-(D9-Pad3)
Routing:
- net Net-(D9-Pad3): track 33.7 -> 26.9 mm
- net /PDO2: track 36.0 -> 41.0 mm, vias 0 -> 1
- net /USB_P: track 30.9 -> 29.1 mm
- net /USB_N: track 25.6 -> 27.1 mm
- net /H1-24: track 419.9 -> 419.0 mm, vias 5 -> 4
- added copper zone on F.Cu, net Net-(C18-Pad1)
- added copper zone on F.Cu, net Net-(C19-Pad2)
- removed copper zone on F.Cu, net Net-(C4-Pad1)
Other:
- rule pad_to_mask_clearance: 0.05 -> 0
