File: element_foxtrot/element_foxtrot.sch (KiCad schematic (older format))
At the start: 127 parts, among them J1 Conn_02x26_Top_Bottom, J2 Conn_02x26_Top_Bottom, J3 Ext_power, J4 USB_C_Receptacle, J5 USB, J6 Program, Q1 SQD40061EL, Q10 2N7002BK, Q2 SQD40061EL, Q3 SQD40061EL, Q4 SQD40061EL, Q5 2N7002BK, Q6 SQD40061EL, Q7 2N7002BK, SW1 switch_3P3T, U1 TL432DBZ, U2 STUSB4500QTR, U3 OKL-T6-W12, U4 OKL-T6-W12, U5 L7985, U7 USBLC6, U8 USBLC6

Commit message: libraries for foxtrot
Parts:
- removed J1, J2: Conn_02x26_Top_Bottom, VST104_footprints:CES-126-01-x-D, symbol Connector_Generic:Conn_02x26_Top_Bottom
- removed J3: Ext_power, symbol Connector:Barrel_Jack
- removed J4: USB_C_Receptacle, symbol Connector:USB_C_Receptacle
- added J5: Ext_Power, VST104_footprints:PJ-063AH, symbol Connector:Barrel_Jack_MountingPin
- added P1: USB_C_Plug, VST104_footprints:CX90M-16P, symbol Connector:USB_C_Plug
- J6: footprint (none) -> VST104_footprints:TSW-105-07-x-S
- J7: renamed from J5; footprint (none) -> VST104_footprints:TSW-104-07-x-S
- SW1: footprint (none) -> VST104_footprints:G-168S-3011
- U1: renamed from U5; footprint (none) -> VST104_footprints:HSOP8_3.9x4.9mm_EP
- U3: renamed from U2; footprint Package_DFN_QFN:QFN-24-1EP_4x4mm_P0.5mm_EP2.7x2.7mm -> VST104_footprints:QFN-24_4.0x4.0mm_EP
- U6: renamed from U7; footprint Package_TO_SOT_SMD:SOT-23-6 -> VST104_footprints:SOT-363_TSSOP-6_2.0x1.25mm
- U7: renamed from U8; footprint Package_TO_SOT_SMD:SOT-666 -> VST104_footprints:SOT-363_TSSOP-6_2.0x1.25mm
- gave numbers to parts that had none: 4
- renumbered C14 to C1, C20 to C10, C3 to C11, C4 to C12, C5 to C13, C6 to C14, C7 to C15, C8 to C16, C9 to C17, C10 to C18, C22 to C19, C15 to C2, C11 to C20, C12 to C21, C13 to C22, C1 to C3, C16 to C4, C17 to C5, C21 to C6, C2 to C7, C18 to C8, C19 to C9, D7 to D10, D8 to D11, D9 to D12, D10 to D13, D11 to D14, D13 to D15, D14 to D16, D12 to D17, D15 to D2, D2 to D3, D3 to D4, D4 to D5, D17 to D6, D5 to D7, D6 to D8, D16 to D9, R8 to R10, R32 to R11, R34 to R12, R9 to R13, R10 to R14, R11 to R15, R12 to R16, R13 to R17, R14 to R18, R15 to R19, R16 to R20, R17 to R21, R26 to R22, R18 to R23, R19 to R24, R27 to R25, R28 to R26, R29 to R27, R20 to R28, R33 to R29, R30 to R3, R35 to R30, R36 to R31, R21 to R32, R22 to R33, R23 to R34, R24 to R35, R25 to R36, R3 to R4, R4 to R5, R31 to R6, R5 to R7, R6 to R8, R7 to R9, TP3 to TP10, TP4 to TP11, TP5 to TP12, TP6 to TP13, TP7 to TP14, TP8 to TP15, TP9 to TP3, TP10 to TP4, TP11 to TP5, TP12 to TP6, TP13 to TP7, TP14 to TP8, TP15 to TP9, U1 to U2, U3 to U4, U4 to U5
Connections:
- wire segments 965 -> 859
Other:
- moved on the sheet: J3, J4

Commit message: ready for wiring
Parts:
- removed C9: 10u, symbol Device:C
- removed D1, D3: ESDA25W, symbol Device:D_Zener_x2_ACom_KKA
- removed D10, D12: 15v, symbol Device:D_Zener
- removed D13: TBAT54S, symbol Device:D_Schottky_x2_Serial_AKC
- removed D17: BAT54JFILM, symbol Device:D_Schottky
- removed D6: ESDA25P35, symbol Device:D_Schottky
- removed D9: ESDA7P120, symbol Device:D_Schottky
- removed P1: USB_C_Plug, VST104_footprints:CX90M-16P, symbol Connector:USB_C_Plug
- removed Q1, Q2, Q3, Q4, Q6, Q8, Q9: SQD40061EL, symbol Device:Q_PMOS_DGS
- removed Q10, Q5, Q7: 2N7002BK, symbol Device:Q_NMOS_DGS
- added 2A1: Fuse, VST104_footprints:R_SMD_0603, symbol Device:Fuse
- added C9: 220u, VST104_footprints:CP_Radial_D6.3mm_P2.50mm_L11.2mm, symbol Device:CP
- added D1, D3: SMAJ15CA, VST104_footprints:D_SMA_DO-214AC_4.3x2.6mm, symbol Device:D_TVS
- added D11, D9: DDZ15CSF, VST104_footprints:D_SOD-323-F_1.25x1.7mm, symbol Device:D_Zener
- added D12: BAV199, VST104_footprints:SOT-23-3_2.9x1.3mm, symbol Device:D_Schottky_x2_Serial_AKC
- added D16: FM4004W, VST104_footprints:D_SMA_DO-214AC_4.3x2.6mm, symbol Device:D
- added D4: ESDA25W5, VST104_footprints:SOT-323-5L_2.0x1.25mm, symbol Device:D_Zener_x2_ACom_KAK
- added J6, J7, J8: TSW-102-07-T-D, VST104_footprints:TSW-102-07-x-D, symbol Connector_Generic:Conn_02x02_Counter_Clockwise
- added P1: CX90M-16P, VST104_footprints:CX90M-16P, symbol VST104:USB_C_16
- added Q1, Q2, Q3, Q4, Q6, Q8, Q9: SQD40061EL, VST104_footprints:TO-252AA_6.5x6.1mm, symbol Device:Q_PMOS_GSD
- added Q10, Q5, Q7: 2N7002BK, VST104_footprints:SOT-23-3_2.9x1.3mm, symbol Device:Q_NMOS_GSD
- C1, C17, C18, C20, C21, C22, C8: footprint (none) -> VST104_footprints:C_SMD_0805
- C10, C11, C12, C13, C14, C19, C2, C3, C4, C5: footprint (none) -> VST104_footprints:C_SMD_0603
- C15, C16: footprint (none) -> VST104_footprints:CP_Radial_D8.0mm_P3.50mm_L11.5mm
- C6: renamed from C7; footprint (none) -> VST104_footprints:C_SMD_0603
- C7: renamed from C6; footprint (none) -> VST104_footprints:C_SMD_0805
- D10: renamed from D11; value TBAT54S -> BAV199; footprint (none) -> VST104_footprints:SOT-23-3_2.9x1.3mm
- D13: renamed from D14; value MAIN_OK -> LED; footprint (none) -> VST104_footprints:D_SMD_0603_LED
- D14: renamed from D15; footprint (none) -> VST104_footprints:D_SMD_0603_LED
- D15: renamed from D16; footprint (none) -> VST104_footprints:D_SMD_0603_LED
- D2: value STPS3L60U -> STPS3L60UFN; footprint (none) -> VST104_footprints:D_SMB-FN_DO-214AA-FN
- D5: renamed from D4; footprint (none) -> VST104_footprints:D_SOD-323_1.65x1.28mm
- D6: renamed from D5; value 15V -> DDZ15CSF; footprint (none) -> VST104_footprints:D_SOD-323-F_1.25x1.7mm
- D7: value VBUS_OK -> LED; footprint (none) -> VST104_footprints:D_SMD_0603_LED
- D8: value EXT_OK -> LED; footprint (none) -> VST104_footprints:D_SMD_0603_LED
- F1, F2, F3, F4, F5, F6: footprint (none) -> VST104_footprints:FUSE_2AG_01110501Z
- L1: footprint (none) -> VST104_footprints:L_SMD_8040_8.0x8.0x4.2mm
- R1, R10, R11, R12, R13, R14, R15, R16, R17, R18, R19, R2, R20, R21, R22, R23, R24, R25, R26, R27, R28, R29, R3, R30, R31, R32, R33, R4, R5, R6, R7, R8, R9: footprint (none) -> VST104_footprints:R_SMD_0603
- U6: value USBLC6 -> USBLC6-4; footprint VST104_footprints:SOT-363_TSSOP-6_2.0x1.25mm -> VST104_footprints:SOT-23-6L_2.9x1.6mm
- U7: value USBLC6 -> USBLC6-2; footprint VST104_footprints:SOT-363_TSSOP-6_2.0x1.25mm -> VST104_footprints:SOT-23-6L_2.9x1.6mm
- renumbered J3 to J1, J4 to J2, J5 to J3, J6 to J4, J7 to J5
Connections:
- wire segments 859 -> 873
- no-connect marks 24 -> 15
Other:
- note removed: "je tento rezistor OK?\n"
- note removed: "môžem na ochranu polarity použiť rovnaký tranzitor,\n ako na zvyšok spínania? (od nášh hovoru som ho zmenil)"
- note removed: "použil som rovnakú diódu akú\npoužíva USB-C chip, môže byť?"
- note removed: "použil som rovnakú ochranu,\nako používa USB-C chip,\nje to okay?\n"
- note removed: "skontrolujte prosím\nparametre tejto diody"
- moved on the sheet: C7

Commit message: tracing foxtrot
Parts:
- removed TP3: TestPoint, VST104_footprints:scope_PAD, symbol Connector:TestPoint
- removed TP9: TestPoint_Alt, VST104_footprints:KSE_PN6095, symbol Connector:TestPoint_Alt
- added D12: LED, VST104_footprints:D_SMD_0805_LED, symbol Device:LED
- added H1, H10, H11, H12, H13, H14, H15, H2, H3, H4, H5, H6, H7, H8, H9: MountingHole_Pad, VST104_footprints:MountingHole_3.2mm_M3_Pad_Via, symbol Mechanical:MountingHole_Pad
- added R19: 1k2, VST104_footprints:R_SMD_0805, symbol Device:R_Small
- 2A1: footprint VST104_footprints:R_SMD_0603 -> VST104_footprints:C_SMD_0805
- C10, C11, C12, C13, C14, C19, C2, C3, C4, C5, C6: footprint VST104_footprints:C_SMD_0603 -> VST104_footprints:C_SMD_0805
- D1: renamed from D14; footprint VST104_footprints:D_SMD_0603_LED -> VST104_footprints:D_SMD_0805_LED
- D10: renamed from D8; footprint VST104_footprints:D_SMD_0603_LED -> VST104_footprints:D_SMD_0805_LED
- D16: renamed from D13; footprint VST104_footprints:D_SMD_0603_LED -> VST104_footprints:D_SMD_0805_LED
- D3: renamed from D15; footprint VST104_footprints:D_SMD_0603_LED -> VST104_footprints:D_SMD_0805_LED
- D9: renamed from D7; footprint VST104_footprints:D_SMD_0603_LED -> VST104_footprints:D_SMD_0805_LED
- R1: renamed from R22; footprint VST104_footprints:R_SMD_0603 -> VST104_footprints:R_SMD_0805
- R10: renamed from R6; footprint VST104_footprints:R_SMD_0603 -> VST104_footprints:R_SMD_0805
- R11: renamed from R7; footprint VST104_footprints:R_SMD_0603 -> VST104_footprints:R_SMD_0805
- R12: renamed from R8; footprint VST104_footprints:R_SMD_0603 -> VST104_footprints:R_SMD_0805
- R13: renamed from R9; footprint VST104_footprints:R_SMD_0603 -> VST104_footprints:R_SMD_0805
- R14: renamed from R10; footprint VST104_footprints:R_SMD_0603 -> VST104_footprints:R_SMD_0805
- R15: renamed from R11; footprint VST104_footprints:R_SMD_0603 -> VST104_footprints:R_SMD_0805
- R16: renamed from R12; footprint VST104_footprints:R_SMD_0603 -> VST104_footprints:R_SMD_0805
- R17: renamed from R13; footprint VST104_footprints:R_SMD_0603 -> VST104_footprints:R_SMD_0805
- R18: renamed from R14; footprint VST104_footprints:R_SMD_0603 -> VST104_footprints:R_SMD_0805
- R2: renamed from R25; footprint VST104_footprints:R_SMD_0603 -> VST104_footprints:R_SMD_0805
- R20: renamed from R15; footprint VST104_footprints:R_SMD_0603 -> VST104_footprints:R_SMD_0805
- R21: renamed from R16; footprint VST104_footprints:R_SMD_0603 -> VST104_footprints:R_SMD_0805
- R22: renamed from R17; footprint VST104_footprints:R_SMD_0603 -> VST104_footprints:R_SMD_0805
- R23: renamed from R18; footprint VST104_footprints:R_SMD_0603 -> VST104_footprints:R_SMD_0805
- R24: renamed from R19; footprint VST104_footprints:R_SMD_0603 -> VST104_footprints:R_SMD_0805
- R25: renamed from R20; footprint VST104_footprints:R_SMD_0603 -> VST104_footprints:R_SMD_0805
- R26: renamed from R21; footprint VST104_footprints:R_SMD_0603 -> VST104_footprints:R_SMD_0805
- R27: renamed from R23; footprint VST104_footprints:R_SMD_0603 -> VST104_footprints:R_SMD_0805
- R28: renamed from R24; footprint VST104_footprints:R_SMD_0603 -> VST104_footprints:R_SMD_0805
- R29: renamed from R28; footprint VST104_footprints:R_SMD_0603 -> VST104_footprints:R_SMD_0805
- R3: renamed from R26; footprint VST104_footprints:R_SMD_0603 -> VST104_footprints:R_SMD_0805
- R30: renamed from R29; footprint VST104_footprints:R_SMD_0603 -> VST104_footprints:R_SMD_0805
- R31: renamed from R30; footprint VST104_footprints:R_SMD_0603 -> VST104_footprints:R_SMD_0805
- R32: renamed from R31; footprint VST104_footprints:R_SMD_0603 -> VST104_footprints:R_SMD_0805
- R33: renamed from R32; footprint VST104_footprints:R_SMD_0603 -> VST104_footprints:R_SMD_0805
- R34: renamed from R33; footprint VST104_footprints:R_SMD_0603 -> VST104_footprints:R_SMD_0805
- R4: renamed from R27; footprint VST104_footprints:R_SMD_0603 -> VST104_footprints:R_SMD_0805
- R5: renamed from R1; footprint VST104_footprints:R_SMD_0603 -> VST104_footprints:R_SMD_0805
- R6: renamed from R2; footprint VST104_footprints:R_SMD_0603 -> VST104_footprints:R_SMD_0805
- R7: renamed from R3; footprint VST104_footprints:R_SMD_0603 -> VST104_footprints:R_SMD_0805
- R8: renamed from R4; footprint VST104_footprints:R_SMD_0603 -> VST104_footprints:R_SMD_0805
- R9: renamed from R5; footprint VST104_footprints:R_SMD_0603 -> VST104_footprints:R_SMD_0805
- SW1: footprint VST104_footprints:G-168S-3011 -> VST104_footprints:EG4319
- U2: value TL432DBZ -> TL432AIDBZR; footprint Package_TO_SOT_SMD:SOT-23 -> VST104_footprints:SOT-23-3_2.9x1.3mm
- renumbered D9 to D11, D10 to D13, D11 to D14, D12 to D15, D16 to D17, D1 to D2, D2 to D4, D3 to D5, D4 to D6, D5 to D7, D6 to D8, Module_4 to Module_1, Module_1 to Module_4, Q10 to Q1, Q9 to Q10, Q1 to Q2, Q2 to Q3, Q3 to Q4, Q4 to Q5, Q5 to Q6, Q6 to Q7, Q7 to Q8, Q8 to Q9, R34 to R35, R35 to R36, R36 to R37, TP11 to TP10, TP12 to TP11, TP13 to TP12, TP14 to TP13, TP15 to TP14, TP4 to TP2, TP1 to TP3, TP2 to TP4, TP10 to TP9
Connections:
- net ALTER: now also J4.4 (Pin_4), R30.2; no longer J4.3 (Pin_3), R32.2
- net CC1: now also D6.3 (K); no longer D6.1 (K)
- net CC2: now also D6.1 (K); no longer D6.3 (K)
- net GND: now also J4.5 (Pin_5), D12.1 (K); no longer J4.2 (Pin_2)
- net SCL: now also J4.3 (Pin_3); no longer J4.4 (Pin_4)
- net SDA: now also J4.2 (Pin_2), R32.2; no longer J4.5 (Pin_5), R30.2
- net at 2A1.2, C10.1, C8.1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: now also R19.1
- new net: D12.2 (A), R19.2
- no-connect marks 15 -> 30
Other:
- moved on the sheet: 2A1, D1, D3, Module_1, Module_4, Q1, R1, R2, R3, R4, TP2

Commit message: ready for check
Parts:
- removed J1, J2: Conn_02x26_Top_Bottom, VST104_footprints:CES-126-01-x-D, symbol Connector_Generic:Conn_02x26_Top_Bottom
- removed J6, J7, J8: TSW-102-07-T-D, VST104_footprints:TSW-102-07-x-D, symbol Connector_Generic:Conn_02x02_Counter_Clockwise
- added H16, H17, H18: MountingHole_Pad, VST104_footprints:MountingHole_3.2mm_M3_Pad_Via, symbol Mechanical:MountingHole_Pad
- added J4, J5, J6: TSW-103-07-x-D, VST104_footprints:TSW-103-07-x-D, symbol Connector_Generic:Conn_02x03_Odd_Even
- added J7, J8: Conn_01x45, VST104_footprints:conn_FPC_45x0.5_505110-4591, symbol VST104:Conn_01x45
- added unit 4 of SW1
- F7: renamed from 2A1; value Fuse -> 2A1
- SW1: footprint VST104_footprints:EG4319 -> (none)
- TP1: renamed from TP2; footprint VST104_footprints:scope_PAD -> VST104_footprints:scope_PAD_1mm
- TP10: renamed from TP11; footprint VST104_footprints:scope_PAD -> VST104_footprints:scope_PAD_2mm
- TP11: renamed from TP12; footprint VST104_footprints:scope_PAD -> VST104_footprints:scope_PAD_2mm
- TP12: renamed from TP13; footprint VST104_footprints:scope_PAD -> VST104_footprints:scope_PAD_2mm
- TP13: renamed from TP14; footprint VST104_footprints:scope_PAD -> VST104_footprints:scope_PAD_2mm
- TP2: renamed from TP3; footprint VST104_footprints:scope_PAD -> VST104_footprints:scope_PAD_1mm
- TP3: renamed from TP4; footprint VST104_footprints:scope_PAD -> VST104_footprints:scope_PAD_1mm
- TP8: renamed from TP9; footprint VST104_footprints:scope_PAD -> VST104_footprints:scope_PAD_2mm
- TP9: renamed from TP10; footprint VST104_footprints:scope_PAD -> VST104_footprints:scope_PAD_2mm
- renumbered D12 to D11, D11 to D12, F6 to F5, F5 to F6, J3 to J1, J4 to J2, J5 to J3, Module_2 to Module_1, Module_3 to Module_2, Module_4 to Module_3, Module_1 to Module_4, Q9 to Q10, Q10 to Q9, R19 to R16, R16 to R17, R17 to R18, R18 to R19, R28 to R27, R27 to R28, TP5 to TP4, TP6 to TP5, TP7 to TP6, TP8 to TP7
Connections:
- net GNDA is gone; now on net GND: Module_1.H2_31 (AGND), Module_2.H2_31 (AGND), Module_3.H2_31 (AGND), Module_4.H2_31 (AGND)
- net GND: now also P1.MH (MOUNT), SW1.16 (3); no longer SW1.9 (1)
- net H1-1: now also J8.4 (Pin_4)
- net H1-10: now also J8.18 (Pin_18)
- net H1-11: now also J8.24 (Pin_24)
- net H1-12: now also J8.22 (Pin_22)
- net H1-13: now also J8.28 (Pin_28)
- net H1-14: now also J8.26 (Pin_26)
- net H1-15: now also J8.32 (Pin_32)
- net H1-16: now also J8.30 (Pin_30)
- net H1-17: now also J8.36 (Pin_36)
- net H1-18: now also J8.34 (Pin_34)
- net H1-19: now also J8.40 (Pin_40)
- net H1-2: now also J8.2 (Pin_2)
- net H1-20: now also J8.38 (Pin_38)
- net H1-21: now also J8.44 (Pin_44)
- net H1-22: now also J8.42 (Pin_42)
- net H1-23: now also J7.3 (Pin_3)
- net H1-24: now also J7.1 (Pin_1)
- net H1-25: now also J7.5 (Pin_5)
- net H1-26: now also J7.4 (Pin_4)
- net H1-27: now also J7.7 (Pin_7)
- net H1-28: now also J7.6 (Pin_6)
- net H1-29: now also J7.9 (Pin_9)
- net H1-3: now also J8.8 (Pin_8)
- net H1-30: now also J7.8 (Pin_8)
- net H1-31: now also J7.11 (Pin_11)
- net H1-32: now also J7.10 (Pin_10)
- net H1-35: now also J7.15 (Pin_15)
- net H1-36: now also J7.13 (Pin_13)
- net H1-37: now also J7.19 (Pin_19)
- net H1-38: now also J7.17 (Pin_17)
- net H1-39: now also J7.23 (Pin_23)
- net H1-4: now also J8.6 (Pin_6)
- net H1-40: now also J7.21 (Pin_21)
- net H1-41: now also J7.27 (Pin_27)
- net H1-42: now also J7.25 (Pin_25)
- net H1-43: now also J7.31 (Pin_31)
- net H1-44: now also J7.29 (Pin_29)
- net H1-45: now also J7.33 (Pin_33)
- net H1-46: now also J7.32 (Pin_32)
- net H1-47: now also J7.37 (Pin_37)
- net H1-48: now also J7.35 (Pin_35)
- net H1-49: now also J7.41 (Pin_41)
- net H1-5: now also J8.12 (Pin_12)
- net H1-50: now also J7.39 (Pin_39)
- net H1-51: now also J7.45 (Pin_45)
- net H1-52: now also J7.43 (Pin_43)
- net H1-6: now also J8.10 (Pin_10)
- net H1-7: now also J8.16 (Pin_16)
- net H1-8: now also J8.14 (Pin_14)
- net H1-9: now also J8.20 (Pin_20)
- net H2-1: now also J8.1 (Pin_1)
- net H2-10: now also J8.19 (Pin_19)
- net H2-11: now also J8.21 (Pin_21)
- net H2-12: now also J8.23 (Pin_23)
- net H2-13: now also J8.25 (Pin_25)
- net H2-14: now also J8.27 (Pin_27)
- net H2-15: now also J8.29 (Pin_29)
- net H2-16: now also J8.31 (Pin_31)
- net H2-17: now also J8.33 (Pin_33)
- net H2-18: now also J8.35 (Pin_35)
- net H2-19: now also J8.37 (Pin_37)
- net H2-2: now also J8.3 (Pin_3)
- net H2-20: now also J8.39 (Pin_39)
- net H2-21: now also J8.41 (Pin_41)
- net H2-22: now also J8.43 (Pin_43)
- net H2-23: now also J8.45 (Pin_45)
- net H2-24: now also J7.2 (Pin_2)
- net H2-3: now also J8.5 (Pin_5)
- net H2-35: now also J7.12 (Pin_12)
- net H2-36: now also J7.14 (Pin_14)
- net H2-37: now also J7.16 (Pin_16)
- net H2-38: now also J7.18 (Pin_18)
- net H2-39: now also J7.20 (Pin_20)
- net H2-4: now also J8.7 (Pin_7)
- net H2-40: now also J7.22 (Pin_22)
- net H2-41: now also J7.24 (Pin_24)
- net H2-42: now also J7.26 (Pin_26)
- net H2-43: now also J7.28 (Pin_28)
- net H2-44: now also J7.30 (Pin_30)
- net H2-47: now also J7.34 (Pin_34)
- net H2-48: now also J7.36 (Pin_36)
- net H2-49: now also J7.38 (Pin_38)
- net H2-5: now also J8.9 (Pin_9)
- net H2-50: now also J7.40 (Pin_40)
- net H2-51: now also J7.42 (Pin_42)
- net H2-52: now also J7.44 (Pin_44)
- net H2-6: now also J8.11 (Pin_11)
- net H2-7: now also J8.13 (Pin_13)
- net H2-8: now also J8.15 (Pin_15)
- net H2-9: now also J8.17 (Pin_17)
- net PDO2: now also SW1.13 (1); no longer SW1.12 (3)
- net SUP_3V3: now also J5.2 (Pin_2), J5.4 (Pin_4), J5.6 (Pin_6)
- net SUP_5V: now also J6.2 (Pin_2), J6.4 (Pin_4), J6.6 (Pin_6)
- net SUP_UNREG: now also J4.2 (Pin_2), J4.4 (Pin_4), J4.6 (Pin_6)
- net at D13.3 (common), U3.16 (VBUS_EN_SNK): now also SW1.1; no longer SW1.4 (3)
- net at C18.1, D17.1 (K), U5.2 (VIN): now also F5.1; no longer F6.1
- net at C22.1, D17.2 (A), R37.2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: now also F6.1; no longer F5.1
- net at R24.2: now also SW1.10; no longer SW1.6
- net at Q10.1 (G), R28.2: now also Q8.3 (D), R29.2; no longer Q8.1 (G), SW1.10
- net at Q9.1 (G), R27.2: now also Q8.1 (G), SW1.14; no longer Q8.3 (D), R29.2
- net at Q6.3 (D): now also SW1.9 (1); no longer SW1.5 (1)
- net at R35.1, TP11.1: now also J4.1 (Pin_1), J4.3 (Pin_3), J4.5 (Pin_5)
- net at R36.1, TP12.1: now also J5.1 (Pin_1), J5.3 (Pin_3), J5.5 (Pin_5)
- net at R37.1, TP13.1: now also J6.1 (Pin_1), J6.3 (Pin_3), J6.5 (Pin_5)
- no-connect marks 30 -> 38
Other:
- moved on the sheet: C1, C10, C11, C12, C13, C14, C15, C16, C17, C18, C19, C2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

Commit message: small updates
Parts:
- removed H13, H14, H15: MountingHole_Pad, VST104_footprints:MountingHole_3.2mm_M3_Pad_Via, symbol Mechanical:MountingHole_Pad
- removed R11, R12, R26: 1k2, VST104_footprints:R_SMD_0805, symbol Device:R_Small
- removed R33: 2k18, VST104_footprints:R_SMD_0805, symbol Device:R_Small
- removed U7: USBLC6-2, VST104_footprints:SOT-23-6L_2.9x1.6mm, symbol Power_Protection:USBLC6-2P6
- added LD1, LD2, LD3: AL5809, VST104_footprints:Power-DI-123_2.8x1.8x1mm, symbol Device:D_ALT
- added R18: 1k05, VST104_footprints:R_SMD_0805, symbol Device:R_Small
- added R20: 1k69, VST104_footprints:R_SMD_0805, symbol Device:R_Small
- added R36: 1k13, VST104_footprints:R_SMD_0805, symbol Device:R_Small
- added U6: USBLC6-4, VST104_footprints:SOT-23-6L_2.9x1.6mm, symbol Power_Protection:USBLC6-4SC6
- D12: renamed from D16; value LED -> green
- D14: renamed from D1; value LED -> yellow
- D15: renamed from D3; value LED -> blue
- D17: renamed from D11; value LED -> green
- D6: renamed from D9; value LED -> red
- D7: renamed from D10; value LED -> red
- R19: renamed from R34; value 1k34 -> 1k65
- R27: renamed from R1; value 250 -> 150
- R30: renamed from R4; value 250 -> 100
- renumbered C3 to C1, C17 to C10, C18 to C11, C20 to C12, C21 to C13, C22 to C14, C19 to C15, C1 to C16, C2 to C17, C4 to C18, C5 to C19, C6 to C2, C8 to C20, C9 to C21, C10 to C22, C7 to C3, C11 to C4, C12 to C5, C13 to C6, C14 to C7, C15 to C8, C16 to C9, D2 to D1, D14 to D10, D15 to D11, D17 to D13, D4 to D16, D5 to D2, D6 to D3, D7 to D4, D8 to D5, D12 to D8, D13 to D9, U4 to DC/DC1, U5 to DC/DC2, H16 to H13, H17 to H14, H18 to H15, J4 to J2, J5 to J3, J6 to J4, J2 to J5, J7 to J6, J3 to J7, Module_4 to Module_1, Module_1 to Module_2, Module_2 to Module_3, Module_3 to Module_4, Q2 to Q1, Q1 to Q10, Q3 to Q2, Q4 to Q3, Q5 to Q4, Q6 to Q5, Q7 to Q6, Q8 to Q7, Q9 to Q8, Q10 to Q9, R5 to R1, R21 to R10, R22 to R11, R23 to R12, R24 to R13, R25 to R14, R27 to R15, R28 to R16, R29 to R17, R6 to R2, R35 to R21, R36 to R22, R37 to R23, R30 to R24, R31 to R25, R32 to R26, R2 to R28, R3 to R29, R8 to R3, R7 to R31, R10 to R32, R15 to R33, R16 to R34, R17 to R35, R9 to R4, R13 to R5, R14 to R6, R18 to R7, R19 to R8, R20 to R9, TP2 to TP1, TP5 to TP10, TP6 to TP11, TP7 to TP12, TP1 to TP13, TP3 to TP2, TP8 to TP3, TP9 to TP4, TP10 to TP5, TP11 to TP6, TP12 to TP7, TP13 to TP8, TP4 to TP9, U2 to U1, U3 to U2, U6 to U5, U1 to U7
Connections:
- net +5V: now also U6.5 (VBUS)
- net GND: now also R20.2, R36.2, U6.2 (GND); no longer R19.2
- net USB_N: now also U6.1 (I/O1)
- net USB_P: now also U6.4 (I/O3)
- net VBUS: now also LD1.2 (A)
- net VSINK: now also LD3.2 (A)
- net VOUT_3V3: now reaches C13.1, DC/DC1.4 (VOUT), DC/DC1.5 (Sense), R22.2, TP4.1
- net at DC/DC1.6 (Trim): now also R18.1
- net at D5.1 (K), Q1.2 (S), Q3.3 (D)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: now also LD2.2 (A)
- net VOUT_5V: now reaches C14.1, D13.2 (A), DC/DC2.4 (VOUT), DC/DC2.5 (Sense), F6.1, R23.2, TP5.1
- net at R13.2: now also SW1.10; no longer SW1.10
- net at Q5.3 (D): now also SW1.9 (1); no longer SW1.9 (1)
- net VOUT_UNREG: now reaches C12.1, F3.1, R21.2, TP3.1
- net at D12.2 (A): now also LD3.1 (K)
- net at D6.2 (A): now also LD1.1 (K)
- net at D7.2 (A): now also LD2.1 (K)
- new net: R19.2, R20.1
- new net: R18.2, R36.1
- no-connect marks 38 -> 37
Other:
- moved on the sheet: R19
