File: element_foxtrot/element_foxtrot.sch (KiCad schematic (older format))
At the start: 145 parts, among them J1 Ext_Power, J2 TSW-103-07-x-D, J3 TSW-103-07-x-D, J4 TSW-103-07-x-D, J5 Program, J6 Conn_01x45, J7 USB, J8 Conn_01x45, P1 CX90M-16P, Q1 SQD40061EL, Q10 2N7002BK, Q2 SQD40061EL, Q3 SQD40061EL, Q4 SQD40061EL, Q5 2N7002BK, Q6 SQD40061EL, Q7 2N7002BK, Q8 SQD40061EL, Q9 SQD40061EL, SW1 switch_3P3T, U1 TL432AIDBZR, U2 STUSB4500QTR, U5 USBLC6-4, U6 USBLC6-4, U7 L7985

Commit message: ready to manufacture
Parts:
- removed R18: 1k05, VST104_footprints:R_SMD_0805, symbol Device:R_Small
- removed R19: 1k65, VST104_footprints:R_SMD_0805, symbol Device:R_Small
- removed R20: 1k69, VST104_footprints:R_SMD_0805, symbol Device:R_Small
- removed R36: 1k13, VST104_footprints:R_SMD_0805, symbol Device:R_Small
- added RV? (x2): 3k3, VST104_footprints:trimer_3296W_10.0x9.5x10.0, symbol Device:R_POT_Small
Connections:
- net GND: now also RV?.1, RV?.1
- net at DC/DC1.6 (Trim): now also RV?.2, RV?.3
- net at DC/DC2.6 (Trim): now also RV?.2, RV?.3
Changed lines of the file:
@@
 L power:GND #PWR044
 U 1 1 7DFA8845
-P 8550 12400
-F 0 "#PWR044" H 8550 12150 50  0001 C CNN
-F 1 "GND" H 8555 12227 50  0000 C CNN
-F 2 "" H 8550 12400 50  0001 C CNN
-F 3 "" H 8550 12400 50  0001 C CNN
-	1    8550 12400
+P 8550 12450
+F 0 "#PWR044" H 8550 12200 50  0001 C CNN
+F 1 "GND" H 8555 12277 50  0000 C CNN
+F 2 "" H 8550 12450 50  0001 C CNN
+F 3 "" H 8550 12450 50  0001 C CNN
+	1    8550 12450
 	1    0    0    -1
 $EndComp
@@
 L power:GND #PWR051
 U 1 1 88AFEF1E
-P 9550 12300
-F 0 "#PWR051" H 9550 12050 50  0001 C CNN
-F 1 "GND" H 9555 12127 50  0000 C CNN
-F 2 "" H 9550 12300 50  0001 C CNN
-F 3 "" H 9550 12300 50  0001 C CNN
-	1    9550 12300
+P 9550 12450
+F 0 "#PWR051" H 9550 12200 50  0001 C CNN
+F 1 "GND" H 9555 12277 50  0000 C CNN
+F 2 "" H 9550 12450 50  0001 C CNN
+F 3 "" H 9550 12450 50  0001 C CNN
+	1    9550 12450
 	1    0    0    -1
 $EndComp
@@
 L power:GND #PWR050
 U 1 1 89644F01
-P 9550 11150
-F 0 "#PWR050" H 9550 10900 50  0001 C CNN
-F 1 "GND" H 9555 10977 50  0000 C CNN
-F 2 "" H 9550 11150 50  0001 C CNN
-F 3 "" H 9550 11150 50  0001 C CNN
-	1    9550 11150
+P 9550 11300
+F 0 "#PWR050" H 9550 11050 50  0001 C CNN
+F 1 "GND" H 9555 11127 50  0000 C CNN
+F 2 "" H 9550 11300 50  0001 C CNN
+F 3 "" H 9550 11300 50  0001 C CNN
+	1    9550 11300
 	1    0    0    -1
 $EndComp
@@
 	7250 12700 7350 12700
 NoConn ~ 8050 11100
-Wire Wire Line
-	9000 11100 9100 11100
 $Comp
 L power:GND #PWR043
 U 1 1 7DFAA219
-P 8550 11250
-F 0 "#PWR043" H 8550 11000 50  0001 C CNN
-F 1 "GND" H 8555 11077 50  0000 C CNN
-F 2 "" H 8550 11250 50  0001 C CNN
-F 3 "" H 8550 11250 50  0001 C CNN
-	1    8550 11250
+P 8550 11300
+F 0 "#PWR043" H 8550 11050 50  0001 C CNN
+F 1 "GND" H 8555 11127 50  0000 C CNN
+F 2 "" H 8550 11300 50  0001 C CNN
+F 3 "" H 8550 11300 50  0001 C CNN
+	1    8550 11300
 	1    0    0    -1
 $EndComp
@@
 Connection ~ 10100 9850
 $Comp
-L Device:R_Small R19
-U 1 1 62B54CD8
-P 9200 12150
-F 0 "R19" H 9259 12196 50  0000 L CNN
-F 1 "1k65" H 9259 12105 50  0000 L CNN
-F 2 "VST104_footprints:R_SMD_0805" H 9200 12150 50  0001 C CNN
-F 3 "~" H 9200 12150 50  0001 C CNN
-	1    9200 12150
-	1    0    0    -1
-$EndComp
-Wire Wire Line
-	9000 12250 9100 12250
-$Comp
 L power:GND #PWR046
 U 1 1 62B54CDF
@@
 VOUT_UNREG
 $Comp
-L Device:R_Small R20
-U 1 1 61915430
-P 9200 12350
-F 0 "R20" H 9259 12396 50  0000 L CNN
-F 1 "1k69" H 9259 12305 50  0000 L CNN
-F 2 "VST104_footprints:R_SMD_0805" H 9200 12350 50  0001 C CNN
-F 3 "~" H 9200 12350 50  0001 C CNN
-	1    9200 12350
-	1    0    0    -1
-$EndComp
-Wire Wire Line
-	9100 12250 9100 12050
-Wire Wire Line
-	9100 12050 9200 12050
-$Comp
-L Device:R_Small R18
-U 1 1 61D216FD
-P 9200 11000
-F 0 "R18" H 9259 11046 50  0000 L CNN
-F 1 "1k05" H 9259 10955 50  0000 L CNN
-F 2 "VST104_footprints:R_SMD_0805" H 9200 11000 50  0001 C CNN
-F 3 "~" H 9200 11000 50  0001 C CNN
-	1    9200 11000
-	1    0    0    -1
-$EndComp
-$Comp
-L power:GND #PWR045
-U 1 1 61D21704
-P 9200 11300
-F 0 "#PWR045" H 9200 11050 50  0001 C CNN
-F 1 "GND" H 9205 11127 50  0000 C CNN
-F 2 "" H 9200 11300 50  0001 C CNN
-F 3 "" H 9200 11300 50  0001 C CNN
-	1    9200 11300
-	1    0    0    -1
-$EndComp
-$Comp
-L Device:R_Small R36
-U 1 1 61D2170A
-P 9200 11200
-F 0 "R36" H 9259 11246 50  0000 L CNN
-F 1 "1k13" H 9259 11155 50  0000 L CNN
-F 2 "VST104_footprints:R_SMD_0805" H 9200 11200 50  0001 C CNN
-F 3 "~" H 9200 11200 50  0001 C CNN
-	1    9200 11200
-	1    0    0    -1
-$EndComp
-Wire Wire Line
-	9100 11100 9100 10900
-Wire Wire Line
-	9100 10900 9200 10900
-$Comp
 L Connector_Generic:Conn_02x03_Odd_Even J3
 U 1 1 60562DCE
@@
 	1    0    0    -1
 $EndComp
+$Comp
+L Device:R_POT_Small RV?
+U 1 1 5F8811C4
+P 9200 12350
+F 0 "RV?" H 9140 12304 50  0000 R CNN
+F 1 "3k3" H 9140 12395 50  0000 R CNN
+F 2 "VST104_footprints:trimer_3296W_10.0x9.5x10.0" H 9200 12350 50  0001 C CNN
+F 3 "https://www.mouser.sk/datasheet/2/54/3296-776415.pdf" H 9200 12350 50  0001 C CNN
+	1    9200 12350
+	-1   0    0    1
+$EndComp
+Wire Wire Line
+	9000 12250 9050 12250
+Wire Wire Line
+	9100 12350 9050 12350
+Wire Wire Line
+	9050 12350 9050 12250
+Connection ~ 9050 12250
+Wire Wire Line
+	9050 12250 9200 12250
+Wire Wire Line
+	9550 12450 9550 12300
+Wire Wire Line
+	8550 12450 8550 12400
+$Comp
+L power:GND #PWR?
+U 1 1 6037F51F
+P 9200 11300
+F 0 "#PWR?" H 9200 11050 50  0001 C CNN
+F 1 "GND" H 9205 11127 50  0000 C CNN
+F 2 "" H 9200 11300 50  0001 C CNN
+F 3 "" H 9200 11300 50  0001 C CNN
+	1    9200 11300
+	1    0    0    -1
+$EndComp
+Wire Wire Line
+	9050 11100 9200 11100
+Wire Wire Line
+	9100 11200 9050 11200
+Wire Wire Line
+	9050 11200 9050 11100
+Wire Wire Line
+	9550 11300 9550 11150
+Wire Wire Line
+	9000 11100 9050 11100
+Connection ~ 9050 11100
+Wire Wire Line
+	8550 11300 8550 11250
+$Comp
+L Device:R_POT_Small RV?
+U 1 1 60E8CEC9
+P 9200 11200
+F 0 "RV?" H 9140 11154 50  0000 R CNN
+F 1 "3k3" H 9140 11245 50  0000 R CNN
+F 2 "VST104_footprints:trimer_3296W_10.0x9.5x10.0" H 9200 11200 50  0001 C CNN
+F 3 "https://www.mouser.sk/datasheet/2/54/3296-776415.pdf" H 9200 11200 50  0001 C CNN
+	1    9200 11200
+	-1   0    0    1
+$EndComp
 $EndSCHEMATC

Commit message: manufacture order
Parts:
- SW1: value switch_3P3T -> EG4319A
- SW1: value switch_3P3T -> EG4319A; footprint (none) -> VST104_footprints:EG4319
- gave numbers to parts that had none: 2
Connections:
- net GND: now also SW1.13 (1), SW1.15 (2); no longer SW1.16 (3)
- net PDO2: now also SW1.16 (3); no longer SW1.13 (1)
- net at D9.3 (common), U2.16 (VBUS_EN_SNK): now also SW1.4 (3); no longer SW1.1
- no-connect marks 37 -> 36
Changed lines of the file:
@@
 	5900 8700 5850 8700
 NoConn ~ 5900 8600
-NoConn ~ 5900 8500
 Wire Wire Line
 	5050 10500 5000 10500
@@
 	0    1    1    0
 $EndComp
-NoConn ~ 5850 12750
 Wire Wire Line
 	5900 12650 5850 12650
@@
 	5850 12850 5900 12850
 Wire Wire Line
-	5850 12750 5900 12750
-Wire Wire Line
 	5500 10500 5450 10500
 Wire Wire Line
@@
 Wire Wire Line
 	5900 8600 5850 8600
-Wire Wire Line
-	5900 8500 5850 8500
 NoConn ~ 5250 12200
 NoConn ~ 5250 12600
@@
 U 1 1 61CCC044
 P 5250 10500
-F 0 "SW1" H 5250 10297 50  0000 C CNN
-F 1 "switch_3P3T" H 5300 10300 50  0001 C CNN
+F 0 "SW1" H 5250 10733 50  0000 C CNN
+F 1 "EG4319A" H 5300 10300 50  0001 C CNN
 F 2 "VST104_footprints:EG4319" H 4850 10200 50  0001 C CNN
-F 3 "" H 4850 10200 50  0001 C CNN
+F 3 "https://www.mouser.sk/datasheet/2/140/EG-345873.pdf" H 4850 10200 50  0001 C CNN
 	1    5250 10500
-	1    0    0    1
+	1    0    0    -1
 $EndComp
 $Comp
@@
 P 5650 8600
 F 0 "SW1" H 5650 8397 50  0000 C CNN
-F 1 "switch_3P3T" H 5700 8400 50  0001 C CNN
+F 1 "EG4319A" H 5700 8400 50  0001 C CNN
 F 2 "VST104_footprints:EG4319" H 5250 8300 50  0001 C CNN
-F 3 "" H 5250 8300 50  0001 C CNN
+F 3 "https://www.mouser.sk/datasheet/2/140/EG-345873.pdf" H 5250 8300 50  0001 C CNN
 	3    5650 8600
 	1    0    0    1
@@
 U 4 1 62114F45
 P 6100 12750
-F 0 "SW1" H 6100 12983 50  0000 C CNN
-F 1 "switch_3P3T" H 6150 12550 50  0001 C CNN
-F 2 "" H 5700 12450 50  0001 C CNN
-F 3 "" H 5700 12450 50  0001 C CNN
+F 0 "SW1" H 6100 12547 50  0000 C CNN
+F 1 "EG4319A" H 6150 12550 50  0001 C CNN
+F 2 "VST104_footprints:EG4319" H 5700 12450 50  0001 C CNN
+F 3 "https://www.mouser.sk/datasheet/2/140/EG-345873.pdf" H 5700 12450 50  0001 C CNN
 	4    6100 12750
-	-1   0    0    -1
+	-1   0    0    1
 $EndComp
 Connection ~ 6300 12750
@@
 P 5700 9250
 F 0 "SW1" H 5700 9047 50  0000 C CNN
-F 1 "switch_3P3T" H 5750 9050 50  0001 C CNN
-F 2 "" H 5300 8950 50  0001 C CNN
-F 3 "" H 5300 8950 50  0001 C CNN
+F 1 "EG4319A" H 5750 9050 50  0001 C CNN
+F 2 "VST104_footprints:EG4319" H 5300 8950 50  0001 C CNN
+F 3 "https://www.mouser.sk/datasheet/2/140/EG-345873.pdf" H 5300 8950 50  0001 C CNN
 	2    5700 9250
 	1    0    0    -1
@@
 $EndComp
 $Comp
-L Device:R_POT_Small RV?
+L Device:R_POT_Small RV2
 U 1 1 5F8811C4
 P 9200 12350
-F 0 "RV?" H 9140 12304 50  0000 R CNN
+F 0 "RV2" H 9140 12304 50  0000 R CNN
 F 1 "3k3" H 9140 12395 50  0000 R CNN
 F 2 "VST104_footprints:trimer_3296W_10.0x9.5x10.0" H 9200 12350 50  0001 C CNN
@@
 	8550 12450 8550 12400
 $Comp
-L power:GND #PWR?
+L power:GND #PWR0101
 U 1 1 6037F51F
 P 9200 11300
-F 0 "#PWR?" H 9200 11050 50  0001 C CNN
+F 0 "#PWR0101" H 9200 11050 50  0001 C CNN
 F 1 "GND" H 9205 11127 50  0000 C CNN
 F 2 "" H 9200 11300 50  0001 C CNN
@@
 	8550 11300 8550 11250
 $Comp
-L Device:R_POT_Small RV?
+L Device:R_POT_Small RV1
 U 1 1 60E8CEC9
 P 9200 11200
-F 0 "RV?" H 9140 11154 50  0000 R CNN
+F 0 "RV1" H 9140 11154 50  0000 R CNN
 F 1 "3k3" H 9140 11245 50  0000 R CNN
 F 2 "VST104_footprints:trimer_3296W_10.0x9.5x10.0" H 9200 11200 50  0001 C CNN
@@
 	-1   0    0    1
 $EndComp
+$Comp
+L power:GND #PWR0102
+U 1 1 5F8114D4
+P 5850 12750
+F 0 "#PWR0102" H 5850 12500 50  0001 C CNN
+F 1 "GND" V 5855 12622 50  0000 R CNN
+F 2 "" H 5850 12750 50  0001 C CNN
+F 3 "" H 5850 12750 50  0001 C CNN
+	1    5850 12750
+	0    1    1    0
+$EndComp
+Wire Wire Line
+	5850 12750 5900 12750
+Wire Wire Line
+	5900 8500 5850 8500
+NoConn ~ 5900 8500
 $EndSCHEMATC

Commit message: almost traced
Parts:
- R34: value 1k2 -> 150
Changed lines of the file:
@@
 P 20350 3650
 F 0 "R34" H 20409 3696 50  0000 L CNN
-F 1 "1k2" H 20409 3605 50  0000 L CNN
+F 1 "150" H 20409 3605 50  0000 L CNN
 F 2 "VST104_footprints:R_SMD_0805" H 20350 3650 50  0001 C CNN
 F 3 "~" H 20350 3650 50  0001 C CNN
