File: element_foxtrot/element_foxtrot.sch (KiCad schematic (older format))
At the start: 143 parts, among them J1 Ext_Power, J2 TSW-103-07-x-D, J3 TSW-103-07-x-D, J4 TSW-103-07-x-D, J5 Program, J6 Conn_01x45, J7 USB, J8 Conn_01x45, P1 CX90M-16P, Q1 SQD40061EL, Q10 2N7002BK, Q2 SQD40061EL, Q3 SQD40061EL, Q4 SQD40061EL, Q5 2N7002BK, Q6 SQD40061EL, Q7 2N7002BK, Q8 SQD40061EL, Q9 SQD40061EL, SW1 EG4319A, U1 TL432AIDBZR, U2 STUSB4500QTR, U5 USBLC6-4, U6 USBLC6-4, U7 L7985

Commit message: updated to v1.1
Parts:
- removed R17: 100, VST104_footprints:R_SMD_0805, symbol Device:R_Small
- added D13: NSR0320MW2T1G, VST104_footprints:D_SOD-323_1.65x1.28mm, symbol Device:D_Schottky
- renumbered D13 to D14, D14 to D15, D15 to D16, D16 to D17, D17 to D18, R21 to R17, R22 to R18, R23 to R19, R24 to R20, R25 to R21, R26 to R22, R27 to R23, R28 to R24, R29 to R25, R30 to R26, R31 to R27, R32 to R28, R33 to R29, R34 to R30, R35 to R31, U5 to U3, U6 to U4, U7 to U5
Connections:
- net at DC/DC2.1 (EN): now also D13.2 (A)
- net at Q7.3 (D), Q9.1 (G), R16.2: now also D13.1 (K)
