File: board_delta/board_delta.sch (KiCad schematic (older format))
At the start: 6 parts

Commit message: almost traced
Parts:
- H1, H2: footprint VST104_footprints:ESQ-126-39-x-D -> VST104_footprints:ESQ-129-39-x-D
- renumbered MH3 to MH2, MH2 to MH3
Other:
- moved on the sheet: MH1, MH2, MH3, MH4
Changed lines of the file:
@@
 F 0 "H2" H 2500 6700 50  0000 C CNN
 F 1 "Conn_02x26_Odd_Even" H 2500 4000 50  0001 C CNN
-F 2 "VST104_footprints:ESQ-126-39-x-D" H 2450 5400 50  0001 C CNN
+F 2 "VST104_footprints:ESQ-129-39-x-D" H 2450 5400 50  0001 C CNN
 F 3 "~" H 2450 5400 50  0001 C CNN
 	1    2450 5400
@@
 F 0 "H1" H 2500 3750 50  0000 C CNN
 F 1 "Conn_02x26_Odd_Even" H 2500 1050 50  0001 C CNN
-F 2 "VST104_footprints:ESQ-126-39-x-D" H 2450 2450 50  0001 C CNN
+F 2 "VST104_footprints:ESQ-129-39-x-D" H 2450 2450 50  0001 C CNN
 F 3 "~" H 2450 2450 50  0001 C CNN
 	1    2450 2450
@@
 $EndComp
 $Comp
-L Mechanical:MountingHole_Pad MH2
+L Mechanical:MountingHole_Pad MH3
 U 1 1 5E50DEC4
-P 7650 6850
-F 0 "MH2" H 7750 6853 50  0000 L CNN
-F 1 "MountingHole_Pad" H 7750 6808 50  0001 L CNN
-F 2 "VST104_footprints:MountingHole_3.2mm_M3_Pad_Via" H 7650 6850 50  0001 C CNN
-F 3 "~" H 7650 6850 50  0001 C CNN
-	1    7650 6850
-	1    0    0    -1
-$EndComp
-NoConn ~ 7250 6950
-NoConn ~ 8400 6950
-NoConn ~ 8050 6950
+P 7525 6750
+F 0 "MH3" H 7625 6753 50  0000 L CNN
+F 1 "MountingHole_Pad" H 7625 6708 50  0001 L CNN
+F 2 "VST104_footprints:MountingHole_3.2mm_M3_Pad_Via" H 7525 6750 50  0001 C CNN
+F 3 "~" H 7525 6750 50  0001 C CNN
+	1    7525 6750
+	1    0    0    -1
+$EndComp
+NoConn ~ 7175 6850
+NoConn ~ 7725 7050
+NoConn ~ 7325 7050
 $Comp
 L Mechanical:MountingHole_Pad MH4
 U 1 1 5E50E2B0
-P 8400 6850
-F 0 "MH4" H 8500 6853 50  0000 L CNN
-F 1 "MountingHole_Pad" H 8500 6808 50  0001 L CNN
-F 2 "VST104_footprints:MountingHole_3.2mm_M3_Pad_Via" H 8400 6850 50  0001 C CNN
-F 3 "~" H 8400 6850 50  0001 C CNN
-	1    8400 6850
-	1    0    0    -1
-$EndComp
-$Comp
-L Mechanical:MountingHole_Pad MH3
+P 7725 6950
+F 0 "MH4" H 7825 6953 50  0000 L CNN
+F 1 "MountingHole_Pad" H 7825 6908 50  0001 L CNN
+F 2 "VST104_footprints:MountingHole_3.2mm_M3_Pad_Via" H 7725 6950 50  0001 C CNN
+F 3 "~" H 7725 6950 50  0001 C CNN
+	1    7725 6950
+	1    0    0    -1
+$EndComp
+$Comp
+L Mechanical:MountingHole_Pad MH2
 U 1 1 5E50E4A0
-P 8050 6850
-F 0 "MH3" H 8150 6853 50  0000 L CNN
-F 1 "MountingHole_Pad" H 8150 6808 50  0001 L CNN
-F 2 "VST104_footprints:MountingHole_3.2mm_M3_Pad_Via" H 8050 6850 50  0001 C CNN
-F 3 "~" H 8050 6850 50  0001 C CNN
-	1    8050 6850
+P 7325 6950
+F 0 "MH2" H 7425 6953 50  0000 L CNN
+F 1 "MountingHole_Pad" H 7425 6908 50  0001 L CNN
+F 2 "VST104_footprints:MountingHole_3.2mm_M3_Pad_Via" H 7325 6950 50  0001 C CNN
+F 3 "~" H 7325 6950 50  0001 C CNN
+	1    7325 6950
 	1    0    0    -1
 $EndComp
@@
 L Mechanical:MountingHole_Pad MH1
 U 1 1 5E50E62D
-P 7250 6850
-F 0 "MH1" H 7350 6853 50  0000 L CNN
-F 1 "MountingHole_Pad" H 7350 6808 50  0001 L CNN
-F 2 "VST104_footprints:MountingHole_3.2mm_M3_Pad_Via" H 7250 6850 50  0001 C CNN
-F 3 "~" H 7250 6850 50  0001 C CNN
-	1    7250 6850
-	1    0    0    -1
-$EndComp
-NoConn ~ 7650 6950
+P 7175 6750
+F 0 "MH1" H 7275 6753 50  0000 L CNN
+F 1 "MountingHole_Pad" H 7275 6708 50  0001 L CNN
+F 2 "VST104_footprints:MountingHole_3.2mm_M3_Pad_Via" H 7175 6750 50  0001 C CNN
+F 3 "~" H 7175 6750 50  0001 C CNN
+	1    7175 6750
+	1    0    0    -1
+$EndComp
+NoConn ~ 7525 6850
 $Comp
 L power:PWR_FLAG #FLG01
 U 1 1 769BCE2E
-P 9950 6850
-F 0 "#FLG01" H 9950 6925 50  0001 C CNN
-F 1 "PWR_FLAG" H 9950 7023 50  0000 C CNN
-F 2 "" H 9950 6850 50  0001 C CNN
-F 3 "~" H 9950 6850 50  0001 C CNN
-	1    9950 6850
+P 8875 6850
+F 0 "#FLG01" H 8875 6925 50  0001 C CNN
+F 1 "PWR_FLAG" H 8875 7023 50  0000 C CNN
+F 2 "" H 8875 6850 50  0001 C CNN
+F 3 "~" H 8875 6850 50  0001 C CNN
+	1    8875 6850
 	1    0    0    -1
 $EndComp
@@
 L power:PWR_FLAG #FLG02
 U 1 1 76BE42BF
-P 10450 6850
-F 0 "#FLG02" H 10450 6925 50  0001 C CNN
-F 1 "PWR_FLAG" H 10450 7023 50  0000 C CNN
-F 2 "" H 10450 6850 50  0001 C CNN
-F 3 "~" H 10450 6850 50  0001 C CNN
-	1    10450 6850
-	1    0    0    -1
-$EndComp
-$Comp
-L power:GND #PWR06
+P 9375 6850
+F 0 "#FLG02" H 9375 6925 50  0001 C CNN
+F 1 "PWR_FLAG" H 9375 7023 50  0000 C CNN
+F 2 "" H 9375 6850 50  0001 C CNN
+F 3 "~" H 9375 6850 50  0001 C CNN
+	1    9375 6850
+	1    0    0    -1
+$EndComp
+$Comp
+L power:GND #PWR0160
 U 1 1 7700DCCC
-P 10900 6900
-F 0 "#PWR06" H 10900 6650 50  0001 C CNN
-F 1 "GND" H 10905 6727 50  0000 C CNN
-F 2 "" H 10900 6900 50  0001 C CNN
-F 3 "" H 10900 6900 50  0001 C CNN
-	1    10900 6900
-	1    0    0    -1
-$EndComp
-Wire Wire Line
-	10900 6850 10900 6900
-Text GLabel 9900 7000 0    50   Input ~ 0
+P 9825 6900
+F 0 "#PWR0160" H 9825 6650 50  0001 C CNN
+F 1 "GND" H 9830 6727 50  0000 C CNN
+F 2 "" H 9825 6900 50  0001 C CNN
+F 3 "" H 9825 6900 50  0001 C CNN
+	1    9825 6900
+	1    0    0    -1
+$EndComp
+Wire Wire Line
+	9825 6850 9825 6900
+Text GLabel 8825 7000 0    50   Input ~ 0
 SUP_5V
-Text GLabel 10400 7000 0    50   Input ~ 0
+Text GLabel 9325 7000 0    50   Input ~ 0
 SUP_3V3
 Wire Wire Line
-	10450 7000 10400 7000
-Wire Wire Line
-	10450 6850 10450 7000
-Wire Wire Line
-	9950 7000 9900 7000
-Wire Wire Line
-	9950 6850 9950 7000
+	9375 7000 9325 7000
+Wire Wire Line
+	9375 6850 9375 7000
+Wire Wire Line
+	8875 7000 8825 7000
+Wire Wire Line
+	8875 6850 8875 7000
 Wire Notes Line width 10
 	1500 1000 3500 1000
-Text Notes 1500 950  0    100  ~ 20
+Text Notes 1500 950  0    65   ~ 13
 LibreCube main headers
 Wire Wire Line
@@
 	3600 6100 2750 6100
 $Comp
-L power:GND #PWR02
+L power:GND #PWR0147
 U 1 1 62558AF2
 P 1400 5600
-F 0 "#PWR02" H 1400 5350 50  0001 C CNN
+F 0 "#PWR0147" H 1400 5350 50  0001 C CNN
 F 1 "GND" V 1405 5472 50  0000 R CNN
 F 2 "" H 1400 5600 50  0001 C CNN
@@
 $EndComp
 $Comp
-L power:GND #PWR04
+L power:GND #PWR0168
 U 1 1 6255D770
 P 3600 5600
-F 0 "#PWR04" H 3600 5350 50  0001 C CNN
+F 0 "#PWR0168" H 3600 5350 50  0001 C CNN
 F 1 "GND" V 3605 5472 50  0000 R CNN
 F 2 "" H 3600 5600 50  0001 C CNN
@@
 USER_3_2
 $Comp
-L power:GND #PWR01
+L power:GND #PWR0146
 U 1 1 646D90AD
 P 1400 2850
-F 0 "#PWR01" H 1400 2600 50  0001 C CNN
+F 0 "#PWR0146" H 1400 2600 50  0001 C CNN
 F 1 "GND" V 1405 2722 50  0000 R CNN
 F 2 "" H 1400 2850 50  0001 C CNN
@@
 $EndComp
 $Comp
-L power:GND #PWR03
+L power:GND #PWR0167
 U 1 1 646DA961
 P 3600 2850
-F 0 "#PWR03" H 3600 2600 50  0001 C CNN
+F 0 "#PWR0167" H 3600 2600 50  0001 C CNN
 F 1 "GND" V 3605 2722 50  0000 R CNN
 F 2 "" H 3600 2850 50  0001 C CNN
@@
 USER_6_1
 $Comp
-L power:GND #PWR05
+L power:GND #PWR0169
 U 1 1 7016B9DA
 P 3600 5700
-F 0 "#PWR05" H 3600 5450 50  0001 C CNN
+F 0 "#PWR0169" H 3600 5450 50  0001 C CNN
 F 1 "GND" V 3605 5572 50  0000 R CNN
 F 2 "" H 3600 5700 50  0001 C CNN
@@
 L power:PWR_FLAG #FLG03
 U 1 1 82F35DD9
-P 10900 6850
-F 0 "#FLG03" H 10900 6925 50  0001 C CNN
-F 1 "PWR_FLAG" H 10900 7023 50  0000 C CNN
-F 2 "" H 10900 6850 50  0001 C CNN
-F 3 "~" H 10900 6850 50  0001 C CNN
-	1    10900 6850
+P 9825 6850
+F 0 "#FLG03" H 9825 6925 50  0001 C CNN
+F 1 "PWR_FLAG" H 9825 7023 50  0000 C CNN
+F 2 "" H 9825 6850 50  0001 C CNN
+F 3 "~" H 9825 6850 50  0001 C CNN
+	1    9825 6850
 	1    0    0    -1
 $EndComp
@@
 NoConn ~ 2250 5700
 $Sheet
-S 5500 1000 2000 2000
-U 68280FAF
-F0 "OBC_left" 100
-F1 "OBC_left.sch" 50
+S 5750 2250 1000 1000
+U 6E7B0394
+F0 "left_OBC" 65
+F1 "left_OBC.sch" 50
 $EndSheet
+Text GLabel 3600 2550 2    50   Input ~ 0
+CPU_WD_2
+Wire Wire Line
+	2750 2550 3600 2550
 Wire Wire Line
 	3600 2950 2750 2950
 Text GLabel 3600 2950 2    50   Input ~ 0
 GLO_KS_2
-Text GLabel 3600 2550 2    50   Input ~ 0
-CPU_WD_2
-Wire Wire Line
-	3600 2550 2750 2550
 $Sheet
-S 8000 3500 2000 2000
-U 5F9EC867
-F0 "OBC_right" 100
-F1 "OBC_right.sch" 50
+S 7000 3500 1000 1000
+U 5F8745FB
+F0 "right_OBC" 65
+F1 "right_OBC.sch" 50
 $EndSheet
 $EndSCHEMATC

Commit message: finished
Parts:
- added F1, F2: R_Small, VST104_footprints:R_SMD_1206, symbol Device:R_Small
- added UA1: Conn_01x03, VST104_footprints:PC104_universal_FPGA, symbol Connector_Generic:Conn_01x03
- added UA2, UA3: Conn_02x12_Counter_Clockwise, VST104_footprints:PC104_SO-24_universal, symbol Connector_Generic:Conn_02x12_Counter_Clockwise
- H1, H2: footprint VST104_footprints:ESQ-129-39-x-D -> VST104_footprints:ESQ-126-39-x-D
Connections:
- net GND: now also UA1.1 (Pin_1)
- net SUP_3V3: now also F1.2
- net SUP_5V: now also F2.2
- new net: F1.1, UA1.2 (Pin_2)
- new net: F2.1, UA1.3 (Pin_3)
- no-connect marks 36 -> 84
Other:
- note added: "Universal SO-24 footprint\n"
Changed lines of the file:
@@
 F 0 "H2" H 2500 6700 50  0000 C CNN
 F 1 "Conn_02x26_Odd_Even" H 2500 4000 50  0001 C CNN
-F 2 "VST104_footprints:ESQ-129-39-x-D" H 2450 5400 50  0001 C CNN
+F 2 "VST104_footprints:ESQ-126-39-x-D" H 2450 5400 50  0001 C CNN
 F 3 "~" H 2450 5400 50  0001 C CNN
 	1    2450 5400
@@
 F 0 "H1" H 2500 3750 50  0000 C CNN
 F 1 "Conn_02x26_Odd_Even" H 2500 1050 50  0001 C CNN
-F 2 "VST104_footprints:ESQ-129-39-x-D" H 2450 2450 50  0001 C CNN
+F 2 "VST104_footprints:ESQ-126-39-x-D" H 2450 2450 50  0001 C CNN
 F 3 "~" H 2450 2450 50  0001 C CNN
 	1    2450 2450
@@
 NoConn ~ 2250 5700
 $Sheet
-S 5750 2250 1000 1000
+S 5250 1000 1500 1500
 U 6E7B0394
 F0 "left_OBC" 65
@@
 GLO_KS_2
 $Sheet
-S 7000 3500 1000 1000
+S 5250 3000 1500 1500
 U 5F8745FB
 F0 "right_OBC" 65
 F1 "right_OBC.sch" 50
 $EndSheet
+$Comp
+L Device:R_Small F2
+U 1 1 5FCC3575
+P 10675 6950
+F 0 "F2" V 10779 6950 50  0000 C CNN
+F 1 "R_Small" V 10570 6950 50  0001 C CNN
+F 2 "VST104_footprints:R_SMD_1206" H 10675 6950 50  0001 C CNN
+F 3 "~" H 10675 6950 50  0001 C CNN
+	1    10675 6950
+	0    1    1    0
+$EndComp
+$Comp
+L Device:R_Small F1
+U 1 1 5FCC40A0
+P 10675 6850
+F 0 "F1" V 10571 6850 50  0000 C CNN
+F 1 "R_Small" V 10570 6850 50  0001 C CNN
+F 2 "VST104_footprints:R_SMD_1206" H 10675 6850 50  0001 C CNN
+F 3 "~" H 10675 6850 50  0001 C CNN
+	1    10675 6850
+	0    1    1    0
+$EndComp
+Wire Wire Line
+	10525 6950 10575 6950
+Wire Wire Line
+	10525 6850 10575 6850
+Wire Wire Line
+	10525 6750 10775 6750
+Text GLabel 10525 6850 0    50   Input ~ 0
+SUP_3V3
+$Comp
+L power:GND #PWR0235
+U 1 1 5FCD7750
+P 10525 6750
+F 0 "#PWR0235" H 10525 6500 50  0001 C CNN
+F 1 "GND" V 10530 6622 50  0000 R CNN
+F 2 "" H 10525 6750 50  0001 C CNN
+F 3 "" H 10525 6750 50  0001 C CNN
+	1    10525 6750
+	0    1    1    0
+$EndComp
+Text GLabel 10525 6950 0    50   Input ~ 0
+SUP_5V
+$Comp
+L Connector_Generic:Conn_01x03 UA1
+U 1 1 5FCC19CF
+P 10975 6850
+F 0 "UA1" H 11055 6846 50  0000 L CNN
+F 1 "Conn_01x03" H 11055 6801 50  0001 L CNN
+F 2 "VST104_footprints:PC104_universal_FPGA" H 10975 6850 50  0001 C CNN
+F 3 "~" H 10975 6850 50  0001 C CNN
+	1    10975 6850
+	1    0    0    -1
+$EndComp
+NoConn ~ 9500 5025
+$Comp
+L Connector_Generic:Conn_02x12_Counter_Clockwise UA2
+U 1 1 5FD15277
+P 9700 5525
+F 0 "UA2" H 9750 6150 50  0000 C CNN
+F 1 "Conn_02x12_Counter_Clockwise" H 9750 6151 50  0001 C CNN
+F 2 "VST104_footprints:PC104_SO-24_universal" H 9700 5525 50  0001 C CNN
+F 3 "~" H 9700 5525 50  0001 C CNN
+	1    9700 5525
+	1    0    0    -1
+$EndComp
+NoConn ~ 9500 5125
+NoConn ~ 9500 5225
+NoConn ~ 9500 5325
+NoConn ~ 9500 5425
+NoConn ~ 9500 5525
+NoConn ~ 9500 5625
+NoConn ~ 9500 5725
+NoConn ~ 9500 5825
+NoConn ~ 9500 5925
+NoConn ~ 9500 6025
+NoConn ~ 9500 6125
+NoConn ~ 10000 5025
+NoConn ~ 10000 5125
+NoConn ~ 10000 5225
+NoConn ~ 10000 5325
+NoConn ~ 10000 5425
+NoConn ~ 10000 5525
+NoConn ~ 10000 5625
+NoConn ~ 10000 5725
+NoConn ~ 10000 5825
+NoConn ~ 10000 5925
+NoConn ~ 10000 6025
+NoConn ~ 10000 6125
+NoConn ~ 10250 5025
+$Comp
+L Connector_Generic:Conn_02x12_Counter_Clockwise UA3
+U 1 1 5FD746D2
+P 10450 5525
+F 0 "UA3" H 10500 6150 50  0000 C CNN
+F 1 "Conn_02x12_Counter_Clockwise" H 10500 6151 50  0001 C CNN
+F 2 "VST104_footprints:PC104_SO-24_universal" H 10450 5525 50  0001 C CNN
+F 3 "~" H 10450 5525 50  0001 C CNN
+	1    10450 5525
+	1    0    0    -1
+$EndComp
+NoConn ~ 10250 5125
+NoConn ~ 10250 5225
+NoConn ~ 10250 5325
+NoConn ~ 10250 5425
+NoConn ~ 10250 5525
+NoConn ~ 10250 5625
+NoConn ~ 10250 5725
+NoConn ~ 10250 5825
+NoConn ~ 10250 5925
+NoConn ~ 10250 6025
+NoConn ~ 10250 6125
+NoConn ~ 10750 5025
+NoConn ~ 10750 5125
+NoConn ~ 10750 5225
+NoConn ~ 10750 5325
+NoConn ~ 10750 5425
+NoConn ~ 10750 5525
+NoConn ~ 10750 5625
+NoConn ~ 10750 5725
+NoConn ~ 10750 5825
+NoConn ~ 10750 5925
+NoConn ~ 10750 6025
+NoConn ~ 10750 6125
+Wire Notes Line width 10
+	9250 6250 11000 6250
+Wire Notes Line width 10
+	9250 6250 9250 4750
+Wire Notes Line width 10
+	11000 6250 11000 4750
+Wire Notes Line width 10
+	11000 4750 9250 4750
+Text Notes 9250 4725 0    65   ~ 13
+Universal SO-24 footprint\n
 $EndSCHEMATC
