File: board_delta/right_OBC.sch (KiCad schematic (older format))
At the start: 231 parts, among them M1 S25FL256L, M2 S25FL256L, M3 S25FL256L, M4 CY15B102Q, M5 CY15B102Q, M6 CY15B102Q, Q1 TPS22965-Q1, Q2 TPS22965-Q1, Q3 TPS22965-Q1, U1 STM32L496ZGTx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

Commit message: finished
Parts:
- removed TRC3: trace_0.173mm, VST104_footprints:trace_arc_0.173mm, symbol Connector:TestPoint_Small
